Commit message: add link_without_rotor.urdf.xacro

File: robots/hydrus/robots/quad/soft_airframe_202509/robot.urdf.xacro (robot description, xacro)
@@ -5,8 +5,9 @@
   <xacro:include filename="$(find hydrus)/urdf/common.xacro" />
   <xacro:include filename="$(find hydrus)/urdf/link.urdf.xacro" />
+  <xacro:include filename="$(find hydrus)/urdf/link_without_rotor.urdf.xacro" />
   <xacro:hydrus_link links="4" self="1" rotor_direction="-1" with_battery = "0" tilt_mode="1" tilt_angle="20" />
   <xacro:hydrus_link links="4" self="2" rotor_direction="1"  with_battery = "0" tilt_mode="1" tilt_angle="20" />
   <xacro:hydrus_link links="4" self="3" rotor_direction="-1" with_battery = "0" tilt_mode="1" tilt_angle="20" />
-  <xacro:hydrus_link links="4" self="4" rotor_direction="1"  with_battery = "0" tilt_mode="1" tilt_angle="20" />
+  <xacro:hydrus_link_without_rotor links="4" self="4" rotor_direction="1"  with_battery = "0" tilt_mode="1" tilt_angle="20" />
   <!-- special battery arrangement -->
   <xacro:extra_module name = "bat1" parent = "link1" visible = "1"
@@ -170,12 +171,12 @@
       <mass value="0.0001"/>
       <!-- this is for avoiding error in gazebo -->
-      <!-- <inertia
+      <inertia
           ixx="0.001" ixy="0.0" ixz="0.0"
           iyy="0.001" iyz="0.0"
-          izz="0.002"/> -->
-      <inertia
+          izz="0.002"/>
+      <!-- <inertia
           ixx="0.00001" ixy="0.0" ixz="0.0"
           iyy="0.00001" iyz="0.0"
-          izz="0.00002"/>
+          izz="0.00002"/> -->
     </inertial>
     <visual>
@@ -196,12 +197,12 @@
       <mass value="0.0001"/>
       <!-- this is for avoiding error in gazebo -->
-      <!-- <inertia
+      <inertia
           ixx="0.001" ixy="0.0" ixz="0.0"
           iyy="0.001" iyz="0.0"
-          izz="0.002"/> -->
-      <inertia
+          izz="0.002"/>
+      <!-- <inertia
           ixx="0.00001" ixy="0.0" ixz="0.0"
           iyy="0.00001" iyz="0.0"
-          izz="0.00002"/>
+          izz="0.00002"/> -->
     </inertial>
     <visual>
@@ -338,13 +339,13 @@
       <!-- this inertia value is 10 times bigger than the real one -->
       <!-- to avoid the instability in gazebo -->
-      <!-- <inertia
+      <inertia
           ixx="0.0022661" ixy="0.0" ixz="0.0"
           iyy="0.0015451" iyz="0.0"
-          izz="0.00032533"/> -->
+          izz="0.00032533"/>
       <!-- original one -->
-      <inertia
+      <!-- <inertia
           ixx="0.00022661" ixy="0.0" ixz="0.0"
           iyy="0.00015451" iyz="0.0"
-          izz="0.000032533"/>
+          izz="0.000032533"/> -->
     </inertial>
     <!-- <collision>

Commit message: reduce the rotor num to 4

File: robots/hydrus/robots/quad/soft_airframe_202509/robot.urdf.xacro (robot description, xacro)
@@ -378,12 +378,12 @@
   </transmission>
   <!-- rotor -->
-  <joint name="rotor5" type="continuous">
+  <joint name="rotor4" type="continuous">
     <limit effort="0.0064" lower="1.0" upper="20.0" velocity="0.5"/>
     <parent link="gimbal_link1"/>
-    <child link="thrust5"/>
+    <child link="thrust4"/>
     <origin rpy="0 0 0" xyz="0.0735 0 0"/>
     <axis xyz="0 0 -1"/>
   </joint>
-  <link name="thrust5">
+  <link name="thrust4">
     <inertial>
       <origin xyz="0 0 0" rpy="0 0 0"/>
@@ -407,11 +407,11 @@
     </visual>
   </link>
-  <xacro:damping_factor link ="thrust5"/>
+  <xacro:damping_factor link ="thrust4"/>
   <transmission name="rotor_tran5">
     <type>transmission_interface/SimpleTransmission</type>
-    <joint name="rotor5">
+    <joint name="rotor4">
       <hardwareInterface>RotorInterface</hardwareInterface>
-    </joint>
-    <actuator name="rotor5">
+    </joint>thrust5
+    <actuator name="rotor4">
       <hardwareInterface>RotorInterface</hardwareInterface>
       <mechanicalReduction>1</mechanicalReduction>

File: robots/hydrus/urdf/link_without_rotor.urdf.xacro (robot description, xacro)
@@ -187,8 +187,8 @@
     <xacro:damping_factor link ="link${self}"/>
     <!-- rotor -->
-    <joint name="rotor${self}" type="continuous">
+    <joint name="rt${self}" type="continuous">
       <limit effort="0.0172" lower="${min_force}" upper="${max_force}" velocity="0.5"/>
       <parent link="link${self}"/>
-      <child link="thrust${self}"/>
+      <child link="th${self}"/>
       <xacro:if value="${tilt_mode == 1}">
         <xacro:if value="${prop_15inch == 1}">
@@ -204,5 +204,5 @@
       <axis xyz="0 0 ${rotor_direction}"/>
     </joint>
-    <link name="thrust${self}">
+    <link name="th${self}">
       <!-- visual & collisiont -->
       <inertial>
@@ -232,5 +232,5 @@
       </visual>
     </link>
-    <xacro:damping_factor link ="thrust${self}"/>
+    <xacro:damping_factor link ="th${self}"/>
     <!-- battery: -->
     <!-- use default battery: -->
@@ -335,16 +335,4 @@
       </transmission>
     </xacro:unless>
-    <transmission name="rotor_tran${self}">
-      <type>transmission_interface/SimpleTransmission</type>
-      <joint name="rotor${self}">
-        <!-- TODO: effort is torque, maybe position is enough -->
-        <hardwareInterface>RotorInterface</hardwareInterface>
-      </joint>
-      <actuator name="rotor${self}">
-        <!-- TODO: effort is torque, maybe position is enough -->
-        <hardwareInterface>RotorInterface</hardwareInterface>
-        <mechanicalReduction>1</mechanicalReduction>
-      </actuator>
-    </transmission>
     <xacro:friction self ="${self}"/>
   </xacro:macro>

Commit message: modify to for the current hardware

File: robots/hydrus/robots/quad/soft_airframe_202509/robot.urdf.xacro (robot description, xacro)
@@ -105,9 +105,14 @@
     <inertial>
       <origin xyz="0.06875 0.000002 0.018960" rpy="0 0 0"/>
-      <mass value="${0.010*2 + 0.012}"/>
-      <inertia
-          ixx="0.00003988" ixy="0.0" ixz="0.0"
-          iyy="0.00010606" iyz="0.0"
-          izz="0.00010185"/>
+      <mass value="0.0001"/>
+      <!-- this is for avoiding error in gazebo -->
+      <!-- <inertia
+          ixx="0.001" ixy="0.0" ixz="0.0"
+          iyy="0.001" iyz="0.0"
+          izz="0.002"/> -->
+      <inertia
+          ixx="0.00001" ixy="0.0" ixz="0.0"
+          iyy="0.00001" iyz="0.0"
+          izz="0.00002"/>
     </inertial>
     <visual>
@@ -126,9 +131,14 @@
     <inertial>
       <origin xyz="0.1175 0.000002 0.019998" rpy="0 0 0"/>
-      <mass value="${0.010*5 + 0.012*2}"/>
-      <inertia
-          ixx="0.00006787" ixy="0.0" ixz="0.0"
-          iyy="0.00049831" iyz="0.0"
-          izz="0.00048990"/>
+      <mass value="0.0001"/>
+      <!-- this is for avoiding error in gazebo -->
+      <!-- <inertia
+          ixx="0.001" ixy="0.0" ixz="0.0"
+          iyy="0.001" iyz="0.0"
+          izz="0.002"/> -->
+      <inertia
+          ixx="0.00001" ixy="0.0" ixz="0.0"
+          iyy="0.00001" iyz="0.0"
+          izz="0.00002"/>
     </inertial>
     <visual>
@@ -147,9 +157,14 @@
     <inertial>
       <origin xyz="0.10740316 0.0 0.003" rpy="0 0 0"/>
-      <mass value="${0.010*2 + 0.012 + 0.070 + 0.016}"/>
-      <inertia
-          ixx="0.00005679" ixy="-0.000000031" ixz="-0.00002256"
-          iyy="0.00028149" iyz="0.000000005"
-          izz="0.00026759"/>
+      <mass value="0.0001"/>
+      <!-- this is for avoiding error in gazebo -->
+      <!-- <inertia
+          ixx="0.001" ixy="0.0" ixz="0.0"
+          iyy="0.001" iyz="0.0"
+          izz="0.002"/> -->
+      <inertia
+          ixx="0.00001" ixy="0.0" ixz="0.0"
+          iyy="0.00001" iyz="0.0"
+          izz="0.00002"/>
     </inertial>
     <visual>
@@ -301,8 +316,14 @@
     <inertial>
       <origin xyz="0.0 0.0 -0.093" rpy="0 0 0"/>
-      <mass value="0.051000"/>
-      <inertia
-          ixx="0.000122" iyy="0.000133" izz="0.000012"
-          ixy="0.000000" ixz="0.000000" iyz="0.000000"/>
+      <mass value="0.0001"/>
+      <!-- this is for avoiding error in gazebo -->
+      <inertia
+          ixx="0.001" ixy="0.0" ixz="0.0"
+          iyy="0.001" iyz="0.0"
+          izz="0.002"/>
+      <!-- <inertia
+          ixx="0.00001" ixy="0.0" ixz="0.0"
+          iyy="0.00001" iyz="0.0"
+          izz="0.00002"/> -->
     </inertial>
     <visual>
@@ -335,16 +356,14 @@
     <inertial>
       <origin xyz="0.0815 0 0" rpy="0 0 0"/>
-      <mass value="0.173"/>
-      <!-- this inertia value is 10 times bigger than the real one -->
-      <!-- to avoid the instability in gazebo -->
-      <!-- <inertia
-          ixx="0.0022661" ixy="0.0" ixz="0.0"
-          iyy="0.0015451" iyz="0.0"
-          izz="0.00032533"/> -->
-      <!-- original one -->
-      <inertia
-          ixx="0.00022661" ixy="0.0" ixz="0.0"
-          iyy="0.00015451" iyz="0.0"
-          izz="0.000032533"/>
+      <mass value="0.0001"/>
+      <!-- this is for avoiding error in gazebo -->
+      <inertia
+          ixx="0.001" ixy="0.0" ixz="0.0"
+          iyy="0.001" iyz="0.0"
+          izz="0.002"/>
+      <!-- <inertia
+          ixx="0.00001" ixy="0.0" ixz="0.0"
+          iyy="0.00001" iyz="0.0"
+          izz="0.00002"/> -->
     </inertial>
     <!-- <collision>

Commit message: allow to transform the soft airframe

File: robots/hydrus/robots/quad/soft_airframe_202509/robot.urdf.xacro (robot description, xacro)
@@ -217,4 +217,56 @@
   </gazebo>
   <xacro:damping_factor link="dummy_link1"/>
+  <link name="dummy_link2">
+    <inertial>
+      <origin xyz="0 0 0" rpy="0 0 0"/>
+      <mass value="0.0001"/>
+      <!-- this is for avoiding error in gazebo -->
+      <!-- <inertia
+          ixx="0.001" ixy="0.0" ixz="0.0"
+          iyy="0.001" iyz="0.0"
+          izz="0.002"/> -->
+      <inertia
+          ixx="0.000016" ixy="-0.000003" ixz="0.000001"
+          iyy="0.000019" iyz="0.000000"
+          izz="0.000022"/>
+    </inertial>
+    <visual>
+      <geometry>
+        <box size="0.05 0.05 0.05"/>
+      </geometry>
+      <origin xyz="0 0 -0.02" rpy="0 0 0"/>
+    </visual>
+  </link>
+  <gazebo reference="dummy_link2">
+    <mu1>0.1</mu1>
+    <mu2>0.1</mu2>
+  </gazebo>
+  <xacro:damping_factor link="dummy_link2"/>
+  <link name="dummy_link3">
+    <inertial>
+      <origin xyz="0 0 0" rpy="0 0 0"/>
+      <mass value="0.0001"/>
+      <!-- this is for avoiding error in gazebo -->
+      <!-- <inertia
+          ixx="0.001" ixy="0.0" ixz="0.0"
+          iyy="0.001" iyz="0.0"
+          izz="0.002"/> -->
+      <inertia
+          ixx="0.000016" ixy="-0.000003" ixz="0.000001"
+          iyy="0.000019" iyz="0.000000"
+          izz="0.000022"/>
+    </inertial>
+    <visual>
+      <geometry>
+        <box size="0.05 0.05 0.05"/>
+      </geometry>
+      <origin xyz="0 0 -0.02" rpy="0 0 0"/>
+    </visual>
+  </link>
+  <gazebo reference="dummy_link3">
+    <mu1>0.1</mu1>
+    <mu2>0.1</mu2>
+  </gazebo>
+  <xacro:damping_factor link="dummy_link3"/>
   <joint name="soft_joint1" type="fixed">
     <parent link="link4"/>
@@ -257,4 +309,20 @@
     <dynamics damping="0.9" friction="0.1"/>
   </joint>
+  <joint name="soft_joint6" type="revolute">
+    <limit effort="5.0" lower="${-pi/2}" upper="${pi/2}" velocity="0.5"/>
+    <parent link="soft_link3"/>
+    <child link="dummy_link2"/>
+    <origin xyz="0.235 0 0" rpy="0 0 0"/>
+    <axis xyz="0 0 1"/>
+    <dynamics damping="0.9" friction="0.1"/>
+  </joint>
+  <joint name="soft_joint7" type="revolute">
+    <limit effort="5.0" lower="${-pi/2}" upper="${pi/2}" velocity="0.5"/>
+    <parent link="soft_link3"/>
+    <child link="dummy_link3"/>
+    <origin xyz="0.235 0 0" rpy="0 0 0"/>
+    <axis xyz="0 0 1"/>
+    <dynamics damping="0.9" friction="0.1"/>
+  </joint>
   <transmission name="soft_joint_tran_2">
     <type>transmission_interface/SimpleTransmission</type>
@@ -293,4 +361,24 @@
     </joint>
     <actuator name="soft_joint_servo5">
+      <hardwareInterface>hardware_interface/EffortJointInterface</hardwareInterface>
+      <mechanicalReduction>1</mechanicalReduction>
+    </actuator>
+  </transmission>
+  <transmission name="soft_joint_tran_6">
+    <type>transmission_interface/SimpleTransmission</type>
+    <joint name="soft_joint6">
+      <hardwareInterface>hardware_interface/EffortJointInterface</hardwareInterface>
+    </joint>
+    <actuator name="soft_joint_servo6">
+      <hardwareInterface>hardware_interface/EffortJointInterface</hardwareInterface>
+      <mechanicalReduction>1</mechanicalReduction>
+    </actuator>
+  </transmission>
+  <transmission name="soft_joint_tran_7">
+    <type>transmission_interface/SimpleTransmission</type>
+    <joint name="soft_joint7">
+      <hardwareInterface>hardware_interface/EffortJointInterface</hardwareInterface>
+    </joint>
+    <actuator name="soft_joint_servo7">
       <hardwareInterface>hardware_interface/EffortJointInterface</hardwareInterface>
       <mechanicalReduction>1</mechanicalReduction>

Commit message: fly with transformed robot modelg

File: robots/hydrus/robots/quad/soft_airframe_202509/robot.urdf.xacro (robot description, xacro)
@@ -217,56 +217,4 @@
   </gazebo>
   <xacro:damping_factor link="servo_link1"/>
-  <link name="dummy_link2">
-    <inertial>
-      <origin xyz="0 0 0" rpy="0 0 0"/>
-      <mass value="0.0001"/>
-      <!-- this is for avoiding error in gazebo -->
-      <!-- <inertia
-          ixx="0.001" ixy="0.0" ixz="0.0"
-          iyy="0.001" iyz="0.0"
-          izz="0.002"/> -->
-      <inertia
-          ixx="0.000016" ixy="-0.000003" ixz="0.000001"
-          iyy="0.000019" iyz="0.000000"
-          izz="0.000022"/>
-    </inertial>
-    <visual>
-      <geometry>
-        <box size="0.05 0.05 0.05"/>
-      </geometry>
-      <origin xyz="0 0 -0.02" rpy="0 0 0"/>
-    </visual>
-  </link>
-  <gazebo reference="dummy_link2">
-    <mu1>0.1</mu1>
-    <mu2>0.1</mu2>
-  </gazebo>
-  <xacro:damping_factor link="dummy_link2"/>
-  <link name="dummy_link3">
-    <inertial>
-      <origin xyz="0 0 0" rpy="0 0 0"/>
-      <mass value="0.0001"/>
-      <!-- this is for avoiding error in gazebo -->
-      <!-- <inertia
-          ixx="0.001" ixy="0.0" ixz="0.0"
-          iyy="0.001" iyz="0.0"
-          izz="0.002"/> -->
-      <inertia
-          ixx="0.000016" ixy="-0.000003" ixz="0.000001"
-          iyy="0.000019" iyz="0.000000"
-          izz="0.000022"/>
-    </inertial>
-    <visual>
-      <geometry>
-        <box size="0.05 0.05 0.05"/>
-      </geometry>
-      <origin xyz="0 0 -0.02" rpy="0 0 0"/>
-    </visual>
-  </link>
-  <gazebo reference="dummy_link3">
-    <mu1>0.1</mu1>
-    <mu2>0.1</mu2>
-  </gazebo>
-  <xacro:damping_factor link="dummy_link3"/>
   <joint name="soft_joint1" type="fixed">
     <parent link="link4"/>
@@ -309,20 +257,4 @@
     <dynamics damping="0.9" friction="0.1"/>
   </joint>
-  <joint name="soft_joint6" type="revolute">
-    <limit effort="5.0" lower="${-pi/2}" upper="${pi/2}" velocity="0.5"/>
-    <parent link="soft_link3"/>
-    <child link="dummy_link2"/>
-    <origin xyz="0.235 0 0" rpy="0 0 0"/>
-    <axis xyz="0 0 1"/>
-    <dynamics damping="0.9" friction="0.1"/>
-  </joint>
-  <joint name="soft_joint7" type="revolute">
-    <limit effort="5.0" lower="${-pi/2}" upper="${pi/2}" velocity="0.5"/>
-    <parent link="soft_link3"/>
-    <child link="dummy_link3"/>
-    <origin xyz="0.235 0 0" rpy="0 0 0"/>
-    <axis xyz="0 0 1"/>
-    <dynamics damping="0.9" friction="0.1"/>
-  </joint>
   <transmission name="soft_joint_tran_2">
     <type>transmission_interface/SimpleTransmission</type>
@@ -361,24 +293,4 @@
     </joint>
     <actuator name="soft_joint_servo5">
-      <hardwareInterface>hardware_interface/EffortJointInterface</hardwareInterface>
-      <mechanicalReduction>1</mechanicalReduction>
-    </actuator>
-  </transmission>
-  <transmission name="soft_joint_tran_6">
-    <type>transmission_interface/SimpleTransmission</type>
-    <joint name="soft_joint6">
-      <hardwareInterface>hardware_interface/EffortJointInterface</hardwareInterface>
-    </joint>
-    <actuator name="soft_joint_servo6">
-      <hardwareInterface>hardware_interface/EffortJointInterface</hardwareInterface>
-      <mechanicalReduction>1</mechanicalReduction>
-    </actuator>
-  </transmission>
-  <transmission name="soft_joint_tran_7">
-    <type>transmission_interface/SimpleTransmission</type>
-    <joint name="soft_joint7">
-      <hardwareInterface>hardware_interface/EffortJointInterface</hardwareInterface>
-    </joint>
-    <actuator name="soft_joint_servo7">
       <hardwareInterface>hardware_interface/EffortJointInterface</hardwareInterface>
       <mechanicalReduction>1</mechanicalReduction>

Commit message: change the servo

File: robots/hydrus/robots/quad/soft_airframe_202509/robot.urdf.xacro (robot description, xacro)
@@ -168,5 +168,5 @@
     <inertial>
       <origin xyz="0 0 0" rpy="0 0 0"/>
-      <mass value="0.064"/>
+      <mass value="0.074"/>
       <!-- this is for avoiding error in gazebo -->
       <!-- <inertia
@@ -194,5 +194,5 @@
     <inertial>
       <origin xyz="0 0 0" rpy="0 0 0"/>
-      <mass value="0.059"/>
+      <mass value="0.069"/>
       <!-- this is for avoiding error in gazebo -->
       <!-- <inertia

Commit message: change the position of spinal

File: robots/hydrus/robots/quad/soft_airframe_202509/robot.urdf.xacro (robot description, xacro)
@@ -37,5 +37,5 @@
   <xacro:extra_module name = "fc" parent = "link3" visible = "1"
                       model_url = "package://hydrus/urdf/mesh/ver2/flight_controller/spinal.dae"> <!-- same with intel euclid -->
-    <origin xyz="${link_length / 2 - 0.2221} ${-4.4*0.001} -0.02135" rpy="0 0 0"/>
+    <origin xyz="${link_length / 2 - 0.2221} ${-4.4*0.001} 0.02135" rpy="0 0 0"/>
     <inertial>
       <mass value = "0.05" />
@@ -168,5 +168,5 @@
     <inertial>
       <origin xyz="0 0 0" rpy="0 0 0"/>
-      <mass value="0.074"/>
+      <mass value="0.064"/>
       <!-- this is for avoiding error in gazebo -->
       <!-- <inertia
@@ -194,5 +194,5 @@
     <inertial>
       <origin xyz="0 0 0" rpy="0 0 0"/>
-      <mass value="0.069"/>
+      <mass value="0.059"/>
       <!-- this is for avoiding error in gazebo -->
       <!-- <inertia
