Commit message: add soft_link2

File: robots/hydrus/robots/quad/soft_airframe_202509/robot.urdf.xacro (robot description, xacro)
@@ -101,13 +101,35 @@
   </xacro:extra_module>
   <!-- end: gps -->
-  <!-- 3 soft_airframe -->
+  <!-- 3 soft_airframe_1 -->
+  <!-- soft_link -->
+  <joint name="soft_joint1" type="fixed">
+    <parent link="link4"/>
+    <child link="soft_link1"/>
+    <origin xyz="0.6 0 0" rpy="0 0 0"/>
+  </joint>
+  <joint name="soft_joint2" type="revolute">
+    <limit effort="5.0" lower="${-pi/2}" upper="${pi/2}" velocity="0.5"/>
+    <parent link="soft_link1"/>
+    <child link="soft_link2"/>
+    <origin xyz="0.1175 0 0" rpy="0 0 0"/>
+    <axis xyz="0 0 1"/>
+    <dynamics damping="0.9" friction="0.1"/>
+  </joint>
+  <joint name="soft_joint3" type="revolute">
+    <limit effort="5.0" lower="${-pi/2}" upper="${pi/2}" velocity="0.5"/>
+    <parent link="soft_link2"/>
+    <child link="soft_link3"/>
+    <origin xyz="0.235 0 0" rpy="0 0 0"/>
+    <axis xyz="0 0 1"/>
+    <dynamics damping="0.9" friction="0.1"/>
+  </joint>
   <link name="soft_link1">
     <inertial>
-      <origin xyz="0.06875 0.000002 0.018960" rpy="0 0 0"/>
-      <mass value="${0.010*2 + 0.012}"/>
-      <inertia
-          ixx="0.00003988" ixy="0.0" ixz="0.0"
-          iyy="0.00010606" iyz="0.0"
-          izz="0.00010185"/>
+      <origin xyz="0.064 0.000002 0.018960" rpy="0 0 0"/>
+      <mass value="0.059"/>
+      <inertia
+          ixx="0.00005433" ixy="0.00000033" ixz="0.0"
+          iyy="0.00047358" iyz="-0.00000369"
+          izz="0.00046011"/>
     </inertial>
     <visual>
@@ -125,10 +147,10 @@
   <link name="soft_link2">
     <inertial>
-      <origin xyz="0.1175 0.000002 0.019998" rpy="0 0 0"/>
-      <mass value="${0.010*5 + 0.012*2}"/>
-      <inertia
-          ixx="0.00006787" ixy="0.0" ixz="0.0"
-          iyy="0.00049831" iyz="0.0"
-          izz="0.00048990"/>
+      <origin xyz="0.118 0.000002 0.019998" rpy="0 0 0"/>
+      <mass value="0.118"/>
+      <inertia
+          ixx="0.00007941" ixy="0.00000218" ixz="0.0"
+          iyy="0.00065133" iyz="0.0"
+          izz="0.00062639"/>
     </inertial>
     <visual>
@@ -147,9 +169,9 @@
     <inertial>
       <origin xyz="0.10740316 0.0 0.003" rpy="0 0 0"/>
-      <mass value="${0.010*2 + 0.012 + 0.070 + 0.016}"/>
-      <inertia
-          ixx="0.00005679" ixy="-0.000000031" ixz="-0.00002256"
-          iyy="0.00028149" iyz="0.000000005"
-          izz="0.00026759"/>
+      <mass value="0.059"/>
+      <inertia
+          ixx="0.00005433" ixy="0.00000033" ixz="0.0"
+          iyy="0.00047358" iyz="-0.00000369"
+          izz="0.00046011"/>
     </inertial>
     <visual>
@@ -165,5 +187,42 @@
   </gazebo>
   <xacro:damping_factor link="soft_link3"/>
-  <link name="servo_link">
+  <transmission name="soft_joint_tran_2">
+    <type>transmission_interface/SimpleTransmission</type>
+    <joint name="soft_joint2">
+      <hardwareInterface>hardware_interface/EffortJointInterface</hardwareInterface>
+    </joint>
+    <actuator name="soft_joint_servo2">
+      <hardwareInterface>hardware_interface/EffortJointInterface</hardwareInterface>
+      <mechanicalReduction>1</mechanicalReduction>
+    </actuator>
+  </transmission>
+  <transmission name="soft_joint_tran_3">
+    <type>transmission_interface/SimpleTransmission</type>
+    <joint name="soft_joint3">
+      <hardwareInterface>hardware_interface/EffortJointInterface</hardwareInterface>
+    </joint>
+    <actuator name="soft_joint_servo3">
+      <hardwareInterface>hardware_interface/EffortJointInterface</hardwareInterface>
+      <mechanicalReduction>1</mechanicalReduction>
+    </actuator>
+  </transmission>
+  <!-- dummy_link -->
+  <joint name="servo_joint1" type="revolute">
+    <limit effort="5.0" lower="${-pi/2}" upper="${pi/2}" velocity="0.5"/>
+    <parent link="link4"/>
+    <child link="servo_link1"/>
+    <origin xyz="0.5 0 0.01" rpy="0 0 0"/>
+    <axis xyz="0 0 1"/>
+    <dynamics damping="0.9" friction="0.1"/>
+  </joint>
+  <joint name="servo_joint2" type="revolute">
+    <limit effort="5.0" lower="${-pi/2}" upper="${pi/2}" velocity="0.5"/>
+    <parent link="link4"/>
+    <child link="servo_link2"/>
+    <origin xyz="0.5 0 -0.01" rpy="0 0 0"/>
+    <axis xyz="0 0 1"/>
+    <dynamics damping="0.9" friction="0.1"/>
+  </joint>
+  <link name="servo_link1">
     <inertial>
       <origin xyz="0 0 0" rpy="0 0 0"/>
@@ -175,7 +234,7 @@
           izz="0.002"/> -->
       <inertia
-          ixx="0.000017" ixy="0.000003" ixz="-0.0000001"
-          iyy="0.000023" iyz="0.000000"
-          izz="0.000025"/>
+          ixx="0.000023" ixy="0.000003" ixz="-0.0000001"
+          iyy="0.000044" iyz="0.000000"
+          izz="0.000043"/>
     </inertial>
     <visual>
@@ -186,10 +245,5 @@
     </visual>
   </link>
-  <gazebo reference="servo_link">
-    <mu1>0.1</mu1>
-    <mu2>0.1</mu2>
-  </gazebo>
-  <xacro:damping_factor link="servo_link"/>
-  <link name="servo_link1">
+  <link name="servo_link2">
     <inertial>
       <origin xyz="0 0 0" rpy="0 0 0"/>
@@ -201,7 +255,7 @@
           izz="0.002"/> -->
       <inertia
-          ixx="0.000016" ixy="-0.000003" ixz="0.000001"
-          iyy="0.000019" iyz="0.000000"
-          izz="0.000022"/>
+          ixx="0.000022" ixy="-0.000003" ixz="0.000001"
+          iyy="0.000042" iyz="0.000000"
+          izz="0.000041"/>
     </inertial>
     <visual>
@@ -212,85 +266,20 @@
     </visual>
   </link>
-  <gazebo reference="servo_link1">
-    <mu1>0.1</mu1>
-    <mu2>0.1</mu2>
-  </gazebo>
-  <xacro:damping_factor link="servo_link1"/>
-  <joint name="soft_joint1" type="fixed">
-    <parent link="link4"/>
-    <child link="soft_link1"/>
-    <origin xyz="0.6 0 0" rpy="0 0 0"/>
-  </joint>
-  <joint name="soft_joint2" type="revolute">
-    <limit effort="5.0" lower="${-pi/2}" upper="${pi/2}" velocity="0.5"/>
-    <parent link="soft_link1"/>
-    <child link="soft_link2"/>
-    <origin xyz="0.1175 0 0" rpy="0 0 0"/>
-    <axis xyz="0 0 1"/>
-    <dynamics damping="0.9" friction="0.1"/>
-  </joint>
-  <joint name="soft_joint3" type="revolute">
-    <limit effort="5.0" lower="${-pi/2}" upper="${pi/2}" velocity="0.5"/>
-    <parent link="soft_link2"/>
-    <child link="soft_link3"/>
-    <origin xyz="0.235 0 0" rpy="0 0 0"/>
-    <axis xyz="0 0 1"/>
-    <dynamics damping="0.9" friction="0.1"/>
-  </joint>
-  <!-- <gazebo reference="soft_link3">
-    <stopCfm>1000</stopCfm>
-  </gazebo> -->
-  <joint name="soft_joint4" type="revolute">
-    <limit effort="5.0" lower="${-pi/2}" upper="${pi/2}" velocity="0.5"/>
-    <parent link="link4"/>
-    <child link="servo_link"/>
-    <origin xyz="0.5 0 0.01" rpy="0 0 0"/>
-    <axis xyz="0 0 1"/>
-    <dynamics damping="0.9" friction="0.1"/>
-  </joint>
-  <joint name="soft_joint5" type="revolute">
-    <limit effort="5.0" lower="${-pi/2}" upper="${pi/2}" velocity="0.5"/>
-    <parent link="link4"/>
-    <child link="servo_link1"/>
-    <origin xyz="0.5 0 -0.01" rpy="0 0 0"/>
-    <axis xyz="0 0 1"/>
-    <dynamics damping="0.9" friction="0.1"/>
-  </joint>
-  <transmission name="soft_joint_tran_2">
-    <type>transmission_interface/SimpleTransmission</type>
-    <joint name="soft_joint2">
-      <hardwareInterface>hardware_interface/EffortJointInterface</hardwareInterface>
-    </joint>
-    <actuator name="soft_joint_servo2">
-      <hardwareInterface>hardware_interface/EffortJointInterface</hardwareInterface>
-      <mechanicalReduction>1</mechanicalReduction>
-    </actuator>
-  </transmission>
-  <transmission name="soft_joint_tran_3">
-    <type>transmission_interface/SimpleTransmission</type>
-    <joint name="soft_joint3">
-      <hardwareInterface>hardware_interface/EffortJointInterface</hardwareInterface>
-    </joint>
-    <actuator name="soft_joint_servo3">
-      <hardwareInterface>hardware_interface/EffortJointInterface</hardwareInterface>
-      <mechanicalReduction>1</mechanicalReduction>
-    </actuator>
-  </transmission>
-  <transmission name="soft_joint_tran_4">
-    <type>transmission_interface/SimpleTransmission</type>
-    <joint name="soft_joint4">
-      <hardwareInterface>hardware_interface/EffortJointInterface</hardwareInterface>
-    </joint>
-    <actuator name="soft_joint_servo4">
-      <hardwareInterface>hardware_interface/EffortJointInterface</hardwareInterface>
-      <mechanicalReduction>1</mechanicalReduction>
-    </actuator>
-  </transmission>
-  <transmission name="soft_joint_tran_5">
-    <type>transmission_interface/SimpleTransmission</type>
-    <joint name="soft_joint5">
-      <hardwareInterface>hardware_interface/EffortJointInterface</hardwareInterface>
-    </joint>
-    <actuator name="soft_joint_servo5">
+  <transmission name="servo_joint_tran_1">
+    <type>transmission_interface/SimpleTransmission</type>
+    <joint name="servo_joint1">
+      <hardwareInterface>hardware_interface/EffortJointInterface</hardwareInterface>
+    </joint>
+    <actuator name="servo_joint_servo1">
+      <hardwareInterface>hardware_interface/EffortJointInterface</hardwareInterface>
+      <mechanicalReduction>1</mechanicalReduction>
+    </actuator>
+  </transmission>
+  <transmission name="servo_joint_tran_2">
+    <type>transmission_interface/SimpleTransmission</type>
+    <joint name="servo_joint2">
+      <hardwareInterface>hardware_interface/EffortJointInterface</hardwareInterface>
+    </joint>
+    <actuator name="servo_joint_servo2">
       <hardwareInterface>hardware_interface/EffortJointInterface</hardwareInterface>
       <mechanicalReduction>1</mechanicalReduction>
@@ -301,5 +290,5 @@
     <inertial>
       <origin xyz="0.0 0.0 -0.093" rpy="0 0 0"/>
-      <mass value="0.051000"/>
+      <mass value="0.016000"/>
       <inertia
           ixx="0.000122" iyy="0.000133" izz="0.000012"
@@ -312,4 +301,10 @@
       <origin xyz="0.01 0.01 -0.075" rpy="0 0 0"/>
     </visual>
+    <collision>
+      <geometry>
+        <box size="0.02 0.02 -0.15"/>
+      </geometry>
+      <origin xyz="0.01 0.01 -0.075" rpy="0 0 0"/>
+    </collision>
   </link>
   <gazebo reference="leg6">
@@ -324,16 +319,16 @@
   </joint>
   <!-- gimbal -->
-  <joint name="gimbal_joint1" type="revolute">
+  <joint name="gimbal_joint5" type="fixed">
     <limit effort="5.0" lower="${-pi}" upper="${pi}" velocity="0.5"/>
     <parent link="soft_link3"/>
-    <child link="gimbal_link1"/>
-    <origin rpy="0 0 0" xyz="0.1595 0 0"/>
+    <child link="gimbal_link5"/>
+    <origin rpy="0 0 0" xyz="0.128 0 0"/>
     <axis xyz="1 0 0"/>
     <dynamics damping="0.9" friction="0.1"/>
   </joint>
-  <link name="gimbal_link1">
+  <link name="gimbal_link5">
     <inertial>
       <origin xyz="0.0815 0 0" rpy="0 0 0"/>
-      <mass value="0.173"/>
+      <mass value="0.222"/>
       <!-- this inertia value is 10 times bigger than the real one -->
       <!-- to avoid the instability in gazebo -->
@@ -348,36 +343,20 @@
           izz="0.000032533"/>
     </inertial>
-    <!-- <collision>
+    <visual>
       <origin xyz="0.0815 0 0" rpy="0 0 0"/>
       <geometry>
-        <cylinder length="0.1" radius="0.05"/>
-      </geometry>
-    </collision> -->
-    <visual>
-      <origin xyz="0.0815 0 0" rpy="0 0 0"/>
-      <geometry>
         <mesh filename="package://hydrus/urdf/mesh/propeller/5inch_propeller_duct_right_v2.dae"/>
       </geometry>
     </visual>
   </link>
-  <gazebo reference="gimbal_link1">
-    <mu1>0.1</mu1>
-    <mu2>0.1</mu2>
-  </gazebo>
-  <xacro:damping_factor link ="gimbal_link1"/>
-  <transmission name="gimbal_tran1">
-    <type>transmission_interface/SimpleTransmission</type>
-    <joint name="gimbal_joint1">
-      <hardwareInterface>hardware_interface/EffortJointInterface</hardwareInterface>
-    </joint>
-    <actuator name="gimbal_servo1">
-      <hardwareInterface>hardware_interface/EffortJointInterface</hardwareInterface>
-      <mechanicalReduction>1</mechanicalReduction>
-    </actuator>
-  </transmission>
+  <gazebo reference="gimbal_link5">
+    <mu1>0.1</mu1>
+    <mu2>0.1</mu2>
+  </gazebo>
+  <xacro:damping_factor link ="gimbal_link5"/>
   <!-- rotor -->
   <joint name="rotor5" type="continuous">
-    <limit effort="0.0064" lower="1.0" upper="20.0" velocity="0.5"/>
-    <parent link="gimbal_link1"/>
+    <limit effort="0.0064" lower="0.0" upper="20.0" velocity="0.5"/>
+    <parent link="gimbal_link5"/>
     <child link="thrust5"/>
     <origin rpy="0 0 0" xyz="0.0735 0 0"/>
@@ -393,10 +372,4 @@
           izz="0.00002"/>
     </inertial>
-    <!-- <collision>
-      <origin rpy="0 0 0" xyz="0 0 0"/>
-      <geometry>
-        <cylinder length="0.1" radius="0.11"/>
-      </geometry>
-    </collision> -->
     <visual>
       <origin rpy="${pi/2} 0 0" xyz="-0.045 0.055 0.06"/>
@@ -417,3 +390,208 @@
     </actuator>
   </transmission>
+  <!-- 3 soft_airframe_2 -->
+  <!-- soft_link -->
+  <joint name="soft_joint4" type="fixed">
+    <parent link="gimbal_link5"/>
+    <child link="soft_link4"/>
+    <origin xyz="0.147 0 0" rpy="0 0 0"/>
+  </joint>
+  <joint name="soft_joint5" type="revolute">
+    <limit effort="5.0" lower="${-pi/2}" upper="${pi/2}" velocity="0.5"/>
+    <parent link="soft_link4"/>
+    <child link="soft_link5"/>
+    <origin xyz="0.2215 0 0" rpy="0 0 0"/>
+    <axis xyz="0 0 1"/>
+    <dynamics damping="0.9" friction="0.1"/>
+  </joint>
+  <joint name="soft_joint6" type="revolute">
+    <limit effort="5.0" lower="${-pi/2}" upper="${pi/2}" velocity="0.5"/>
+    <parent link="soft_link5"/>
+    <child link="soft_link6"/>
+    <origin xyz="0.235 0 0" rpy="0 0 0"/>
+    <axis xyz="0 0 1"/>
+    <dynamics damping="0.9" friction="0.1"/>
+  </joint>
+  <link name="soft_link4">
+    <inertial>
+      <origin xyz="0.101 0.000002 0.018960" rpy="0 0 0"/>
+      <mass value="${0.059 + 0.157}"/>
+      <inertia
+          ixx="0.00013185" ixy="-0.00000146" ixz="0.00000096"
+          iyy="0.00055113" iyz="-0.00000218"
+          izz="0.00050648"/>
+    </inertial>
+    <visual>
+      <geometry>
+        <box size="0.2215 0.03 0.04"/>
+      </geometry>
+      <origin xyz="0.11075 0 0.02" rpy="0 0 0"/>
+    </visual>
+  </link>
+  <gazebo reference="soft_link4">
+    <mu1>0.1</mu1>
+    <mu2>0.1</mu2>
+  </gazebo>
+  <xacro:damping_factor link="soft_link4"/>
+  <link name="soft_link5">
+    <inertial>
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