Commit message: create dummy links for transforming robot model

File: robots/delta/robots/quad/20240722/delta.urdf.xacro (robot description, xacro)
@@ -171,5 +171,5 @@
     <limit effort="5.0" lower="${-pi/2}" upper="${pi/2}" velocity="0.5"/>
     <parent link="link4"/>
-    <child link="servo_link"/>
+    <child link="servo_link1"/>
     <origin xyz="0.5 0 0.01" rpy="0 0 0"/>
     <axis xyz="0 0 1"/>
@@ -179,10 +179,24 @@
     <limit effort="5.0" lower="${-pi/2}" upper="${pi/2}" velocity="0.5"/>
     <parent link="link4"/>
-    <child link="servo_link1"/>
+    <child link="servo_link2"/>
     <origin xyz="0.5 0 -0.01" rpy="0 0 0"/>
     <axis xyz="0 0 1"/>
     <dynamics damping="0.9" friction="0.1"/>
   </joint>
-  <link name="servo_link">
+  <joint name="soft_joint6" type="revolute">
+    <limit effort="5.0" lower="${-pi/2}" upper="${pi/2}" velocity="0.5"/>
+    <parent link="link4"/>
+    <child link="dummy_link1"/>
+    <origin rpy="0 0 0" xyz="0.0735 0 0"/>
+    <axis xyz="0 0 -1"/>
+  </joint>
+  <joint name="soft_joint7" type="revolute">
+    <limit effort="5.0" lower="${-pi/2}" upper="${pi/2}" velocity="0.5"/>
+    <parent link="link4"/>
+    <child link="dummy_link2"/>
+    <origin rpy="0 0 0" xyz="0.0735 0 0"/>
+    <axis xyz="0 0 -1"/>
+  </joint>
+  <link name="servo_link1">
     <inertial>
       <origin xyz="0 0 0" rpy="0 0 0"/>
@@ -205,10 +219,5 @@
     </visual>
   </link>
-  <gazebo reference="servo_link">
-    <mu1>0.1</mu1>
-    <mu2>0.1</mu2>
-  </gazebo>
-  <xacro:damping_factor link="servo_link"/>
-  <link name="servo_link1">
+  <link name="servo_link2">
     <inertial>
       <origin xyz="0 0 0" rpy="0 0 0"/>
@@ -231,9 +240,24 @@
     </visual>
   </link>
-  <gazebo reference="servo_link1">
-    <mu1>0.1</mu1>
-    <mu2>0.1</mu2>
-  </gazebo>
-  <xacro:damping_factor link="servo_link1"/>
+  <link name="dummy_link1">
+    <inertial>
+      <origin xyz="0 0 0" rpy="0 0 0"/>
+      <mass value="0.0001"/>
+      <inertia
+          ixx="0.00001" ixy="0.0" ixz="0.0"
+          iyy="0.00001" iyz="0.0"
+          izz="0.00002"/>
+    </inertial>
+  </link>
+  <link name="dummy_link2">
+    <inertial>
+      <origin xyz="0 0 0" rpy="0 0 0"/>
+      <mass value="0.0001"/>
+      <inertia
+          ixx="0.00001" ixy="0.0" ixz="0.0"
+          iyy="0.00001" iyz="0.0"
+          izz="0.00002"/>
+    </inertial>
+  </link>
   <transmission name="soft_joint_tran_4">
     <type>transmission_interface/SimpleTransmission</type>
@@ -252,4 +276,24 @@
     </joint>
     <actuator name="soft_joint_servo5">
+      <hardwareInterface>hardware_interface/EffortJointInterface</hardwareInterface>
+      <mechanicalReduction>1</mechanicalReduction>
+    </actuator>
+  </transmission>
+  <transmission name="soft_joint_tran_6">
+    <type>transmission_interface/SimpleTransmission</type>
+    <joint name="soft_joint6">
+      <hardwareInterface>hardware_interface/EffortJointInterface</hardwareInterface>
+    </joint>
+    <actuator name="soft_joint_servo6">
+      <hardwareInterface>hardware_interface/EffortJointInterface</hardwareInterface>
+      <mechanicalReduction>1</mechanicalReduction>
+    </actuator>
+  </transmission>
+  <transmission name="soft_joint_tran_7">
+    <type>transmission_interface/SimpleTransmission</type>
+    <joint name="soft_joint7">
+      <hardwareInterface>hardware_interface/EffortJointInterface</hardwareInterface>
+    </joint>
+    <actuator name="soft_joint_servo7">
       <hardwareInterface>hardware_interface/EffortJointInterface</hardwareInterface>
       <mechanicalReduction>1</mechanicalReduction>

Commit message: seperate Servo.yaml and Servo_sim.yaml and succeeded

File: robots/delta/robots/quad/20240722/delta.urdf.xacro (robot description, xacro)
@@ -260,44 +260,44 @@
     </inertial>
   </link>
-  <transmission name="soft_joint_tran_4">
-    <type>transmission_interface/SimpleTransmission</type>
-    <joint name="soft_joint4">
-      <hardwareInterface>hardware_interface/EffortJointInterface</hardwareInterface>
-    </joint>
-    <actuator name="soft_joint_servo4">
-      <hardwareInterface>hardware_interface/EffortJointInterface</hardwareInterface>
-      <mechanicalReduction>1</mechanicalReduction>
-    </actuator>
-  </transmission>
-  <transmission name="soft_joint_tran_5">
-    <type>transmission_interface/SimpleTransmission</type>
-    <joint name="soft_joint5">
-      <hardwareInterface>hardware_interface/EffortJointInterface</hardwareInterface>
-    </joint>
-    <actuator name="soft_joint_servo5">
-      <hardwareInterface>hardware_interface/EffortJointInterface</hardwareInterface>
-      <mechanicalReduction>1</mechanicalReduction>
-    </actuator>
-  </transmission>
-  <transmission name="soft_joint_tran_6">
-    <type>transmission_interface/SimpleTransmission</type>
-    <joint name="soft_joint6">
-      <hardwareInterface>hardware_interface/EffortJointInterface</hardwareInterface>
-    </joint>
-    <actuator name="soft_joint_servo6">
-      <hardwareInterface>hardware_interface/EffortJointInterface</hardwareInterface>
-      <mechanicalReduction>1</mechanicalReduction>
-    </actuator>
-  </transmission>
-  <transmission name="soft_joint_tran_7">
-    <type>transmission_interface/SimpleTransmission</type>
-    <joint name="soft_joint7">
-      <hardwareInterface>hardware_interface/EffortJointInterface</hardwareInterface>
-    </joint>
-    <actuator name="soft_joint_servo7">
-      <hardwareInterface>hardware_interface/EffortJointInterface</hardwareInterface>
-      <mechanicalReduction>1</mechanicalReduction>
-    </actuator>
-  </transmission>
+  <!-- <transmission name="soft_joint_tran_4"> -->
+  <!--   <type>transmission_interface/SimpleTransmission</type> -->
+  <!--   <joint name="soft_joint4"> -->
+  <!--     <hardwareInterface>hardware_interface/EffortJointInterface</hardwareInterface> -->
+  <!--   </joint> -->
+  <!--   <actuator name="soft_joint_servo4"> -->
+  <!--     <hardwareInterface>hardware_interface/EffortJointInterface</hardwareInterface> -->
+  <!--     <mechanicalReduction>1</mechanicalReduction> -->
+  <!--   </actuator> -->
+  <!-- </transmission> -->
+  <!-- <transmission name="soft_joint_tran_5"> -->
+  <!--   <type>transmission_interface/SimpleTransmission</type> -->
+  <!--   <joint name="soft_joint5"> -->
+  <!--     <hardwareInterface>hardware_interface/EffortJointInterface</hardwareInterface> -->
+  <!--   </joint> -->
+  <!--   <actuator name="soft_joint_servo5"> -->
+  <!--     <hardwareInterface>hardware_interface/EffortJointInterface</hardwareInterface> -->
+  <!--     <mechanicalReduction>1</mechanicalReduction> -->
+  <!--   </actuator> -->
+  <!-- </transmission> -->
+  <!-- <transmission name="soft_joint_tran_6"> -->
+  <!--   <type>transmission_interface/SimpleTransmission</type> -->
+  <!--   <joint name="soft_joint6"> -->
+  <!--     <hardwareInterface>hardware_interface/EffortJointInterface</hardwareInterface> -->
+  <!--   </joint> -->
+  <!--   <actuator name="soft_joint_servo6"> -->
+  <!--     <hardwareInterface>hardware_interface/EffortJointInterface</hardwareInterface> -->
+  <!--     <mechanicalReduction>1</mechanicalReduction> -->
+  <!--   </actuator> -->
+  <!-- </transmission> -->
+  <!-- <transmission name="soft_joint_tran_7"> -->
+  <!--   <type>transmission_interface/SimpleTransmission</type> -->
+  <!--   <joint name="soft_joint7"> -->
+  <!--     <hardwareInterface>hardware_interface/EffortJointInterface</hardwareInterface> -->
+  <!--   </joint> -->
+  <!--   <actuator name="soft_joint_servo7"> -->
+  <!--     <hardwareInterface>hardware_interface/EffortJointInterface</hardwareInterface> -->
+  <!--     <mechanicalReduction>1</mechanicalReduction> -->
+  <!--   </actuator> -->
+  <!-- </transmission> -->
   <!-- leg -->
   <link name="leg6">

Commit message: add soft_link3 and rotor6 and tested in simulator

File: robots/delta/robots/quad/20240722/delta.urdf.xacro (robot description, xacro)
@@ -495,6 +495,78 @@
     </visual>
   </link>
+  <!-- gimbal -->
+  <joint name="gimbal_joint6" type="fixed">
+    <limit effort="5.0" lower="${-pi}" upper="${pi}" velocity="0.5"/>
+    <parent link="soft_link6"/>
+    <child link="gimbal_link6"/>
+    <origin rpy="0 0 0" xyz="0.128 0 0"/>
+    <axis xyz="1 0 0"/>
+    <dynamics damping="0.9" friction="0.1"/>
+  </joint>
+  <link name="gimbal_link6">
+    <inertial>
+      <origin xyz="0.0815 0 0" rpy="0 0 0"/>
+      <mass value="${0.222}"/>
+      <!-- this inertia value is 10 times bigger than the real one -->
+      <!-- to avoid the instability in gazebo -->
+      <!-- <inertia
+          ixx="0.0022661" ixy="0.0" ixz="0.0"
+          iyy="0.0015451" iyz="0.0"
+          izz="0.00032533"/> -->
+      <!-- original one -->
+      <inertia
+          ixx="0.00022661" ixy="0.0" ixz="0.0"
+          iyy="0.00015451" iyz="0.0"
+          izz="0.000032533"/>
+    </inertial>
+    <visual>
+      <origin xyz="0.0815 0 0" rpy="0 0 0"/>
+      <geometry>
+        <mesh filename="package://delta/urdf/mesh/20240722/5inch_propeller_duct_right_v2.dae"/>
+      </geometry>
+    </visual>
+  </link>
+  <gazebo reference="gimbal_link6">
+    <mu1>0.1</mu1>
+    <mu2>0.1</mu2>
+  </gazebo>
+  <xacro:damping_factor link ="gimbal_link6"/>
+  <!-- rotor -->
+  <joint name="rotor6" type="continuous">
+    <limit effort="0.0064" lower="0.0" upper="20.0" velocity="0.5"/>
+    <parent link="gimbal_link6"/>
+    <child link="thrust6"/>
+    <origin rpy="0 0 0" xyz="0.0735 0 0"/>
+    <axis xyz="0 0 -1"/>
+  </joint>
+  <link name="thrust6">
+    <inertial>
+      <origin xyz="0 0 0" rpy="0 0 0"/>
+      <mass value="0.0001"/>
+      <inertia
+          ixx="0.00001" ixy="0.0" ixz="0.0"
+          iyy="0.00001" iyz="0.0"
+          izz="0.00002"/>
+    </inertial>
+    <visual>
+      <origin rpy="${pi/2} 0 0" xyz="-0.045 0.055 0.06"/>
+      <geometry>
+        <mesh filename="package://delta/urdf/mesh/20240722/TriBlade_5045.dae"/>
+      </geometry>
+    </visual>
+  </link>
+  <xacro:damping_factor link ="thrust6"/>
+  <transmission name="rotor_tran6">
+    <type>transmission_interface/SimpleTransmission</type>
+    <joint name="rotor6">
+      <hardwareInterface>RotorInterface</hardwareInterface>
+    </joint>
+    <actuator name="rotor6">
+      <hardwareInterface>RotorInterface</hardwareInterface>
+      <mechanicalReduction>1</mechanicalReduction>
+    </actuator>
+  </transmission>
   <!-- leg -->
-  <!-- <link name="leg7">
+  <link name="leg7">
     <inertial>
       <origin xyz="0.0 0.0 -0.093" rpy="0 0 0"/>
@@ -510,4 +582,10 @@
       <origin xyz="0.01 0.01 -0.075" rpy="0 0 0"/>
     </visual>
+    <collision>
+      <geometry>
+        <box size="0.02 0.02 -0.15"/>
+      </geometry>
+      <origin xyz="0.01 0.01 -0.075" rpy="0 0 0"/>
+    </collision>
   </link>
   <gazebo reference="leg7">
@@ -520,4 +598,169 @@
     <child link="leg7"/>
     <origin xyz="0.1 0 0" rpy="0 0 0"/>
-  </joint> -->
+  </joint>
+  <!-- 3 soft_airframe_3 -->
+  <!-- soft_link -->
+  <joint name="soft_joint7" type="fixed">
+    <parent link="gimbal_link6"/>
+    <child link="soft_link7"/>
+    <origin xyz="0.147 0 0" rpy="0 0 0"/>
+  </joint>
+  <joint name="soft_joint8" type="revolute">
+    <limit effort="5.0" lower="${-pi}" upper="${pi}" velocity="0.5"/>
+    <parent link="soft_link7"/>
+    <child link="soft_link8"/>
+    <origin xyz="0.1175 0 0" rpy="0 0 0"/>
+    <axis xyz="0 0 1"/>
+    <dynamics damping="0.2" friction="0.1"/>
+  </joint>
+  <joint name="soft_joint9" type="revolute">
+    <limit effort="5.0" lower="${-pi}" upper="${pi}" velocity="0.5"/>
+    <parent link="soft_link8"/>
+    <child link="soft_link9"/>
+    <origin xyz="0.235 0 0" rpy="0 0 0"/>
+    <axis xyz="0 0 1"/>
+    <dynamics damping="0.2" friction="0.1"/>
+  </joint>
+  <link name="soft_link7">
+    <inertial>
+      <origin xyz="0.101 0.000002 0.018960" rpy="0 0 0"/>
+      <mass value="0.059"/>
+      <inertia
+          ixx="0.00005433" ixy="0.00000033" ixz="0.0"
+          iyy="0.00047358" iyz="-0.00000369"
+          izz="0.00046011"/>
+    </inertial>
+    <visual>
+      <geometry>
+        <box size="0.1175 0.03 0.04"/>
+      </geometry>
+      <origin xyz="0.05875 0 0.02" rpy="0 0 0"/>
+    </visual>
+  </link>
+  <gazebo reference="soft_link7">
+    <mu1>0.1</mu1>
+    <mu2>0.1</mu2>
+  </gazebo>
+  <xacro:damping_factor link="soft_link7"/>
+  <link name="soft_link8">
+    <inertial>
+      <origin xyz="0.118 0.000002 0.019998" rpy="0 0 0"/>
+      <mass value="0.118"/>
+      <inertia
+          ixx="0.00007941" ixy="0.00000218" ixz="0.0"
+          iyy="0.00065133" iyz="0.0"
+          izz="0.00062639"/>
+    </inertial>
+    <visual>
+      <geometry>
+        <box size="0.235 0.03 0.04"/>
+      </geometry>
+      <origin xyz="0.1175 0.000002 0.019998" rpy="0 0 0"/>
+    </visual>
+  </link>
+  <gazebo reference="soft_link8">
+    <mu1>0.1</mu1>
+    <mu2>0.1</mu2>
+  </gazebo>
+  <xacro:damping_factor link="soft_link8"/>
+  <link name="soft_link9">
+    <inertial>
+      <origin xyz="0.10740316 0.0 0.003" rpy="0 0 0"/>
+      <mass value="0.059"/>
+      <inertia
+          ixx="0.00005433" ixy="0.00000033" ixz="0.0"
+          iyy="0.00047358" iyz="-0.00000369"
+          izz="0.00046011"/>
+    </inertial>
+    <visual>
+      <geometry>
+        <box size="${0.1175 + 0.054} 0.03 0.04"/>
+      </geometry>
+      <origin xyz="0.05875 0 0.02" rpy="0 0 0"/>
+    </visual>
+  </link>
+  <gazebo reference="soft_link9">
+    <mu1>0.1</mu1>
+    <mu2>0.1</mu2>
+  </gazebo>
+  <xacro:damping_factor link="soft_link9"/>
+  <transmission name="soft_joint_tran_8">
+    <type>transmission_interface/SimpleTransmission</type>
+    <joint name="soft_joint8">
+      <hardwareInterface>hardware_interface/EffortJointInterface</hardwareInterface>
+    </joint>
+    <actuator name="soft_joint_servo8">
+      <hardwareInterface>hardware_interface/EffortJointInterface</hardwareInterface>
+      <mechanicalReduction>1</mechanicalReduction>
+    </actuator>
+  </transmission>
+  <transmission name="soft_joint_tran_9">
+    <type>transmission_interface/SimpleTransmission</type>
+    <joint name="soft_joint9">
+      <hardwareInterface>hardware_interface/EffortJointInterface</hardwareInterface>
+    </joint>
+    <actuator name="soft_joint_servo9">
+      <hardwareInterface>hardware_interface/EffortJointInterface</hardwareInterface>
+      <mechanicalReduction>1</mechanicalReduction>
+    </actuator>
+  </transmission>
+  <!-- dummy_link -->
+  <joint name="servo_joint5" type="fixed">
+    <limit effort="5.0" lower="${-pi/2}" upper="${pi/2}" velocity="0.5"/>
+    <parent link="soft_link9"/>
+    <child link="servo_link5"/>
+    <origin xyz="0.1 0 0.01" rpy="0 0 0"/>
+    <axis xyz="0 0 1"/>
+    <dynamics damping="0.9" friction="0.1"/>
+  </joint>
+  <joint name="servo_joint6" type="fixed">
+    <limit effort="5.0" lower="${-pi/2}" upper="${pi/2}" velocity="0.5"/>
+    <parent link="soft_link6"/>
+    <child link="servo_link6"/>
+    <origin xyz="0.1 0 -0.01" rpy="0 0 0"/>
+    <axis xyz="0 0 1"/>
+    <dynamics damping="0.9" friction="0.1"/>
+  </joint>
+  <link name="servo_link5">
+    <inertial>
+      <origin xyz="0 0 0" rpy="0 0 0"/>
+      <mass value="0.073"/>
+      <!-- this is for avoiding error in gazebo -->
+      <!-- <inertia
+          ixx="0.001" ixy="0.0" ixz="0.0"
+          iyy="0.001" iyz="0.0"
+          izz="0.002"/> -->
+      <inertia
+          ixx="0.000023" ixy="0.000003" ixz="-0.0000001"
+          iyy="0.000044" iyz="0.000000"
+          izz="0.000043"/>
+    </inertial>
+    <visual>
+      <geometry>
+        <box size="0.05 0.05 0.05"/>
+      </geometry>
+      <origin xyz="0 0 -0.02" rpy="0 0 0"/>
+    </visual>
+  </link>
+  <link name="servo_link6">
+    <inertial>
+      <origin xyz="0 0 0" rpy="0 0 0"/>
+      <mass value="0.068"/>
+      <!-- this is for avoiding error in gazebo -->
+      <!-- <inertia
+          ixx="0.001" ixy="0.0" ixz="0.0"
+          iyy="0.001" iyz="0.0"
+          izz="0.002"/> -->
+      <inertia
+          ixx="0.000022" ixy="-0.000003" ixz="0.000001"
+          iyy="0.000042" iyz="0.000000"
+          izz="0.000041"/>
+    </inertial>
+    <visual>
+      <geometry>
+        <box size="0.05 0.05 0.05"/>
+      </geometry>
+      <origin xyz="0 0 -0.02" rpy="0 0 0"/>
+    </visual>
+  </link>
 </robot>

Commit message: delete unnecessary urdfs

File: robots/delta/robots/quad/20240722/delta.urdf.xacro (robot description, xacro)
@@ -188,9 +188,4 @@
       <origin xyz="0 0 0" rpy="0 0 0"/>
       <mass value="0.073"/>
-      <!-- this is for avoiding error in gazebo -->
-      <!-- <inertia
-          ixx="0.001" ixy="0.0" ixz="0.0"
-          iyy="0.001" iyz="0.0"
-          izz="0.002"/> -->
       <inertia
           ixx="0.000023" ixy="0.000003" ixz="-0.0000001"
@@ -209,9 +204,4 @@
       <origin xyz="0 0 0" rpy="0 0 0"/>
       <mass value="0.068"/>
-      <!-- this is for avoiding error in gazebo -->
-      <!-- <inertia
-          ixx="0.001" ixy="0.0" ixz="0.0"
-          iyy="0.001" iyz="0.0"
-          izz="0.002"/> -->
       <inertia
           ixx="0.000022" ixy="-0.000003" ixz="0.000001"
@@ -271,11 +261,4 @@
       <origin xyz="0.0815 0 0" rpy="0 0 0"/>
       <mass value="${0.222}"/>
-      <!-- this inertia value is 10 times bigger than the real one -->
-      <!-- to avoid the instability in gazebo -->
-      <!-- <inertia
-          ixx="0.0022661" ixy="0.0" ixz="0.0"
-          iyy="0.0015451" iyz="0.0"
-          izz="0.00032533"/> -->
-      <!-- original one -->
       <inertia
           ixx="0.00022661" ixy="0.0" ixz="0.0"
@@ -457,9 +440,4 @@
       <origin xyz="0 0 0" rpy="0 0 0"/>
       <mass value="0.073"/>
-      <!-- this is for avoiding error in gazebo -->
-      <!-- <inertia
-          ixx="0.001" ixy="0.0" ixz="0.0"
-          iyy="0.001" iyz="0.0"
-          izz="0.002"/> -->
       <inertia
           ixx="0.000023" ixy="0.000003" ixz="-0.0000001"
@@ -478,9 +456,4 @@
       <origin xyz="0 0 0" rpy="0 0 0"/>
       <mass value="0.068"/>
-      <!-- this is for avoiding error in gazebo -->
-      <!-- <inertia
-          ixx="0.001" ixy="0.0" ixz="0.0"
-          iyy="0.001" iyz="0.0"
-          izz="0.002"/> -->
       <inertia
           ixx="0.000022" ixy="-0.000003" ixz="0.000001"
@@ -508,11 +481,4 @@
       <origin xyz="0.0815 0 0" rpy="0 0 0"/>
       <mass value="${0.222}"/>
-      <!-- this inertia value is 10 times bigger than the real one -->
-      <!-- to avoid the instability in gazebo -->
-      <!-- <inertia
-          ixx="0.0022661" ixy="0.0" ixz="0.0"
-          iyy="0.0015451" iyz="0.0"
-          izz="0.00032533"/> -->
-      <!-- original one -->
       <inertia
           ixx="0.00022661" ixy="0.0" ixz="0.0"
@@ -726,9 +692,4 @@
       <origin xyz="0 0 0" rpy="0 0 0"/>
       <mass value="0.073"/>
-      <!-- this is for avoiding error in gazebo -->
-      <!-- <inertia
-          ixx="0.001" ixy="0.0" ixz="0.0"
-          iyy="0.001" iyz="0.0"
-          izz="0.002"/> -->
       <inertia
           ixx="0.000023" ixy="0.000003" ixz="-0.0000001"
@@ -747,9 +708,4 @@
       <origin xyz="0 0 0" rpy="0 0 0"/>
       <mass value="0.068"/>
-      <!-- this is for avoiding error in gazebo -->
-      <!-- <inertia
-          ixx="0.001" ixy="0.0" ixz="0.0"
-          iyy="0.001" iyz="0.0"
-          izz="0.002"/> -->
       <inertia
           ixx="0.000022" ixy="-0.000003" ixz="0.000001"

Commit message: update urdf

File: robots/delta/robots/quad/20240722/delta.urdf.xacro (robot description, xacro)
@@ -95,7 +95,8 @@
     <visual>
       <geometry>
-        <box size="0.1175 0.03 0.04"/>
-      </geometry>
-      <origin xyz="0.05875 0 0.02" rpy="0 0 0"/>
+        <!-- <box size="0.1175 0.03 0.04"/> -->
+        <box size="0.15 0.03 0.04"/>
+      </geometry>
+      <origin xyz="0.02875 0 0.02" rpy="0 0 0"/>
     </visual>
   </link>
@@ -198,10 +199,10 @@
           izz="0.000043"/>
     </inertial>
-    <visual>
+    <!-- <visual>
       <geometry>
         <box size="0.05 0.05 0.05"/>
       </geometry>
       <origin xyz="0 0 -0.02" rpy="0 0 0"/>
-    </visual>
+    </visual> -->
   </link>
   <link name="servo_link2">
@@ -219,10 +220,10 @@
           izz="0.000041"/>
     </inertial>
-    <visual>
+    <!-- <visual>
       <geometry>
         <box size="0.05 0.05 0.05"/>
       </geometry>
       <origin xyz="0 0 -0.02" rpy="0 0 0"/>
-    </visual>
+    </visual> -->
   </link>
   <!-- leg -->
@@ -236,8 +237,8 @@
     </inertial>
     <visual>
-      <geometry>
-        <box size="0.02 0.02 -0.15"/>
-      </geometry>
-      <origin xyz="0.01 0.01 -0.075" rpy="0 0 0"/>
+      <origin rpy="0 0 ${pi/2}" xyz="0 -0.05 -0.15"/>
+      <geometry>
+        <mesh filename="package://delta/urdf/mesh/20240722/leg_joint_soft.dae"/>
+      </geometry>
     </visual>
     <collision>
@@ -406,7 +407,7 @@
     <visual>
       <geometry>
-        <box size="${0.1175 + 0.054} 0.03 0.04"/>
-      </geometry>
-      <origin xyz="0.05875 0 0.02" rpy="0 0 0"/>
+        <box size="${0.1175 + 0.054 + 0.03} 0.03 0.04"/>
+      </geometry>
+      <origin xyz="0.08875 0 0.02" rpy="0 0 0"/>
     </visual>
   </link>
@@ -467,10 +468,10 @@
           izz="0.000043"/>
     </inertial>
-    <visual>
+    <!-- <visual>
       <geometry>
         <box size="0.05 0.05 0.05"/>
       </geometry>
       <origin xyz="0 0 -0.02" rpy="0 0 0"/>
-    </visual>
+    </visual> -->
   </link>
   <link name="servo_link4">
@@ -488,10 +489,10 @@
           izz="0.000041"/>
     </inertial>
-    <visual>
+    <!-- <visual>
       <geometry>
         <box size="0.05 0.05 0.05"/>
       </geometry>
       <origin xyz="0 0 -0.02" rpy="0 0 0"/>
-    </visual>
+    </visual> -->
   </link>
   <!-- leg -->
