Commit message: update for 3 rigid links and 3 soft links

File: robots/delta/robots/quad/20240722/delta.urdf.xacro (robot description, xacro)
@@ -6,6 +6,6 @@
   <xacro:delta_module self="1" child="2" rotor_direction="1" rotor_tilt="0" battery="0"/>
   <xacro:delta_module self="2" child="3" rotor_direction="-1" rotor_tilt="0" battery="0"/>
-  <xacro:delta_module self="3" child="4" rotor_direction="1" rotor_tilt="0"  battery="0"/>
-  <xacro:delta_module self="4" child="4" rotor_direction="-1" rotor_tilt="0" battery="0"/>
+  <xacro:delta_module self="3" child="3" rotor_direction="1" rotor_tilt="0"  battery="0"/>
+  <!-- <xacro:delta_module self="4" child="4" rotor_direction="-1" rotor_tilt="0" battery="0"/> -->
   <!-- dummy root link for KDL -->
   <link name="root">
@@ -64,5 +64,5 @@
   <!-- soft_link -->
   <joint name="soft_joint1" type="fixed">
-    <parent link="link4"/>
+    <parent link="link3"/>
     <child link="soft_link1"/>
     <origin xyz="0.6 0 0" rpy="0 0 0"/>
@@ -170,5 +170,5 @@
   <joint name="servo_joint1" type="fixed">
     <limit effort="5.0" lower="${-pi/2}" upper="${pi/2}" velocity="0.5"/>
-    <parent link="link4"/>
+    <parent link="link3"/>
     <child link="servo_link1"/>
     <origin xyz="0.5 0 0.01" rpy="0 0 0"/>
@@ -178,5 +178,5 @@
   <joint name="servo_joint2" type="fixed">
     <limit effort="5.0" lower="${-pi/2}" upper="${pi/2}" velocity="0.5"/>
-    <parent link="link4"/>
+    <parent link="link3"/>
     <child link="servo_link2"/>
     <origin xyz="0.5 0 -0.01" rpy="0 0 0"/>
@@ -279,7 +279,227 @@
   <xacro:damping_factor link ="gimbal_link5"/>
   <!-- rotor -->
+  <joint name="rotor4" type="continuous">
+    <limit effort="0.0064" lower="0.0" upper="20.0" velocity="0.5"/>
+    <parent link="gimbal_link5"/>
+    <child link="thrust4"/>
+    <origin rpy="0 0 0" xyz="0.0735 0 0"/>
+    <axis xyz="0 0 -1"/>
+  </joint>
+  <link name="thrust4">
+    <inertial>
+      <origin xyz="0 0 0" rpy="0 0 0"/>
+      <mass value="0.0001"/>
+      <inertia
+          ixx="0.00001" ixy="0.0" ixz="0.0"
+          iyy="0.00001" iyz="0.0"
+          izz="0.00002"/>
+    </inertial>
+    <visual>
+      <origin rpy="${pi/2} 0 0" xyz="-0.045 0.055 0.06"/>
+      <geometry>
+        <mesh filename="package://delta/urdf/mesh/20240722/TriBlade_5045.dae"/>
+      </geometry>
+    </visual>
+  </link>
+  <xacro:damping_factor link ="thrust4"/>
+  <transmission name="rotor_tran4">
+    <type>transmission_interface/SimpleTransmission</type>
+    <joint name="rotor4">
+      <hardwareInterface>RotorInterface</hardwareInterface>
+    </joint>
+    <actuator name="rotor4">
+      <hardwareInterface>RotorInterface</hardwareInterface>
+      <mechanicalReduction>1</mechanicalReduction>
+    </actuator>
+  </transmission>
+  <!-- 3 soft_airframe_2 -->
+  <!-- soft_link -->
+  <joint name="soft_joint4" type="fixed">
+    <parent link="gimbal_link5"/>
+    <child link="soft_link4"/>
+    <origin xyz="0.147 0 0" rpy="0 0 0"/>
+  </joint>
+  <joint name="soft_joint5" type="revolute">
+    <limit effort="5.0" lower="${-pi}" upper="${pi}" velocity="0.5"/>
+    <parent link="soft_link4"/>
+    <child link="soft_link5"/>
+    <origin xyz="0.1175 0 0" rpy="0 0 0"/>
+    <axis xyz="0 0 1"/>
+    <dynamics damping="0.2" friction="0.1"/>
+  </joint>
+  <joint name="soft_joint6" type="revolute">
+    <limit effort="5.0" lower="${-pi}" upper="${pi}" velocity="0.5"/>
+    <parent link="soft_link5"/>
+    <child link="soft_link6"/>
+    <origin xyz="0.235 0 0" rpy="0 0 0"/>
+    <axis xyz="0 0 1"/>
+    <dynamics damping="0.2" friction="0.1"/>
+  </joint>
+  <link name="soft_link4">
+    <inertial>
+      <origin xyz="0.101 0.000002 0.018960" rpy="0 0 0"/>
+      <mass value="0.059"/>
+      <inertia
+          ixx="0.00005433" ixy="0.00000033" ixz="0.0"
+          iyy="0.00047358" iyz="-0.00000369"
+          izz="0.00046011"/>
+    </inertial>
+    <visual>
+      <geometry>
+        <box size="0.1175 0.03 0.04"/>
+      </geometry>
+      <origin xyz="0.05875 0 0.02" rpy="0 0 0"/>
+    </visual>
+  </link>
+  <gazebo reference="soft_link4">
+    <mu1>0.1</mu1>
+    <mu2>0.1</mu2>
+  </gazebo>
+  <xacro:damping_factor link="soft_link4"/>
+  <link name="soft_link5">
+    <inertial>
+      <origin xyz="0.118 0.000002 0.019998" rpy="0 0 0"/>
+      <mass value="0.118"/>
+      <inertia
+          ixx="0.00007941" ixy="0.00000218" ixz="0.0"
+          iyy="0.00065133" iyz="0.0"
+          izz="0.00062639"/>
+    </inertial>
+    <visual>
+      <geometry>
+        <box size="0.235 0.03 0.04"/>
+      </geometry>
+      <origin xyz="0.1175 0.000002 0.019998" rpy="0 0 0"/>
+    </visual>
+  </link>
+  <gazebo reference="soft_link5">
+    <mu1>0.1</mu1>
+    <mu2>0.1</mu2>
+  </gazebo>
+  <xacro:damping_factor link="soft_link5"/>
+  <link name="soft_link6">
+    <inertial>
+      <origin xyz="0.10740316 0.0 0.003" rpy="0 0 0"/>
+      <mass value="0.059"/>
+      <inertia
+          ixx="0.00005433" ixy="0.00000033" ixz="0.0"
+          iyy="0.00047358" iyz="-0.00000369"
+          izz="0.00046011"/>
+    </inertial>
+    <visual>
+      <geometry>
+        <box size="${0.1175 + 0.054} 0.03 0.04"/>
+      </geometry>
+      <origin xyz="0.05875 0 0.02" rpy="0 0 0"/>
+    </visual>
+  </link>
+  <gazebo reference="soft_link6">
+    <mu1>0.1</mu1>
+    <mu2>0.1</mu2>
+  </gazebo>
+  <xacro:damping_factor link="soft_link6"/>
+  <transmission name="soft_joint_tran_5">
+    <type>transmission_interface/SimpleTransmission</type>
+    <joint name="soft_joint5">
+      <hardwareInterface>hardware_interface/EffortJointInterface</hardwareInterface>
+    </joint>
+    <actuator name="soft_joint_servo5">
+      <hardwareInterface>hardware_interface/EffortJointInterface</hardwareInterface>
+      <mechanicalReduction>1</mechanicalReduction>
+    </actuator>
+  </transmission>
+  <transmission name="soft_joint_tran_6">
+    <type>transmission_interface/SimpleTransmission</type>
+    <joint name="soft_joint6">
+      <hardwareInterface>hardware_interface/EffortJointInterface</hardwareInterface>
+    </joint>
+    <actuator name="soft_joint_servo6">
+      <hardwareInterface>hardware_interface/EffortJointInterface</hardwareInterface>
+      <mechanicalReduction>1</mechanicalReduction>
+    </actuator>
+  </transmission>
+  <!-- dummy_link -->
+  <joint name="servo_joint3" type="fixed">
+    <limit effort="5.0" lower="${-pi/2}" upper="${pi/2}" velocity="0.5"/>
+    <parent link="soft_link6"/>
+    <child link="servo_link3"/>
+    <origin xyz="0.1 0 0.01" rpy="0 0 0"/>
+    <axis xyz="0 0 1"/>
+    <dynamics damping="0.9" friction="0.1"/>
+  </joint>
+  <joint name="servo_joint4" type="fixed">
+    <limit effort="5.0" lower="${-pi/2}" upper="${pi/2}" velocity="0.5"/>
+    <parent link="soft_link6"/>
+    <child link="servo_link4"/>
+    <origin xyz="0.1 0 -0.01" rpy="0 0 0"/>
+    <axis xyz="0 0 1"/>
+    <dynamics damping="0.9" friction="0.1"/>
+  </joint>
+  <link name="servo_link3">
+    <inertial>
+      <origin xyz="0 0 0" rpy="0 0 0"/>
+      <mass value="0.073"/>
+      <inertia
+          ixx="0.000023" ixy="0.000003" ixz="-0.0000001"
+          iyy="0.000044" iyz="0.000000"
+          izz="0.000043"/>
+    </inertial>
+    <visual>
+      <geometry>
+        <box size="0.05 0.05 0.05"/>
+      </geometry>
+      <origin xyz="0 0 -0.02" rpy="0 0 0"/>
+    </visual>
+  </link>
+  <link name="servo_link4">
+    <inertial>
+      <origin xyz="0 0 0" rpy="0 0 0"/>
+      <mass value="0.068"/>
+      <inertia
+          ixx="0.000022" ixy="-0.000003" ixz="0.000001"
+          iyy="0.000042" iyz="0.000000"
+          izz="0.000041"/>
+    </inertial>
+    <visual>
+      <geometry>
+        <box size="0.05 0.05 0.05"/>
+      </geometry>
+      <origin xyz="0 0 -0.02" rpy="0 0 0"/>
+    </visual>
+  </link>
+  <!-- gimbal -->
+  <joint name="gimbal_joint6" type="fixed">
+    <limit effort="5.0" lower="${-pi}" upper="${pi}" velocity="0.5"/>
+    <parent link="soft_link6"/>
+    <child link="gimbal_link6"/>
+    <origin rpy="0 0 0" xyz="0.128 0 0"/>
+    <axis xyz="1 0 0"/>
+    <dynamics damping="0.9" friction="0.1"/>
+  </joint>
+  <link name="gimbal_link6">
+    <inertial>
+      <origin xyz="0.0815 0 0" rpy="0 0 0"/>
+      <mass value="${0.222}"/>
+      <inertia
+          ixx="0.00022661" ixy="0.0" ixz="0.0"
+          iyy="0.00015451" iyz="0.0"
+          izz="0.000032533"/>
+    </inertial>
+    <visual>
+      <origin xyz="0.0815 0 0" rpy="0 0 0"/>
+      <geometry>
+        <mesh filename="package://delta/urdf/mesh/20240722/5inch_propeller_duct_right_v2.dae"/>
+      </geometry>
+    </visual>
+  </link>
+  <gazebo reference="gimbal_link6">
+    <mu1>0.1</mu1>
+    <mu2>0.1</mu2>
+  </gazebo>
+  <xacro:damping_factor link ="gimbal_link6"/>
+  <!-- rotor -->
   <joint name="rotor5" type="continuous">
     <limit effort="0.0064" lower="0.0" upper="20.0" velocity="0.5"/>
-    <parent link="gimbal_link5"/>
+    <parent link="gimbal_link6"/>
     <child link="thrust5"/>
     <origin rpy="0 0 0" xyz="0.0735 0 0"/>
@@ -313,224 +533,4 @@
     </actuator>
   </transmission>
-  <!-- 3 soft_airframe_2 -->
-  <!-- soft_link -->
-  <joint name="soft_joint4" type="fixed">
-    <parent link="gimbal_link5"/>
-    <child link="soft_link4"/>
-    <origin xyz="0.147 0 0" rpy="0 0 0"/>
-  </joint>
-  <joint name="soft_joint5" type="revolute">
-    <limit effort="5.0" lower="${-pi}" upper="${pi}" velocity="0.5"/>
-    <parent link="soft_link4"/>
-    <child link="soft_link5"/>
-    <origin xyz="0.1175 0 0" rpy="0 0 0"/>
-    <axis xyz="0 0 1"/>
-    <dynamics damping="0.2" friction="0.1"/>
-  </joint>
-  <joint name="soft_joint6" type="revolute">
-    <limit effort="5.0" lower="${-pi}" upper="${pi}" velocity="0.5"/>
-    <parent link="soft_link5"/>
-    <child link="soft_link6"/>
-    <origin xyz="0.235 0 0" rpy="0 0 0"/>
-    <axis xyz="0 0 1"/>
-    <dynamics damping="0.2" friction="0.1"/>
-  </joint>
-  <link name="soft_link4">
-    <inertial>
-      <origin xyz="0.101 0.000002 0.018960" rpy="0 0 0"/>
-      <mass value="0.059"/>
-      <inertia
-          ixx="0.00005433" ixy="0.00000033" ixz="0.0"
-          iyy="0.00047358" iyz="-0.00000369"
-          izz="0.00046011"/>
-    </inertial>
-    <visual>
-      <geometry>
-        <box size="0.1175 0.03 0.04"/>
-      </geometry>
-      <origin xyz="0.05875 0 0.02" rpy="0 0 0"/>
-    </visual>
-  </link>
-  <gazebo reference="soft_link4">
-    <mu1>0.1</mu1>
-    <mu2>0.1</mu2>
-  </gazebo>
-  <xacro:damping_factor link="soft_link4"/>
-  <link name="soft_link5">
-    <inertial>
-      <origin xyz="0.118 0.000002 0.019998" rpy="0 0 0"/>
-      <mass value="0.118"/>
-      <inertia
-          ixx="0.00007941" ixy="0.00000218" ixz="0.0"
-          iyy="0.00065133" iyz="0.0"
-          izz="0.00062639"/>
-    </inertial>
-    <visual>
-      <geometry>
-        <box size="0.235 0.03 0.04"/>
-      </geometry>
-      <origin xyz="0.1175 0.000002 0.019998" rpy="0 0 0"/>
-    </visual>
-  </link>
-  <gazebo reference="soft_link5">
-    <mu1>0.1</mu1>
-    <mu2>0.1</mu2>
-  </gazebo>
-  <xacro:damping_factor link="soft_link5"/>
-  <link name="soft_link6">
-    <inertial>
-      <origin xyz="0.10740316 0.0 0.003" rpy="0 0 0"/>
-      <mass value="0.059"/>
-      <inertia
-          ixx="0.00005433" ixy="0.00000033" ixz="0.0"
-          iyy="0.00047358" iyz="-0.00000369"
-          izz="0.00046011"/>
-    </inertial>
-    <visual>
-      <geometry>
-        <box size="${0.1175 + 0.054} 0.03 0.04"/>
-      </geometry>
-      <origin xyz="0.05875 0 0.02" rpy="0 0 0"/>
-    </visual>
-  </link>
-  <gazebo reference="soft_link6">
-    <mu1>0.1</mu1>
-    <mu2>0.1</mu2>
-  </gazebo>
-  <xacro:damping_factor link="soft_link6"/>
-  <transmission name="soft_joint_tran_5">
-    <type>transmission_interface/SimpleTransmission</type>
-    <joint name="soft_joint5">
-      <hardwareInterface>hardware_interface/EffortJointInterface</hardwareInterface>
-    </joint>
-    <actuator name="soft_joint_servo5">
-      <hardwareInterface>hardware_interface/EffortJointInterface</hardwareInterface>
-      <mechanicalReduction>1</mechanicalReduction>
-    </actuator>
-  </transmission>
-  <transmission name="soft_joint_tran_6">
-    <type>transmission_interface/SimpleTransmission</type>
-    <joint name="soft_joint6">
-      <hardwareInterface>hardware_interface/EffortJointInterface</hardwareInterface>
-    </joint>
-    <actuator name="soft_joint_servo6">
-      <hardwareInterface>hardware_interface/EffortJointInterface</hardwareInterface>
-      <mechanicalReduction>1</mechanicalReduction>
-    </actuator>
-  </transmission>
-  <!-- dummy_link -->
-  <joint name="servo_joint3" type="fixed">
-    <limit effort="5.0" lower="${-pi/2}" upper="${pi/2}" velocity="0.5"/>
-    <parent link="soft_link6"/>
-    <child link="servo_link3"/>
-    <origin xyz="0.1 0 0.01" rpy="0 0 0"/>
-    <axis xyz="0 0 1"/>
-    <dynamics damping="0.9" friction="0.1"/>
-  </joint>
-  <joint name="servo_joint4" type="fixed">
-    <limit effort="5.0" lower="${-pi/2}" upper="${pi/2}" velocity="0.5"/>
-    <parent link="soft_link6"/>
-    <child link="servo_link4"/>
-    <origin xyz="0.1 0 -0.01" rpy="0 0 0"/>
-    <axis xyz="0 0 1"/>
-    <dynamics damping="0.9" friction="0.1"/>
-  </joint>
-  <link name="servo_link3">
-    <inertial>
-      <origin xyz="0 0 0" rpy="0 0 0"/>
-      <mass value="0.073"/>
-      <inertia
-          ixx="0.000023" ixy="0.000003" ixz="-0.0000001"
-          iyy="0.000044" iyz="0.000000"
-          izz="0.000043"/>
-    </inertial>
-    <visual>
-      <geometry>
-        <box size="0.05 0.05 0.05"/>
-      </geometry>
-      <origin xyz="0 0 -0.02" rpy="0 0 0"/>
-    </visual>
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