Commit message: add soft_airframe urdf

File: robots/hydrus/robots/quad/soft_airframe_202605/robot.gazebo.xacro (robot description, xacro)
@@ -4,5 +4,5 @@
   <xacro:arg name="robot_name" default="hydrus" />
   <!-- robot urdf -->
-  <xacro:include filename="$(find hydrus)/robots/quad/default_mode_201907/robot.urdf.xacro" />
+  <xacro:include filename="$(find hydrus)/robots/quad/soft_airframe_202605/robot.urdf.xacro" />
   <!-- gazebo plugin for default controller and sensors -->
   <xacro:include filename="$(find aerial_robot_simulation)/xacro/spinal.gazebo.xacro" />

File: robots/hydrus/robots/quad/soft_airframe_202605/robot.urdf.xacro (robot description, xacro)
@@ -1,96 +1,41 @@
 <?xml version="1.0"?>
 <robot
-    xmlns:xacro="http://www.ros.org/wiki/xacro" name="hydrus" >
+    xmlns:xacro="http://www.ros.org/wiki/xacro" name="serial_soft_airframe" >
   <!-- basic kinematics model -->
   <xacro:include filename="$(find hydrus)/urdf/common.xacro" />
-  <xacro:include filename="$(find hydrus)/urdf/link.urdf.xacro" />
-  <xacro:hydrus_link links="4" self="1" rotor_direction="-1" with_battery = "0" />
-  <xacro:hydrus_link links="4" self="2" rotor_direction="1"  with_battery = "0" />
-  <xacro:hydrus_link links="4" self="3" rotor_direction="-1" with_battery = "0" />
-  <xacro:hydrus_link links="4" self="4" rotor_direction="1"  with_battery = "0" />
-  <!-- special battery arrangement -->
-  <xacro:extra_module name = "bat1" parent = "link1" visible = "1"
-                      model_url = "package://hydrus/urdf/mesh/battery/Kypom-3000-6s.dae" >
-    <origin xyz="${link_length/2} 0.0 -0.048" rpy="0 0 0"/>
+  <xacro:include filename="$(find hydrus)/urdf/soft_link.urdf.xacro" />
+  <!-- Dummy root link for KDL. There are no ordinary rigid airframe links. -->
+  <link name="root">
     <inertial>
       <origin xyz="0 0 0" rpy="0 0 0"/>
-      <mass value="0.4108"/>
+      <mass value="0.00001"/>
       <inertia
-          ixx="0.0001" iyy="0.0006" izz="0.0006"
-          ixy="0.0" ixz="0.0"  iyz="0.0"/>
+          ixx="0.000001" ixy="0.0" ixz="0.0"
+          iyy="0.000001" iyz="0.0"
+          izz="0.000002"/>
+    </inertial>
+  </link>
+  <joint name="root_joint" type="fixed">
+    <parent link="root"/>
+    <child link="servo_link1"/>
+    <origin rpy="0 0 0" xyz="0 0 0"/>
+    <axis xyz="0 0 1"/>
+  </joint>
+  <!-- flight controller -->
+  <xacro:extra_module name="fc_link" parent="root" visible="1" model_url="package://hydrus/urdf/mesh/ver2/flight_controller/spinal.dae">
+    <origin xyz="0.0735 0 0" rpy="0 0 0"/>
+    <inertial>
+      <origin xyz="0.02700000 0.00000000 0.01130642" rpy="0 0 0"/>
+      <mass value="0.02687673"/>
+      <inertia
+          ixx="0.00001064" ixy="0.00000000" ixz="0.00000000"
+          iyy="0.00001198" iyz="0.00000000"
+          izz="0.00001584"/>
     </inertial>
   </xacro:extra_module>
-  <xacro:extra_module name = "bat2" parent = "link4" visible = "1"
-                      model_url = "package://hydrus/urdf/mesh/battery/Kypom-3000-6s.dae" >
-    <origin xyz="${link_length/2} 0.0 -0.048" rpy="0 0 0"/>
+  <xacro:extra_module name="fc" parent="fc_link">
+    <origin xyz="0.0099 -0.0012 -0.019" rpy="0 0 0"/>
     <inertial>
-      <origin xyz="0 0 0" rpy="0 0 0"/>
-      <mass value="0.4108"/>
-      <inertia
-          ixx="0.0001" iyy="0.0006" izz="0.0006"
-          ixy="0.0" ixz="0.0"  iyz="0.0"/>
-    </inertial>
-  </xacro:extra_module>
-  <!-- onboard -->
-  <!-- 1.  processor -->
-  <!-- 1.1 flight controller -->
-  <xacro:extra_module name = "fc" parent = "link2" visible = "1"
-                      model_url = "package://hydrus/urdf/mesh/ver2/flight_controller/spinal.dae"> <!-- same with intel euclid -->
-    <origin xyz="${link_length / 2 + 0.2221} ${-4.4*0.001} 0.02135" rpy="0 0 0"/>
-    <inertial>
-      <mass value = "0.05" />
-      <origin xyz="${13*0.001} ${4.4*0.001} ${-9*0.001}" rpy="0 0 0"/>
-      <inertia
-          ixx="0.00001" ixy="0.0" ixz="0.0"
-          iyy="0.00001" iyz="0.0"
-          izz="0.00002"/>
-    </inertial>
-  </xacro:extra_module>
-  <!-- end: flight controller -->
-  <!-- 1.2 processor: jetson tx2 -->
-  <!-- confirm the inertial parameter with real machine -->
-  <xacro:extra_module name = "pc" parent = "link3" visible = "1"
-                      model_url = "package://hydrus/urdf/mesh/ver2/processor/jetson_tx2_unit.dae" >
-    <origin xyz="${link_length / 2 - 0.23775} 0.0 ${-0.01}" rpy="0 0 0"/>
-    <inertial>
-      <mass value = "0.181" />
-      <origin xyz="${18 * 0.001} ${4 * 0.001} ${-18 * 0.001}" rpy="0 0 0"/>
-      <inertia
-          ixx="0.00007" ixy="0.0" ixz="0.0"
-          iyy="0.00003" iyz="0.0"
-          izz="0.00009"/>
-    </inertial>
-  </xacro:extra_module>
-  <!-- end: processor: jetson tx2 -->
-  <!-- 2.  sensor -->
-  <!-- 2.1 leddar one -->
-  <xacro:extra_module name = "leddarone" parent = "link3" visible = "1"
-                      model_url = "package://hydrus/urdf/mesh/sensor/leddar_one_tx2_attached_mode.dae">
-    <origin xyz="${link_length/2 - 0.1855} 0.0 -0.0626" rpy="${pi} 0 0"/>
-    <inertial>
-      <origin xyz="-0.008 0.0 0.0" rpy="0 0 0"/>
-      <mass value="0.025"/>
-      <inertia
-          ixx="0.00001" iyy="0.000006" izz="0.00001"
-          ixy="0.000000" ixz="0.000000" iyz="0.000000"/>
-    </inertial>
-  </xacro:extra_module>
-  <!-- end: leddar one -->
-  <!-- 2.2 gps -->
-  <xacro:extra_module name = "gps" parent = "link2" visible = "1"
-                      model_url = "package://hydrus/urdf/mesh/sensor/gps_ublox_m8n.dae">
-    <origin xyz="${link_length/2 + 0.1925} 0.0 0.152" rpy="0 0 0"/>
-    <inertial>
-      <origin xyz="0.000000 0.000000 -0.013" rpy="0 0 0"/>
-      <mass value="0.042"/>
-      <inertia
-          ixx="0.00006" iyy="0.00006" izz="0.000007"
-          ixy="0.000000" ixz="0.000000" iyz="0.000000"/>
-    </inertial>
-  </xacro:extra_module>
-  <xacro:extra_module name = "magnet" parent = "gps">
-    <origin xyz="0 0 0" rpy="0 0 0"/>
-    <inertial>
-      <mass value = "0.00001" />
+      <mass value="0.00001"/>
       <origin xyz="0 0 0" rpy="0 0 0"/>
       <inertia
@@ -100,4 +45,42 @@
     </inertial>
   </xacro:extra_module>
-  <!-- end: gps -->
+  <!-- onboard computer -->
+  <xacro:extra_module name="vim4" parent="root" visible="1" model_url="package://hydrus/urdf/mesh/vim4.dae">
+    <origin xyz="0.3635 0.01 0" rpy="${-pi/2} 0 0"/>
+    <inertial>
+      <origin xyz="0.00146548 0.00262274 0.01119251" rpy="0 0 0"/>
+      <mass value="0.06613440"/>
+      <inertia
+          ixx="0.00001715" ixy="-0.00000087" ixz="0.00000023"
+          iyy="0.00003523" iyz="0.00000039"
+          izz="0.00004879"/>
+    </inertial>
+  </xacro:extra_module>
+  <!-- Four soft-link modules connected in series.
+       Module i creates:
+         servo_link{i}, soft_link{3*i-2}, soft_link{3*i-1}, soft_link{3*i}, gimbal_link{i}, thrust{i}
+  -->
+  <xacro:soft_link_module
+      i="1"
+      parent="root"
+      rotor_direction="1"
+      parent_to_soft_x="0.0"
+      parent_to_servo_x="0.0" />
+  <xacro:soft_link_module
+      i="2"
+      parent="gimbal_link1"
+      rotor_direction="-1" />
+  <!-- The third module has a slightly longer and larger servo body. -->
+  <xacro:soft_link_module
+      i="3"
+      parent="gimbal_link2"
+      rotor_direction="1"
+      servo_size_x="0.08"
+      servo_size_y="0.06"
+      servo_size_z="0.06"
+      servo_mass="0.18" />
+  <xacro:soft_link_module
+      i="4"
+      parent="gimbal_link3"
+      rotor_direction="-1" />
 </robot>
