Commit message: update urdf

File: robots/hydrus/robots/quad/soft_airframe_202605/robot.urdf.xacro (robot description, xacro)
@@ -16,10 +16,4 @@
     </inertial>
   </link>
-  <joint name="root_joint" type="fixed">
-    <parent link="root"/>
-    <child link="servo_link1"/>
-    <origin rpy="0 0 0" xyz="0 0 0"/>
-    <axis xyz="0 0 1"/>
-  </joint>
   <!-- flight controller -->
   <xacro:extra_module name="fc_link" parent="root" visible="1" model_url="package://hydrus/urdf/mesh/ver2/flight_controller/spinal.dae">

File: robots/hydrus/urdf/common.xacro (robot description, xacro)
@@ -17,5 +17,5 @@
   <xacro:property name="leg_collision_model_height" value="0.1715" />
   <!-- dynamics -->
-  <m_f_rate value="-0.0172" /> <!-- drug torque rate -->
+  <m_f_rate value="-0.0064" /> <!-- drug torque rate -->
   <xacro:property name="max_force" value="20.0" /> <!-- [N] -->
   <xacro:property name="min_force" value="1.0" /> <!-- [N] -->

File: robots/hydrus/urdf/soft_link.urdf.xacro (robot description, xacro)
@@ -6,4 +6,6 @@
       - servo_link${i}: a single combined servo body corresponding to old servo_link(2*i-1) + servo_link(2*i)
       - soft_link${3*i-2}, soft_link${3*i-1}, soft_link${3*i}
+      - leg${2*i-1}: attached at the root of soft_link${3*i-2}
+      - leg${2*i}: attached at the tip of soft_link${3*i}
       - gimbal_link${i}
       - thrust${i}
@@ -26,4 +28,8 @@
       soft_width:=0.03
       soft_height:=0.04
+      leg_length:=0.05
+      leg_size_x:=0.02
+      leg_size_y:=0.02
+      leg_mass:=0.005
       gimbal_offset_x:=0.128
       rotor_offset_x:=0.0735
@@ -33,4 +39,6 @@
     <xacro:property name="s1" value="${3 * i - 1}" />
     <xacro:property name="s2" value="${3 * i}" />
+    <xacro:property name="l0" value="${2 * i - 1}" />
+    <xacro:property name="l1" value="${2 * i}" />
     <!-- Combined servo body at the root of this module. -->
     <joint name="servo_joint${i}" type="fixed">
@@ -169,4 +177,70 @@
     </gazebo>
     <xacro:damping_factor link="soft_link${s2}"/>
+    <!-- Leg attached at the root of soft_link${s0}: leg${l0} -->
+    <joint name="leg_joint${l0}" type="fixed">
+      <parent link="soft_link${s0}"/>
+      <child link="leg${l0}"/>
+      <origin xyz="0 0 ${-leg_length * 0.5}" rpy="0 0 0"/>
+    </joint>
+    <link name="leg${l0}">
+      <inertial>
+        <origin xyz="0 0 ${-leg_length * 0.5}" rpy="0 0 0"/>
+        <mass value="${leg_mass}"/>
+        <inertia
+            ixx="0.00001" ixy="0.0" ixz="0.0"
+            iyy="0.00001" iyz="0.0"
+            izz="0.00001"/>
+      </inertial>
+      <visual>
+        <geometry>
+          <box size="${leg_size_x} ${leg_size_y} ${leg_length}"/>
+        </geometry>
+        <origin xyz="0 0 ${-leg_length * 0.5}" rpy="0 0 0"/>
+      </visual>
+      <collision>
+        <geometry>
+          <box size="${leg_size_x} ${leg_size_y} ${leg_length}"/>
+        </geometry>
+        <origin xyz="0 0 ${-leg_length * 0.5}" rpy="0 0 0"/>
+      </collision>
+    </link>
+    <gazebo reference="leg${l0}">
+      <mu1>0.1</mu1>
+      <mu2>0.1</mu2>
+    </gazebo>
+    <xacro:damping_factor link="leg${l0}"/>
+    <!-- Leg attached at the tip of soft_link${s2}: leg${l1} -->
+    <joint name="leg_joint${l1}" type="fixed">
+      <parent link="soft_link${s2}"/>
+      <child link="leg${l1}"/>
+      <origin xyz="${soft_l3} 0 ${-leg_length * 0.5}" rpy="0 0 0"/>
+    </joint>
+    <link name="leg${l1}">
+      <inertial>
+        <origin xyz="0 0 ${-leg_length * 0.5}" rpy="0 0 0"/>
+        <mass value="${leg_mass}"/>
+        <inertia
+            ixx="0.00001" ixy="0.0" ixz="0.0"
+            iyy="0.00001" iyz="0.0"
+            izz="0.00001"/>
+      </inertial>
+      <visual>
+        <geometry>
+          <box size="${leg_size_x} ${leg_size_y} ${leg_length}"/>
+        </geometry>
+        <origin xyz="0 0 ${-leg_length * 0.5}" rpy="0 0 0"/>
+      </visual>
+      <collision>
+        <geometry>
+          <box size="${leg_size_x} ${leg_size_y} ${leg_length}"/>
+        </geometry>
+        <origin xyz="0 0 ${-leg_length * 0.5}" rpy="0 0 0"/>
+      </collision>
+    </link>
+    <gazebo reference="leg${l1}">
+      <mu1>0.1</mu1>
+      <mu2>0.1</mu2>
+    </gazebo>
+    <xacro:damping_factor link="leg${l1}"/>
     <transmission name="soft_joint_tran_${s1}">
       <type>transmission_interface/SimpleTransmission</type>

Commit message: update urdf

File: robots/hydrus/robots/quad/soft_airframe_202605/robot.urdf.xacro (robot description, xacro)
@@ -17,6 +17,6 @@
   </link>
   <!-- flight controller -->
-  <xacro:extra_module name="fc_link" parent="root" visible="1" model_url="package://hydrus/urdf/mesh/ver2/flight_controller/spinal.dae">
-    <origin xyz="0.0735 0 0" rpy="0 0 0"/>
+  <xacro:extra_module name="fc_link" parent="servo_link3" visible="1" model_url="package://hydrus/urdf/mesh/ver2/flight_controller/spinal.dae">
+    <origin xyz="0.05 0 0.01" rpy="0 0 0"/>
     <inertial>
       <origin xyz="0.02700000 0.00000000 0.01130642" rpy="0 0 0"/>
@@ -40,6 +40,6 @@
   </xacro:extra_module>
   <!-- onboard computer -->
-  <xacro:extra_module name="vim4" parent="root" visible="1" model_url="package://hydrus/urdf/mesh/vim4.dae">
-    <origin xyz="0.3635 0.01 0" rpy="${-pi/2} 0 0"/>
+  <xacro:extra_module name="vim4" parent="servo_link3" visible="1" model_url="package://hydrus/urdf/mesh/vim4.dae">
+    <origin xyz="0.05 0 -0.01" rpy="0 0 0"/>
     <inertial>
       <origin xyz="0.00146548 0.00262274 0.01119251" rpy="0 0 0"/>
@@ -59,5 +59,4 @@
       parent="root"
       rotor_direction="1"
-      parent_to_soft_x="0.0"
       parent_to_servo_x="0.0" />
   <xacro:soft_link_module
@@ -70,7 +69,7 @@
       parent="gimbal_link2"
       rotor_direction="1"
-      servo_size_x="0.08"
+      servo_size_x="0.156"
       servo_size_y="0.06"
-      servo_size_z="0.06"
+      servo_size_z="0.01"
       servo_mass="0.18" />
   <xacro:soft_link_module

File: robots/hydrus/urdf/soft_link.urdf.xacro (robot description, xacro)
@@ -16,8 +16,7 @@
       parent
       rotor_direction:=1
-      parent_to_soft_x:=0.147
-      parent_to_servo_x:=0.0
-      servo_z_offset:=0.0
-      servo_size_x:=0.05
+      parent_to_servo_x:=0.147
+      parent_to_servo_cog:=0.0567
+      servo_size_x:=0.096
       servo_size_y:=0.05
       servo_size_z:=0.05
@@ -28,9 +27,8 @@
       soft_width:=0.03
       soft_height:=0.04
-      leg_length:=0.05
+      leg_length:=0.120
       leg_size_x:=0.02
       leg_size_y:=0.02
-      leg_mass:=0.005
-      gimbal_offset_x:=0.128
+      leg_mass:=0.04993
       rotor_offset_x:=0.0735
       gimbal_mesh:=package://hydrus/urdf/mesh/5inch_propeller_duct_right_v2.dae
@@ -45,14 +43,14 @@
       <parent link="${parent}"/>
       <child link="servo_link${i}"/>
-      <origin xyz="${parent_to_servo_x} 0 ${servo_z_offset}" rpy="0 0 0"/>
+      <origin xyz="${parent_to_servo_x} 0 0" rpy="0 0 0"/>
     </joint>
     <link name="servo_link${i}">
       <inertial>
-        <origin xyz="0 0 0" rpy="0 0 0"/>
+        <origin xyz="${parent_to_servo_cog} 0 0" rpy="0 0 0"/>
         <mass value="${servo_mass}"/>
         <inertia
-            ixx="0.000045" ixy="0.0" ixz="0.0"
-            iyy="0.000086" iyz="0.0"
-            izz="0.000084"/>
+            ixx="0.00006467" ixy="0.0" ixz="0.0"
+            iyy="0.00012455" iyz="0.0"
+            izz="0.00009760"/>
       </inertial>
       <visual>
@@ -60,12 +58,6 @@
           <box size="${servo_size_x} ${servo_size_y} ${servo_size_z}"/>
         </geometry>
-        <origin xyz="0 0 0" rpy="0 0 0"/>
-      </visual>
-      <collision>
-        <geometry>
-          <box size="${servo_size_x} ${servo_size_y} ${servo_size_z}"/>
-        </geometry>
-        <origin xyz="0 0 0" rpy="0 0 0"/>
-      </collision>
+        <origin xyz="${parent_to_servo_cog} 0 0" rpy="0 0 0"/>
+      </visual>
     </link>
     <gazebo reference="servo_link${i}">
@@ -76,7 +68,7 @@
     <!-- Three-segment soft continuum approximation. -->
     <joint name="soft_joint${s0}" type="fixed">
-      <parent link="${parent}"/>
+      <parent link="servo_link${i}"/>
       <child link="soft_link${s0}"/>
-      <origin xyz="${parent_to_soft_x} 0 0" rpy="0 0 0"/>
+      <origin xyz="${servo_size_x} 0 0" rpy="0 0 0"/>
     </joint>
     <joint name="soft_joint${s1}" type="revolute">
@@ -98,5 +90,5 @@
     <link name="soft_link${s0}">
       <inertial>
-        <origin xyz="${soft_l1 * 0.5} 0.000002 ${soft_height * 0.5}" rpy="0 0 0"/>
+        <origin xyz="${soft_l1 * 0.5} 0.000002 0" rpy="0 0 0"/>
         <mass value="0.059"/>
         <inertia
@@ -109,12 +101,6 @@
           <box size="${soft_l1} ${soft_width} ${soft_height}"/>
         </geometry>
-        <origin xyz="${soft_l1 * 0.5} 0 ${soft_height * 0.5}" rpy="0 0 0"/>
-      </visual>
-      <collision>
-        <geometry>
-          <box size="${soft_l1} ${soft_width} ${soft_height}"/>
-        </geometry>
-        <origin xyz="${soft_l1 * 0.5} 0 ${soft_height * 0.5}" rpy="0 0 0"/>
-      </collision>
+        <origin xyz="${soft_l1 * 0.5} 0 0" rpy="0 0 0"/>
+      </visual>
     </link>
     <gazebo reference="soft_link${s0}">
@@ -125,5 +111,5 @@
     <link name="soft_link${s1}">
       <inertial>
-        <origin xyz="${soft_l2 * 0.5} 0.000002 ${soft_height * 0.5}" rpy="0 0 0"/>
+        <origin xyz="${soft_l2 * 0.5} 0.000002 0" rpy="0 0 0"/>
         <mass value="0.118"/>
         <inertia
@@ -136,12 +122,6 @@
           <box size="${soft_l2} ${soft_width} ${soft_height}"/>
         </geometry>
-        <origin xyz="${soft_l2 * 0.5} 0 ${soft_height * 0.5}" rpy="0 0 0"/>
-      </visual>
-      <collision>
-        <geometry>
-          <box size="${soft_l2} ${soft_width} ${soft_height}"/>
-        </geometry>
-        <origin xyz="${soft_l2 * 0.5} 0 ${soft_height * 0.5}" rpy="0 0 0"/>
-      </collision>
+        <origin xyz="${soft_l2 * 0.5} 0 0" rpy="0 0 0"/>
+      </visual>
     </link>
     <gazebo reference="soft_link${s1}">
@@ -152,5 +132,5 @@
     <link name="soft_link${s2}">
       <inertial>
-        <origin xyz="${soft_l3 * 0.5} 0.0 ${soft_height * 0.5}" rpy="0 0 0"/>
+        <origin xyz="${soft_l3 * 0.5} 0.0 0" rpy="0 0 0"/>
         <mass value="0.059"/>
         <inertia
@@ -163,12 +143,6 @@
           <box size="${soft_l3} ${soft_width} ${soft_height}"/>
         </geometry>
-        <origin xyz="${soft_l3 * 0.5} 0 ${soft_height * 0.5}" rpy="0 0 0"/>
-      </visual>
-      <collision>
-        <geometry>
-          <box size="${soft_l3} ${soft_width} ${soft_height}"/>
-        </geometry>
-        <origin xyz="${soft_l3 * 0.5} 0 ${soft_height * 0.5}" rpy="0 0 0"/>
-      </collision>
+        <origin xyz="${soft_l3 * 0.5} 0 0" rpy="0 0 0"/>
+      </visual>
     </link>
     <gazebo reference="soft_link${s2}">
@@ -181,14 +155,14 @@
       <parent link="soft_link${s0}"/>
       <child link="leg${l0}"/>
-      <origin xyz="0 0 ${-leg_length * 0.5}" rpy="0 0 0"/>
+      <origin xyz="0 0 -0.041" rpy="0 0 0"/>
     </joint>
     <link name="leg${l0}">
       <inertial>
-        <origin xyz="0 0 ${-leg_length * 0.5}" rpy="0 0 0"/>
+        <origin xyz="0 0 -0.096" rpy="0 0 0"/>
         <mass value="${leg_mass}"/>
         <inertia
-            ixx="0.00001" ixy="0.0" ixz="0.0"
-            iyy="0.00001" iyz="0.0"
-            izz="0.00001"/>
+            ixx="0.00009073" ixy="0.0" ixz="0.0"
+            iyy="0.00005301" iyz="0.0"
+            izz="0.00003904"/>
       </inertial>
       <visual>
@@ -214,14 +188,14 @@
       <parent link="soft_link${s2}"/>
       <child link="leg${l1}"/>
-      <origin xyz="${soft_l3} 0 ${-leg_length * 0.5}" rpy="0 0 0"/>
+      <origin xyz="${soft_l3} 0 -0.041" rpy="0 0 0"/>
     </joint>
     <link name="leg${l1}">
       <inertial>
-        <origin xyz="0 0 ${-leg_length * 0.5}" rpy="0 0 0"/>
+        <origin xyz="0 0 -0.096" rpy="0 0 0"/>
         <mass value="${leg_mass}"/>
         <inertia
-            ixx="0.00001" ixy="0.0" ixz="0.0"
-            iyy="0.00001" iyz="0.0"
-            izz="0.00001"/>
+            ixx="0.00009073" ixy="0.0" ixz="0.0"
+            iyy="0.00005301" iyz="0.0"
+            izz="0.00003904"/>
       </inertial>
       <visual>
@@ -267,5 +241,5 @@
       <parent link="soft_link${s2}"/>
       <child link="gimbal_link${i}"/>
-      <origin xyz="${gimbal_offset_x} 0 0" rpy="0 0 0"/>
+      <origin xyz="${soft_l3} 0 0" rpy="0 0 0"/>
       <axis xyz="1 0 0"/>
       <dynamics damping="0.9" friction="0.1"/>
@@ -273,5 +247,5 @@
     <link name="gimbal_link${i}">
       <inertial>
-        <origin xyz="0.0815 0 0" rpy="0 0 0"/>
+        <origin xyz="0.0735 0 0" rpy="0 0 0"/>
         <mass value="0.222"/>
         <inertia
@@ -281,5 +255,5 @@
       </inertial>
       <visual>
-        <origin xyz="0.0815 0 0" rpy="0 0 0"/>
+        <origin xyz="0.0735 0 0" rpy="0 0 0"/>
         <geometry>
           <mesh filename="${gimbal_mesh}"/>
@@ -293,5 +267,5 @@
     <xacro:damping_factor link="gimbal_link${i}"/>
     <joint name="rotor${i}" type="continuous">
-      <limit effort="0.0064" lower="0.0" upper="20.0" velocity="0.5"/>
+      <limit effort="0.0172" lower="0.0" upper="20.0" velocity="0.5"/>
       <parent link="gimbal_link${i}"/>
       <child link="thrust${i}"/>

Commit message: split into five segments

File: robots/hydrus/robots/quad/soft_airframe_202605/robot.urdf.xacro (robot description, xacro)
@@ -53,5 +53,5 @@
   <!-- Four soft-link modules connected in series.
        Module i creates:
-         servo_link{i}, soft_link{3*i-2}, soft_link{3*i-1}, soft_link{3*i}, gimbal_link{i}, thrust{i}
+         servo_link{i}, soft_link{5*i-4..5*i}, gimbal_link{i}, thrust{i}
   -->
   <xacro:soft_link_module

File: robots/hydrus/urdf/soft_link.urdf.xacro (robot description, xacro)
@@ -19,8 +19,8 @@
     A macro for one soft-link module.
     Module i consists of:
-      - soft_link${3*i-2}, soft_link${3*i-1}, soft_link${3*i}
+      - soft_link${5*i-4}, soft_link${5*i-3}, soft_link${5*i-2}, soft_link${5*i-1}, soft_link${5*i}
       - servo_link${i}: a single combined servo body corresponding to old servo_link(2*i-1) + servo_link(2*i)
-      - leg${2*i-1}: attached at the root of soft_link${3*i-2}
-      - leg${2*i}: attached at the tip of soft_link${3*i}
+      - leg${2*i-1}: attached at the root of soft_link${5*i-4}
+      - leg${2*i}: attached at the tip of soft_link${5*i}
       - gimbal_link${i}
       - thrust${i}
@@ -37,7 +37,9 @@
       servo_size_z:=0.05
       servo_mass:=0.141
-      soft_l1:=0.1175
-      soft_l2:=0.235
+      soft_l1:=0.05875
+      soft_l2:=0.1175
       soft_l3:=0.1175
+      soft_l4:=0.1175
+      soft_l5:=0.05875
       soft_width:=0.03
       soft_height:=0.04
@@ -49,10 +51,12 @@
       gimbal_mesh:=package://hydrus/urdf/mesh/5inch_propeller_duct_right_v2.dae
       propeller_mesh:=package://hydrus/urdf/mesh/TriBlade_5045.dae">
-    <xacro:property name="s0" value="${3 * i - 2}" />
-    <xacro:property name="s1" value="${3 * i - 1}" />
-    <xacro:property name="s2" value="${3 * i}" />
+    <xacro:property name="s0" value="${5 * i - 4}" />
+    <xacro:property name="s1" value="${5 * i - 3}" />
+    <xacro:property name="s2" value="${5 * i - 2}" />
+    <xacro:property name="s3" value="${5 * i - 1}" />
+    <xacro:property name="s4" value="${5 * i}" />
     <xacro:property name="l0" value="${2 * i - 1}" />
     <xacro:property name="l1" value="${2 * i}" />
-    <!-- Three-segment soft continuum approximation. -->
+    <!-- Five-segment soft continuum approximation (1/8, 1/4, 1/4, 1/4, 1/8). -->
     <joint name="soft_joint${s0}" type="fixed">
       <parent link="${parent}"/>
@@ -76,7 +80,45 @@
       <dynamics damping="0.2" friction="0.1"/>
     </joint>
+    <joint name="soft_joint${s3}" type="revolute">
+      <limit effort="5.0" lower="${-pi}" upper="${pi}" velocity="0.5"/>
+      <parent link="soft_link${s2}"/>
+      <child link="soft_link${s3}"/>
+      <origin xyz="${soft_l3} 0 0" rpy="0 0 0"/>
+      <axis xyz="0 0 1"/>
+      <dynamics damping="0.2" friction="0.1"/>
+    </joint>
+    <joint name="soft_joint${s4}" type="revolute">
+      <limit effort="5.0" lower="${-pi}" upper="${pi}" velocity="0.5"/>
+      <parent link="soft_link${s3}"/>
+      <child link="soft_link${s4}"/>
+      <origin xyz="${soft_l4} 0 0" rpy="0 0 0"/>
+      <axis xyz="0 0 1"/>
+      <dynamics damping="0.2" friction="0.1"/>
+    </joint>
     <link name="soft_link${s0}">
       <inertial>
         <origin xyz="${soft_l1 * 0.5} 0.000002 0" rpy="0 0 0"/>
+        <mass value="0.0295"/>
+        <inertia
+            ixx="0.000027165" ixy="0.00000004125" ixz="0.0"
+            iyy="0.0000591975" iyz="-0.00000046125"
+            izz="0.00005751375"/>
+      </inertial>
+      <visual>
+        <geometry>
+          <box size="${soft_l1} ${soft_width} ${soft_height}"/>
+        </geometry>
+        <material name="soft_link_material"/>
+        <origin xyz="${soft_l1 * 0.5} 0 0" rpy="0 0 0"/>
+      </visual>
+    </link>
+    <gazebo reference="soft_link${s0}">
+      <mu1>0.1</mu1>
+      <mu2>0.1</mu2>
+    </gazebo>
+    <xacro:damping_factor link="soft_link${s0}"/>
+    <link name="soft_link${s1}">
+      <inertial>
+        <origin xyz="${soft_l2 * 0.5} 0.000002 0" rpy="0 0 0"/>
         <mass value="0.059"/>
         <inertia
@@ -87,26 +129,4 @@
       <visual>
         <geometry>
-          <box size="${soft_l1} ${soft_width} ${soft_height}"/>
-        </geometry>
-        <material name="soft_link_material"/>
-        <origin xyz="${soft_l1 * 0.5} 0 0" rpy="0 0 0"/>
-      </visual>
-    </link>
-    <gazebo reference="soft_link${s0}">
-      <mu1>0.1</mu1>
-      <mu2>0.1</mu2>
-    </gazebo>
-    <xacro:damping_factor link="soft_link${s0}"/>
-    <link name="soft_link${s1}">
-      <inertial>
-        <origin xyz="${soft_l2 * 0.5} 0.000002 0" rpy="0 0 0"/>
-        <mass value="0.118"/>
-        <inertia
-            ixx="0.00007941" ixy="0.00000218" ixz="0.0"
-            iyy="0.00065133" iyz="0.0"
-            izz="0.00062639"/>
-      </inertial>
-      <visual>
-        <geometry>
           <box size="${soft_l2} ${soft_width} ${soft_height}"/>
         </geometry>
@@ -122,5 +142,5 @@
     <link name="soft_link${s2}">
       <inertial>
-        <origin xyz="${soft_l3 * 0.5} 0.0 0" rpy="0 0 0"/>
+        <origin xyz="${soft_l3 * 0.5} 0.000002 0" rpy="0 0 0"/>
         <mass value="0.059"/>
         <inertia
@@ -142,9 +162,53 @@
     </gazebo>
     <xacro:damping_factor link="soft_link${s2}"/>
+    <link name="soft_link${s3}">
+      <inertial>
+        <origin xyz="${soft_l4 * 0.5} 0.000002 0" rpy="0 0 0"/>
+        <mass value="0.059"/>
+        <inertia
+            ixx="0.00005433" ixy="0.00000033" ixz="0.0"
+            iyy="0.00047358" iyz="-0.00000369"
+            izz="0.00046011"/>
+      </inertial>
+      <visual>
+        <geometry>
+          <box size="${soft_l4} ${soft_width} ${soft_height}"/>
+        </geometry>
+        <material name="soft_link_material"/>
+        <origin xyz="${soft_l4 * 0.5} 0 0" rpy="0 0 0"/>
+      </visual>
+    </link>
+    <gazebo reference="soft_link${s3}">
+      <mu1>0.1</mu1>
+      <mu2>0.1</mu2>
+    </gazebo>
+    <xacro:damping_factor link="soft_link${s3}"/>
+    <link name="soft_link${s4}">
+      <inertial>
+        <origin xyz="${soft_l5 * 0.5} 0.000002 0" rpy="0 0 0"/>
+        <mass value="0.0295"/>
+        <inertia
+            ixx="0.000027165" ixy="0.00000004125" ixz="0.0"
+            iyy="0.0000591975" iyz="-0.00000046125"
+            izz="0.00005751375"/>
+      </inertial>
+      <visual>
+        <geometry>
+          <box size="${soft_l5} ${soft_width} ${soft_height}"/>
+        </geometry>
+        <material name="soft_link_material"/>
+        <origin xyz="${soft_l5 * 0.5} 0 0" rpy="0 0 0"/>
+      </visual>
+    </link>
+    <gazebo reference="soft_link${s4}">
+      <mu1>0.1</mu1>
+      <mu2>0.1</mu2>
+    </gazebo>
+    <xacro:damping_factor link="soft_link${s4}"/>
     <!-- Combined servo body after the soft-link chain. -->
     <joint name="servo_joint${i}" type="fixed">
-      <parent link="soft_link${s2}"/>
+      <parent link="soft_link${s4}"/>
       <child link="servo_link${i}"/>
-      <origin xyz="${soft_l3} 0 0" rpy="0 0 0"/>
+      <origin xyz="${soft_l5} 0 0" rpy="0 0 0"/>
     </joint>
     <link name="servo_link${i}">
@@ -204,9 +268,9 @@
     </gazebo>
     <xacro:damping_factor link="leg${l0}"/>
-    <!-- Leg attached at the tip of soft_link${s2}: leg${l1} -->
+    <!-- Leg attached at the tip of soft_link${s4}: leg${l1} -->
     <joint name="leg_joint${l1}" type="fixed">
-      <parent link="soft_link${s2}"/>
+      <parent link="soft_link${s4}"/>
       <child link="leg${l1}"/>
-      <origin xyz="${soft_l3} 0 -0.041" rpy="0 0 0"/>
+      <origin xyz="${soft_l5} 0 -0.041" rpy="0 0 0"/>
     </joint>
     <link name="leg${l1}">
@@ -254,4 +318,24 @@
       </joint>
       <actuator name="soft_joint_servo${s2}">
+        <hardwareInterface>hardware_interface/EffortJointInterface</hardwareInterface>
+        <mechanicalReduction>1</mechanicalReduction>
+      </actuator>
+    </transmission>
+    <transmission name="soft_joint_tran_${s3}">
+      <type>transmission_interface/SimpleTransmission</type>
+      <joint name="soft_joint${s3}">
+        <hardwareInterface>hardware_interface/EffortJointInterface</hardwareInterface>
+      </joint>
+      <actuator name="soft_joint_servo${s3}">
+        <hardwareInterface>hardware_interface/EffortJointInterface</hardwareInterface>
+        <mechanicalReduction>1</mechanicalReduction>
+      </actuator>
+    </transmission>
+    <transmission name="soft_joint_tran_${s4}">
+      <type>transmission_interface/SimpleTransmission</type>
+      <joint name="soft_joint${s4}">
+        <hardwareInterface>hardware_interface/EffortJointInterface</hardwareInterface>
+      </joint>
+      <actuator name="soft_joint_servo${s4}">
         <hardwareInterface>hardware_interface/EffortJointInterface</hardwareInterface>
         <mechanicalReduction>1</mechanicalReduction>
