Commit message: tilt the model

File: robots/hydrus/robots/quad/soft_airframe_202605/robot.urdf.xacro (robot description, xacro)
@@ -59,5 +59,6 @@
       parent="root"
       rotor_direction="-1"
-      parent_to_servo_x="0.0" />
+      parent_to_servo_x="0.0"
+      tilt_angle="-0.174" />
   <xacro:soft_link_module
       i="2"
@@ -67,13 +68,16 @@
       servo_size_y="0.06"
       servo_size_z="0.01"
-      servo_mass="0.18" />
+      servo_mass="0.18"
+      tilt_angle="0.174" />
   <!-- The third module has a slightly longer and larger servo body. -->
   <xacro:soft_link_module
       i="3"
       parent="gimbal_link2"
-      rotor_direction="-1" />
+      rotor_direction="-1"
+      tilt_angle="-0.174" />
   <xacro:soft_link_module
       i="4"
       parent="gimbal_link3"
-      rotor_direction="1" />
+      rotor_direction="1"
+      tilt_angle="0.174" />
 </robot>

File: robots/hydrus/urdf/soft_link.urdf.xacro (robot description, xacro)
@@ -49,4 +49,5 @@
       leg_mass:=0.04993
       rotor_offset_x:=0.0735
+      tilt_angle:=0.174
       gimbal_mesh:=package://hydrus/urdf/mesh/5inch_propeller_duct_right_v2.dae
       propeller_mesh:=package://hydrus/urdf/mesh/TriBlade_5045.dae">
@@ -352,5 +353,5 @@
     <link name="gimbal_link${i}">
       <inertial>
-        <origin xyz="0.0735 0 0" rpy="0 0 0"/>
+        <origin xyz="0.0735 0 0" rpy="0 ${tilt_angle} 0"/>
         <mass value="0.222"/>
         <inertia
@@ -360,5 +361,5 @@
       </inertial>
       <visual>
-        <origin xyz="0.0735 0 0" rpy="0 0 0"/>
+        <origin xyz="0.0735 0 0" rpy="0 ${tilt_angle} 0"/>
         <geometry>
           <mesh filename="${gimbal_mesh}"/>

Commit message: tilt with gazebo

File: robots/hydrus/robots/quad/soft_airframe_202605/robot.urdf.xacro (robot description, xacro)
@@ -59,5 +59,7 @@
       parent="root"
       rotor_direction="-1"
-      parent_to_servo_x="0.0" />
+      parent_to_servo_x="0.0"
+      prev_tilt_angle="0"
+      tilt_angle="-0.174" />
   <xacro:soft_link_module
       i="2"
@@ -67,13 +69,19 @@
       servo_size_y="0.06"
       servo_size_z="0.01"
-      servo_mass="0.18" />
+      servo_mass="0.18"
+      prev_tilt_angle="0.174"
+      tilt_angle="0.174" />
   <!-- The third module has a slightly longer and larger servo body. -->
   <xacro:soft_link_module
       i="3"
       parent="gimbal_link2"
-      rotor_direction="-1" />
+      rotor_direction="-1"
+      prev_tilt_angle="-0.174"
+      tilt_angle="-0.174" />
   <xacro:soft_link_module
       i="4"
       parent="gimbal_link3"
-      rotor_direction="1" />
+      rotor_direction="1"
+      prev_tilt_angle="0.174"
+      tilt_angle="0.174" />
 </robot>

File: robots/hydrus/urdf/soft_link.urdf.xacro (robot description, xacro)
@@ -47,4 +47,6 @@
       leg_mass:=0.04993
       rotor_offset_x:=0.0735
+      tilt_angle:=-0.174
+      prev_tilt_angle:=0.174
       gimbal_mesh:=package://hydrus/urdf/mesh/5inch_propeller_duct_right_v2.dae
       propeller_mesh:=package://hydrus/urdf/mesh/TriBlade_5045.dae">
@@ -58,5 +60,5 @@
       <parent link="${parent}"/>
       <child link="soft_link${s0}"/>
-      <origin xyz="${parent_to_servo_x} 0 0" rpy="0 0 0"/>
+      <origin xyz="${parent_to_servo_x} 0 0" rpy="0 ${prev_tilt_angle} 0"/>
     </joint>
     <joint name="soft_joint${s1}" type="revolute">
@@ -262,5 +264,5 @@
       <parent link="servo_link${i}"/>
       <child link="gimbal_link${i}"/>
-      <origin xyz="${servo_size_x} 0 0" rpy="0 0 0"/>
+      <origin xyz="${servo_size_x} 0 0" rpy="0 ${tilt_angle} 0"/>
       <axis xyz="1 0 0"/>
       <dynamics damping="0.9" friction="0.1"/>
