Commit message: update urdf

File: robots/hydrus/robots/quad/soft_airframe_202605/robot.urdf.xacro (robot description, xacro)
@@ -61,5 +61,6 @@
       parent_to_servo_x="0.0"
       prev_tilt_angle="0"
-      tilt_angle="0.174" />
+      tilt_angle="0.174"
+      soft_weight_sum="0.251" />
   <xacro:soft_link_module
       i="2"

File: robots/hydrus/urdf/soft_link.urdf.xacro (robot description, xacro)
@@ -51,4 +51,5 @@
       tilt_angle:=-0.174
       prev_tilt_angle:=0.174
+      soft_weight_sum:=0.311
       gimbal_mesh:=package://hydrus/urdf/mesh/5inch_propeller_duct_right_v2.dae
       propeller_mesh:=package://hydrus/urdf/mesh/TriBlade_5045.dae">
@@ -104,5 +105,5 @@
       <inertial>
         <origin xyz="${soft_l1 * 0.5} 0.000002 0" rpy="0 0 0"/>
-        <mass value="0.0295"/>
+        <mass value="${soft_weight_sum/4/2}"/>
         <inertia
             ixx="0.000027165" ixy="0.00000004125" ixz="0.0"
@@ -126,5 +127,5 @@
       <inertial>
         <origin xyz="${soft_l2 * 0.5} 0.000002 0" rpy="0 0 0"/>
-        <mass value="0.059"/>
+        <mass value="${soft_weight_sum/4}"/>
         <inertia
             ixx="0.00005433" ixy="0.00000033" ixz="0.0"
@@ -148,5 +149,5 @@
       <inertial>
         <origin xyz="${soft_l3 * 0.5} 0.000002 0" rpy="0 0 0"/>
-        <mass value="0.059"/>
+        <mass value="${soft_weight_sum/4}"/>
         <inertia
             ixx="0.00005433" ixy="0.00000033" ixz="0.0"
@@ -170,5 +171,5 @@
       <inertial>
         <origin xyz="${soft_l4 * 0.5} 0.000002 0" rpy="0 0 0"/>
-        <mass value="0.059"/>
+        <mass value="${soft_weight_sum/4}"/>
         <inertia
             ixx="0.00005433" ixy="0.00000033" ixz="0.0"
@@ -192,5 +193,5 @@
       <inertial>
         <origin xyz="${soft_l5 * 0.5} 0.000002 0" rpy="0 0 0"/>
-        <mass value="0.0295"/>
+        <mass value="${soft_weight_sum/4/2}"/>
         <inertia
             ixx="0.000027165" ixy="0.00000004125" ixz="0.0"
@@ -358,5 +359,6 @@
       <inertial>
         <origin xyz="0.0735 0 0" rpy="0 0 0"/>
-        <mass value="0.222"/>
+        <!-- 0.032 is the mass of ESC -->
+        <mass value="${0.222 + 0.032}"/>
         <inertia
             ixx="0.00022661" ixy="0.0" ixz="0.0"
