Commit message: fix urdf source

File: robots/uuv_d/urdf/mesh/proto_type/urdf/proto_type_dae.urdf (robot description, URDF)
Before this commit: robot proto_type, 9 links, 8 joints
Links:
- link base_link: geometry collision mesh filename=package://proto_type/meshes/base_link.stl; visual mesh filename=package://proto_type/meshes/base_link.dae
- link thruster_0: geometry collision mesh filename=package://proto_type/meshes/thruster_0.stl; visual mesh filename=package://proto_type/meshes/thruster_0.dae
- link thruster_1: geometry collision mesh filename=package://proto_type/meshes/thruster_1.stl; visual mesh filename=package://proto_type/meshes/thruster_1.dae
- link thruster_2: geometry collision mesh filename=package://proto_type/meshes/thruster_2.stl; visual mesh filename=package://proto_type/meshes/thruster_2.dae
- link thruster_3: geometry collision mesh filename=package://proto_type/meshes/thruster_3.stl; visual mesh filename=package://proto_type/meshes/thruster_3.dae
- link thruster_4: geometry collision mesh filename=package://proto_type/meshes/thruster_4.stl; visual mesh filename=package://proto_type/meshes/thruster_4.dae
- link thruster_5: geometry collision mesh filename=package://proto_type/meshes/thruster_5.stl; visual mesh filename=package://proto_type/meshes/thruster_5.dae
- link thruster_6: geometry collision mesh filename=package://proto_type/meshes/thruster_6.stl; visual mesh filename=package://proto_type/meshes/thruster_6.dae
- link thruster_7: geometry collision mesh filename=package://proto_type/meshes/thruster_7.stl; visual mesh filename=package://proto_type/meshes/thruster_7.dae
