Commit message: update urdf

File: robots/uuv_d/robots/quad/default_mode_201907/robot.urdf.xacro (robot description, xacro)
@@ -1,4 +1,21 @@
 <?xml version='1.0' encoding='UTF-8'?>
 <robot xmlns:xacro="http://www.ros.org/wiki/xacro" name="proto_type">
+<m_f_rate value="-0.0172" />
+  <link name="root">
+      <inertial>
+        <origin xyz="0 0 0" rpy="0 0 0"/>
+        <mass value="0.00001"/>
+        <inertia
+            ixx="0.000001" ixy="0.0" ixz="0.0"
+            iyy="0.000001" iyz="0.0"
+            izz="0.000001"/>
+      </inertial>
+    </link>
+    <joint name="root_joint" type="fixed">
+      <parent link="root"/>
+      <child link="base_link"/>
+      <origin rpy="0 0 0" xyz="0 0 0"/>
+      <axis xyz="0 0 1"/>
+    </joint>
   <link name="base_link">
     <inertial>
@@ -21,4 +38,46 @@
     </collision>
   </link>
+  <link name="fc">
+      <inertial>
+        <origin xyz="0 0 0" rpy="0 0 0"/>
+        <mass value="0.00001"/>
+        <inertia
+            ixx="0.000001" ixy="0.0" ixz="0.0"
+            iyy="0.000001" iyz="0.0"
+            izz="0.000001"/>
+      </inertial>
+    </link>
+    <joint name="fc_joint" type="fixed">
+      <child link="fc"/>
+      <parent link="base_link"/>
+      <origin rpy="0 0 0" xyz="0 0 0"/>
+      <axis xyz="0 0 1"/>
+    </joint>
+  <xacro:macro name="add_rotor_and_thrust" params="id parent min_thrust max_thrust direction">
+    <link name="thrust${id}">
+      <inertial>
+        <origin xyz="0 0 0" rpy="0 0 0"/>
+        <mass value="0.0001"/>
+        <inertia ixx="0.00001" ixy="0.0" ixz="0.0" iyy="0.00001" iyz="0.0" izz="0.00002"/>
+      </inertial>
+    </link>
+    <joint name="rotor${id}" type="continuous">
+      <limit effort="100.0" lower="${min_thrust}" upper="${max_thrust}" velocity="50.0"/>
+      <parent link="${parent}"/>
+      <child link="thrust${id}"/>
+      <origin xyz="0 0 0" rpy="0 0 0"/>
+      <axis xyz="0 0 ${direction}"/>
+    </joint>
+    <transmission name="rotor_tran${id}">
+      <type>transmission_interface/SimpleTransmission</type>
+      <joint name="rotor${id}">
+        <hardwareInterface>RotorInterface</hardwareInterface>
+      </joint>
+      <actuator name="actuator_rotor_${id}">
+        <hardwareInterface>RotorInterface</hardwareInterface>
+        <mechanicalReduction>1</mechanicalReduction>
+      </actuator>
+    </transmission>
+  </xacro:macro>
   <link name="thruster_0">
     <inertial>
@@ -264,3 +323,13 @@
     <color rgba="0.79216 0.81961 0.93333 1.     "/>
   </material>
+  <xacro:property name="min_t" value="-20.0" />
+  <xacro:property name="max_t" value="20.0" />
+  <xacro:add_rotor_and_thrust id="1" parent="thruster_0" min_thrust="${min_t}" max_thrust="${max_t}" direction="1"/>
+  <xacro:add_rotor_and_thrust id="2" parent="thruster_1" min_thrust="${min_t}" max_thrust="${max_t}" direction="-1"/>
+  <xacro:add_rotor_and_thrust id="3" parent="thruster_2" min_thrust="${min_t}" max_thrust="${max_t}" direction="1"/>
+  <xacro:add_rotor_and_thrust id="4" parent="thruster_3" min_thrust="${min_t}" max_thrust="${max_t}" direction="-1"/>
+  <xacro:add_rotor_and_thrust id="5" parent="thruster_4" min_thrust="${min_t}" max_thrust="${max_t}" direction="1"/>
+  <xacro:add_rotor_and_thrust id="6" parent="thruster_5" min_thrust="${min_t}" max_thrust="${max_t}" direction="-1"/>
+  <xacro:add_rotor_and_thrust id="7" parent="thruster_6" min_thrust="${min_t}" max_thrust="${max_t}" direction="1"/>
+  <xacro:add_rotor_and_thrust id="8" parent="thruster_7" min_thrust="${min_t}" max_thrust="${max_t}" direction="-1"/>
 </robot>

Commit message: fix urdf thruster->booster

File: robots/uuv_d/robots/quad/default_mode_201907/robot.urdf.xacro (robot description, xacro)
@@ -80,5 +80,5 @@
     </transmission>
   </xacro:macro>
-  <link name="thruster_0">
+  <link name="booster_0">
     <inertial>
       <origin xyz="-0.014292 -0.0143 0.017717" rpy="0.0 -0.0 0.0"/>
@@ -100,5 +100,5 @@
     </collision>
   </link>
-  <link name="thruster_1">
+  <link name="booster_1">
     <inertial>
       <origin xyz="0.0143 -0.014292 0.017717" rpy="0.0 -0.0 0.0"/>
@@ -120,5 +120,5 @@
     </collision>
   </link>
-  <link name="thruster_2">
+  <link name="booster_2">
     <inertial>
       <origin xyz="-0.0143 0.014292 0.017717" rpy="0.0 -0.0 0.0"/>
@@ -140,5 +140,5 @@
     </collision>
   </link>
-  <link name="thruster_3">
+  <link name="booster_3">
     <inertial>
       <origin xyz="0.014292 0.0143 0.017717" rpy="0.0 -0.0 0.0"/>
@@ -160,5 +160,5 @@
     </collision>
   </link>
-  <link name="thruster_4">
+  <link name="booster_4">
     <inertial>
       <origin xyz="0.014292 -0.0143 -0.017717" rpy="0.0 -0.0 0.0"/>
@@ -180,5 +180,5 @@
     </collision>
   </link>
-  <link name="thruster_5">
+  <link name="booster_5">
     <inertial>
       <origin xyz="0.204989569717696 -0.0142922441746005 -0.0177167300549156" rpy="0.0 -0.0 0.0"/>
@@ -200,5 +200,5 @@
     </collision>
   </link>
-  <link name="thruster_6">
+  <link name="booster_6">
     <inertial>
       <origin xyz="0.205 0.0143 -0.017717" rpy="0.0 -0.0 0.0"/>
@@ -220,5 +220,5 @@
     </collision>
   </link>
-  <link name="thruster_7">
+  <link name="booster_7">
     <inertial>
       <origin xyz="-0.014292 0.0143 -0.017717" rpy="0.0 -0.0 0.0"/>
@@ -240,57 +240,57 @@
     </collision>
   </link>
-  <joint name="thruster_0" type="continuous">
-    <limit effort="0.0" velocity="0.0"/>
-    <parent link="base_link"/>
-    <child link="thruster_0"/>
+  <joint name="booster_0" type="continuous">
+    <limit effort="0.0" velocity="0.0"/>
+    <parent link="base_link"/>
+    <child link="booster_0"/>
     <axis xyz="-0.49999886 -0.49999886  0.70710839"/>
     <origin xyz="0.10964 0.096917 -0.39159" rpy="0.0 -0.0 0.0"/>
   </joint>
-  <joint name="thruster_1" type="continuous">
-    <limit effort="0.0" velocity="0.0"/>
-    <parent link="base_link"/>
-    <child link="thruster_1"/>
+  <joint name="booster_1" type="continuous">
+    <limit effort="0.0" velocity="0.0"/>
+    <parent link="base_link"/>
+    <child link="booster_1"/>
     <axis xyz=" 0.49999886 -0.49999886  0.70710839"/>
     <origin xyz="-0.10964 0.096917 -0.39159" rpy="0.0 -0.0 0.0"/>
   </joint>
-  <joint name="thruster_2" type="continuous">
-    <limit effort="0.0" velocity="0.0"/>
-    <parent link="base_link"/>
-    <child link="thruster_2"/>
+  <joint name="booster_2" type="continuous">
+    <limit effort="0.0" velocity="0.0"/>
+    <parent link="base_link"/>
+    <child link="booster_2"/>
     <axis xyz="-0.49999886  0.49999886  0.70710839"/>
     <origin xyz="0.10964 -0.096917 -0.39159" rpy="0.0 -0.0 0.0"/>
   </joint>
-  <joint name="thruster_3" type="continuous">
-    <limit effort="0.0" velocity="0.0"/>
-    <parent link="base_link"/>
-    <child link="thruster_3"/>
+  <joint name="booster_3" type="continuous">
+    <limit effort="0.0" velocity="0.0"/>
+    <parent link="base_link"/>
+    <child link="booster_3"/>
     <axis xyz="0.49999886 0.49999886 0.70710839"/>
     <origin xyz="-0.10964 -0.096917 -0.39159" rpy="0.0 -0.0 0.0"/>
   </joint>
-  <joint name="thruster_4" type="continuous">
-    <limit effort="0.0" velocity="0.0"/>
-    <parent link="base_link"/>
-    <child link="thruster_4"/>
+  <joint name="booster_4" type="continuous">
+    <limit effort="0.0" velocity="0.0"/>
+    <parent link="base_link"/>
+    <child link="booster_4"/>
     <axis xyz=" 0.49999886 -0.49999886 -0.70710839"/>
     <origin xyz="-0.10964 0.096917 -0.040214" rpy="0.0 -0.0 0.0"/>
   </joint>
-  <joint name="thruster_5" type="continuous">
-    <limit effort="0.0" velocity="0.0"/>
-    <parent link="base_link"/>
-    <child link="thruster_5"/>
+  <joint name="booster_5" type="continuous">
+    <limit effort="0.0" velocity="0.0"/>
+    <parent link="base_link"/>
+    <child link="booster_5"/>
     <axis xyz="-0.49999886 -0.49999886 -0.70710839"/>
     <origin xyz="-0.10964 0.096917 -0.040214" rpy="0.0 -0.0 0.0"/>
   </joint>
-  <joint name="thruster_6" type="continuous">
-    <limit effort="0.0" velocity="0.0"/>
-    <parent link="base_link"/>
-    <child link="thruster_6"/>
+  <joint name="booster_6" type="continuous">
+    <limit effort="0.0" velocity="0.0"/>
+    <parent link="base_link"/>
+    <child link="booster_6"/>
     <axis xyz=" 0.49999886  0.49999886 -0.70710839"/>
     <origin xyz="-0.10964 -0.096917 -0.040214" rpy="0.0 -0.0 0.0"/>
   </joint>
-  <joint name="thruster_7" type="continuous">
-    <limit effort="0.0" velocity="0.0"/>
-    <parent link="base_link"/>
-    <child link="thruster_7"/>
+  <joint name="booster_7" type="continuous">
+    <limit effort="0.0" velocity="0.0"/>
+    <parent link="base_link"/>
+    <child link="booster_7"/>
     <axis xyz="-0.49999886  0.49999886 -0.70710839"/>
     <origin xyz="0.10964 -0.096917 -0.040214" rpy="0.0 -0.0 0.0"/>
@@ -325,11 +325,11 @@
   <xacro:property name="min_t" value="-20.0" />
   <xacro:property name="max_t" value="20.0" />
-  <xacro:add_rotor_and_thrust id="1" parent="thruster_0" min_thrust="${min_t}" max_thrust="${max_t}" direction="1"/>
-  <xacro:add_rotor_and_thrust id="2" parent="thruster_1" min_thrust="${min_t}" max_thrust="${max_t}" direction="-1"/>
-  <xacro:add_rotor_and_thrust id="3" parent="thruster_2" min_thrust="${min_t}" max_thrust="${max_t}" direction="1"/>
-  <xacro:add_rotor_and_thrust id="4" parent="thruster_3" min_thrust="${min_t}" max_thrust="${max_t}" direction="-1"/>
-  <xacro:add_rotor_and_thrust id="5" parent="thruster_4" min_thrust="${min_t}" max_thrust="${max_t}" direction="1"/>
-  <xacro:add_rotor_and_thrust id="6" parent="thruster_5" min_thrust="${min_t}" max_thrust="${max_t}" direction="-1"/>
-  <xacro:add_rotor_and_thrust id="7" parent="thruster_6" min_thrust="${min_t}" max_thrust="${max_t}" direction="1"/>
-  <xacro:add_rotor_and_thrust id="8" parent="thruster_7" min_thrust="${min_t}" max_thrust="${max_t}" direction="-1"/>
+  <xacro:add_rotor_and_thrust id="1" parent="booster_0" min_thrust="${min_t}" max_thrust="${max_t}" direction="1"/>
+  <xacro:add_rotor_and_thrust id="2" parent="booster_1" min_thrust="${min_t}" max_thrust="${max_t}" direction="-1"/>
+  <xacro:add_rotor_and_thrust id="3" parent="booster_2" min_thrust="${min_t}" max_thrust="${max_t}" direction="1"/>
+  <xacro:add_rotor_and_thrust id="4" parent="booster_3" min_thrust="${min_t}" max_thrust="${max_t}" direction="-1"/>
+  <xacro:add_rotor_and_thrust id="5" parent="booster_4" min_thrust="${min_t}" max_thrust="${max_t}" direction="1"/>
+  <xacro:add_rotor_and_thrust id="6" parent="booster_5" min_thrust="${min_t}" max_thrust="${max_t}" direction="-1"/>
+  <xacro:add_rotor_and_thrust id="7" parent="booster_6" min_thrust="${min_t}" max_thrust="${max_t}" direction="1"/>
+  <xacro:add_rotor_and_thrust id="8" parent="booster_7" min_thrust="${min_t}" max_thrust="${max_t}" direction="-1"/>
 </robot>
