Commit message: change debug setting

File: robots/uuv_d/robots/quad/default_mode_201907/robot.urdf.xacro (robot description, xacro)
@@ -20,7 +20,7 @@
   <link name="base_link">
     <inertial>
-      <origin xyz="-4.2558171182705e-06 1.1225964209836e-05 -0.215899999907217" rpy="0.0 -0.0 0.0"/>
-      <mass value="1.90859968353568"/>
-      <inertia ixx="0.0162419971330382" ixy="4.56271680930171e-05" ixz="-4.69435220066161e-11" iyy="0.0168438204899763" iyz="-1.78508266758785e-11" izz="0.0050226778184606"/>
+      <origin xyz="-4.2558e-06 1.1226e-05 -0.2159" rpy="0.0 -0.0 0.0"/>
+      <mass value="1.9086"/>
+      <inertia ixx="0.016242" ixy="4.5627e-05" ixz="-4.7038e-11" iyy="0.016844" iyz="-1.7865e-11" izz="0.0050227"/>
     </inertial>
     <visual>
@@ -38,47 +38,5 @@
     </collision>
   </link>
-  <link name="fc">
-      <inertial>
-        <origin xyz="0 0 0" rpy="0 0 0"/>
-        <mass value="0.00001"/>
-        <inertia
-            ixx="0.000001" ixy="0.0" ixz="0.0"
-            iyy="0.000001" iyz="0.0"
-            izz="0.000001"/>
-      </inertial>
-    </link>
-    <joint name="fc_joint" type="fixed">
-      <child link="fc"/>
-      <parent link="base_link"/>
-      <origin rpy="0 0 0" xyz="0 0 0"/>
-      <axis xyz="0 0 1"/>
-    </joint>
-  <xacro:macro name="add_rotor_and_thrust" params="id parent min_thrust max_thrust direction">
-    <link name="thrust${id}">
-      <inertial>
-        <origin xyz="0 0 0" rpy="0 0 0"/>
-        <mass value="0.0001"/>
-        <inertia ixx="0.00001" ixy="0.0" ixz="0.0" iyy="0.00001" iyz="0.0" izz="0.00002"/>
-      </inertial>
-    </link>
-    <joint name="rotor${id}" type="continuous">
-      <limit effort="100.0" lower="${min_thrust}" upper="${max_thrust}" velocity="50.0"/>
-      <parent link="${parent}"/>
-      <child link="thrust${id}"/>
-      <origin xyz="0 0 0" rpy="0 0 0"/>
-      <axis xyz="0 0 ${direction}"/>
-    </joint>
-    <transmission name="rotor_tran${id}">
-      <type>transmission_interface/SimpleTransmission</type>
-      <joint name="rotor${id}">
-        <hardwareInterface>RotorInterface</hardwareInterface>
-      </joint>
-      <actuator name="actuator_rotor_${id}">
-        <hardwareInterface>RotorInterface</hardwareInterface>
-        <mechanicalReduction>1</mechanicalReduction>
-      </actuator>
-    </transmission>
-  </xacro:macro>
-  <link name="booster_0">
+  <link name="t1">
     <inertial>
       <origin xyz="-0.014292 -0.0143 0.017717" rpy="0.0 -0.0 0.0"/>
@@ -88,5 +46,5 @@
     <visual>
       <geometry>
-        <mesh filename="package://uuv_d/urdf/mesh/proto_type/meshes/thruster_0.dae"/>
+        <mesh filename="package://uuv_d/urdf/mesh/proto_type/meshes/t1.dae"/>
       </geometry>
       <material name="__unnamed_material_2"/>
@@ -95,10 +53,30 @@
     <collision>
       <geometry>
-        <mesh filename="package://uuv_d/urdf/mesh/proto_type/meshes/thruster_0.stl"/>
-      </geometry>
-      <origin xyz="0.0 0.0 0.0" rpy="0.0 -0.0 0.0"/>
-    </collision>
-  </link>
-  <link name="booster_1">
+        <mesh filename="package://uuv_d/urdf/mesh/proto_type/meshes/t1.stl"/>
+      </geometry>
+      <origin xyz="0.0 0.0 0.0" rpy="0.0 -0.0 0.0"/>
+    </collision>
+  </link>
+  <link name="thrust1">
+    <inertial>
+      <origin xyz="3.3307e-15 3.525e-15 -0.001" rpy="0.0 -0.0 0.0"/>
+      <mass value="0.0028342"/>
+      <inertia ixx="6.5251e-07" ixy="-1.0853e-21" ixz="1.8529e-22" iyy="6.5251e-07" iyz="-3.7058e-22" izz="1.3031e-06"/>
+    </inertial>
+    <visual>
+      <geometry>
+        <mesh filename="package://uuv_d/urdf/mesh/proto_type/meshes/thrust1.dae"/>
+      </geometry>
+      <material name="__unnamed_material_3"/>
+      <origin xyz="0.0 0.0 0.0" rpy="0.0 -0.0 0.0"/>
+    </visual>
+    <collision>
+      <geometry>
+        <mesh filename="package://uuv_d/urdf/mesh/proto_type/meshes/thrust1.stl"/>
+      </geometry>
+      <origin xyz="0.0 0.0 0.0" rpy="0.0 -0.0 0.0"/>
+    </collision>
+  </link>
+  <link name="t2">
     <inertial>
       <origin xyz="0.0143 -0.014292 0.017717" rpy="0.0 -0.0 0.0"/>
@@ -108,17 +86,37 @@
     <visual>
       <geometry>
-        <mesh filename="package://uuv_d/urdf/mesh/proto_type/meshes/thruster_1.dae"/>
-      </geometry>
-      <material name="__unnamed_material_3"/>
-      <origin xyz="0.0 0.0 0.0" rpy="0.0 -0.0 0.0"/>
-    </visual>
-    <collision>
-      <geometry>
-        <mesh filename="package://uuv_d/urdf/mesh/proto_type/meshes/thruster_1.stl"/>
-      </geometry>
-      <origin xyz="0.0 0.0 0.0" rpy="0.0 -0.0 0.0"/>
-    </collision>
-  </link>
-  <link name="booster_2">
+        <mesh filename="package://uuv_d/urdf/mesh/proto_type/meshes/t2.dae"/>
+      </geometry>
+      <material name="__unnamed_material_4"/>
+      <origin xyz="0.0 0.0 0.0" rpy="0.0 -0.0 0.0"/>
+    </visual>
+    <collision>
+      <geometry>
+        <mesh filename="package://uuv_d/urdf/mesh/proto_type/meshes/t2.stl"/>
+      </geometry>
+      <origin xyz="0.0 0.0 0.0" rpy="0.0 -0.0 0.0"/>
+    </collision>
+  </link>
+  <link name="thrust2">
+    <inertial>
+      <origin xyz="2.2204e-16 8.3267e-17 0.001" rpy="0.0 -0.0 0.0"/>
+      <mass value="0.0028342"/>
+      <inertia ixx="6.5251e-07" ixy="-3.5867e-21" ixz="-2.647e-22" iyy="6.5251e-07" iyz="-1.3235e-22" izz="1.3031e-06"/>
+    </inertial>
+    <visual>
+      <geometry>
+        <mesh filename="package://uuv_d/urdf/mesh/proto_type/meshes/thrust2.dae"/>
+      </geometry>
+      <material name="__unnamed_material_5"/>
+      <origin xyz="0.0 0.0 0.0" rpy="0.0 -0.0 0.0"/>
+    </visual>
+    <collision>
+      <geometry>
+        <mesh filename="package://uuv_d/urdf/mesh/proto_type/meshes/thrust2.stl"/>
+      </geometry>
+      <origin xyz="0.0 0.0 0.0" rpy="0.0 -0.0 0.0"/>
+    </collision>
+  </link>
+  <link name="t3">
     <inertial>
       <origin xyz="-0.0143 0.014292 0.017717" rpy="0.0 -0.0 0.0"/>
@@ -128,17 +126,37 @@
     <visual>
       <geometry>
-        <mesh filename="package://uuv_d/urdf/mesh/proto_type/meshes/thruster_2.dae"/>
-      </geometry>
-      <material name="__unnamed_material_4"/>
-      <origin xyz="0.0 0.0 0.0" rpy="0.0 -0.0 0.0"/>
-    </visual>
-    <collision>
-      <geometry>
-        <mesh filename="package://uuv_d/urdf/mesh/proto_type/meshes/thruster_2.stl"/>
-      </geometry>
-      <origin xyz="0.0 0.0 0.0" rpy="0.0 -0.0 0.0"/>
-    </collision>
-  </link>
-  <link name="booster_3">
+        <mesh filename="package://uuv_d/urdf/mesh/proto_type/meshes/t3.dae"/>
+      </geometry>
+      <material name="__unnamed_material_6"/>
+      <origin xyz="0.0 0.0 0.0" rpy="0.0 -0.0 0.0"/>
+    </visual>
+    <collision>
+      <geometry>
+        <mesh filename="package://uuv_d/urdf/mesh/proto_type/meshes/t3.stl"/>
+      </geometry>
+      <origin xyz="0.0 0.0 0.0" rpy="0.0 -0.0 0.0"/>
+    </collision>
+  </link>
+  <link name="thrust3">
+    <inertial>
+      <origin xyz="-2.22044604925031e-16 4.9960036108132e-16 0.00100000000000011" rpy="0.0 -0.0 0.0"/>
+      <mass value="0.00283424938765202"/>
+      <inertia ixx="6.52506444943004e-07" ixy="5.12190235292835e-21" ixz="6.35274710440725e-22" iyy="6.52506444943007e-07" iyz="-2.64697796016969e-23" izz="1.30312339029424e-06"/>
+    </inertial>
+    <visual>
+      <geometry>
+        <mesh filename="package://uuv_d/urdf/mesh/proto_type/meshes/thrust3.dae"/>
+      </geometry>
+      <material name="__unnamed_material_7"/>
+      <origin xyz="0.0 0.0 0.0" rpy="0.0 -0.0 0.0"/>
+    </visual>
+    <collision>
+      <geometry>
+        <mesh filename="package://uuv_d/urdf/mesh/proto_type/meshes/thrust3.stl"/>
+      </geometry>
+      <origin xyz="0.0 0.0 0.0" rpy="0.0 -0.0 0.0"/>
+    </collision>
+  </link>
+  <link name="t4">
     <inertial>
       <origin xyz="0.014292 0.0143 0.017717" rpy="0.0 -0.0 0.0"/>
@@ -148,17 +166,37 @@
     <visual>
       <geometry>
-        <mesh filename="package://uuv_d/urdf/mesh/proto_type/meshes/thruster_3.dae"/>
-      </geometry>
-      <material name="__unnamed_material_5"/>
-      <origin xyz="0.0 0.0 0.0" rpy="0.0 -0.0 0.0"/>
-    </visual>
-    <collision>
-      <geometry>
-        <mesh filename="package://uuv_d/urdf/mesh/proto_type/meshes/thruster_3.stl"/>
-      </geometry>
-      <origin xyz="0.0 0.0 0.0" rpy="0.0 -0.0 0.0"/>
-    </collision>
-  </link>
-  <link name="booster_4">
+        <mesh filename="package://uuv_d/urdf/mesh/proto_type/meshes/t4.dae"/>
+      </geometry>
+      <material name="__unnamed_material_8"/>
+      <origin xyz="0.0 0.0 0.0" rpy="0.0 -0.0 0.0"/>
+    </visual>
+    <collision>
+      <geometry>
+        <mesh filename="package://uuv_d/urdf/mesh/proto_type/meshes/t4.stl"/>
+      </geometry>
+      <origin xyz="0.0 0.0 0.0" rpy="0.0 -0.0 0.0"/>
+    </collision>
+  </link>
+  <link name="thrust4">
+    <inertial>
+      <origin xyz="-3.33066907387547e-16 -2.4008572907519e-15 0.000999999999999834" rpy="0.0 -0.0 0.0"/>
+      <mass value="0.00283424938765202"/>
+      <inertia ixx="6.52506444943007e-07" ixy="1.87935435172048e-21" ixz="-1.19114008207636e-22" iyy="6.52506444943005e-07" iyz="3.97046694025453e-22" izz="1.30312339029424e-06"/>
+    </inertial>
+    <visual>
+      <geometry>
+        <mesh filename="package://uuv_d/urdf/mesh/proto_type/meshes/thrust4.dae"/>
+      </geometry>
+      <material name="__unnamed_material_9"/>
+      <origin xyz="0.0 0.0 0.0" rpy="0.0 -0.0 0.0"/>
+    </visual>
+    <collision>
+      <geometry>
+        <mesh filename="package://uuv_d/urdf/mesh/proto_type/meshes/thrust4.stl"/>
+      </geometry>
+      <origin xyz="0.0 0.0 0.0" rpy="0.0 -0.0 0.0"/>
+    </collision>
+  </link>
+  <link name="t5">
     <inertial>
       <origin xyz="0.014292 -0.0143 -0.017717" rpy="0.0 -0.0 0.0"/>
@@ -168,134 +206,259 @@
     <visual>
       <geometry>
-        <mesh filename="package://uuv_d/urdf/mesh/proto_type/meshes/thruster_4.dae"/>
-      </geometry>
-      <material name="__unnamed_material_6"/>
-      <origin xyz="0.0 0.0 0.0" rpy="0.0 -0.0 0.0"/>
-    </visual>
-    <collision>
-      <geometry>
-        <mesh filename="package://uuv_d/urdf/mesh/proto_type/meshes/thruster_4.stl"/>
-      </geometry>
-      <origin xyz="0.0 0.0 0.0" rpy="0.0 -0.0 0.0"/>
-    </collision>
-  </link>
-  <link name="booster_5">
-    <inertial>
-      <origin xyz="0.204989569717696 -0.0142922441746005 -0.0177167300549156" rpy="0.0 -0.0 0.0"/>
-      <mass value="0.0993924873705004"/>
-      <inertia ixx="7.91363117744372e-05" ixy="6.13947103624969e-08" ixz="3.80401853538402e-06" iyy="7.91541243411415e-05" iyz="3.781720562086e-06" izz="7.67197078219348e-05"/>
-    </inertial>
-    <visual>
-      <geometry>
-        <mesh filename="package://uuv_d/urdf/mesh/proto_type/meshes/thruster_5.dae"/>
-      </geometry>
-      <material name="__unnamed_material_7"/>
-      <origin xyz="0.0 0.0 0.0" rpy="0.0 -0.0 0.0"/>
-    </visual>
-    <collision>
-      <geometry>
-        <mesh filename="package://uuv_d/urdf/mesh/proto_type/meshes/thruster_5.stl"/>
-      </geometry>
-      <origin xyz="0.0 0.0 0.0" rpy="0.0 -0.0 0.0"/>
-    </collision>
-  </link>
-  <link name="booster_6">
-    <inertial>
-      <origin xyz="0.205 0.0143 -0.017717" rpy="0.0 -0.0 0.0"/>
-      <mass value="0.099392"/>
-      <inertia ixx="7.9154e-05" ixy="-6.1395e-08" ixz="3.7817e-06" iyy="7.9136e-05" iyz="-3.804e-06" izz="7.672e-05"/>
-    </inertial>
-    <visual>
-      <geometry>
-        <mesh filename="package://uuv_d/urdf/mesh/proto_type/meshes/thruster_6.dae"/>
-      </geometry>
-      <material name="__unnamed_material_8"/>
-      <origin xyz="0.0 0.0 0.0" rpy="0.0 -0.0 0.0"/>
-    </visual>
-    <collision>
-      <geometry>
-        <mesh filename="package://uuv_d/urdf/mesh/proto_type/meshes/thruster_6.stl"/>
-      </geometry>
-      <origin xyz="0.0 0.0 0.0" rpy="0.0 -0.0 0.0"/>
-    </collision>
-  </link>
-  <link name="booster_7">
-    <inertial>
-      <origin xyz="-0.014292 0.0143 -0.017717" rpy="0.0 -0.0 0.0"/>
-      <mass value="0.099392"/>
-      <inertia ixx="7.9154e-05" ixy="-6.1395e-08" ixz="3.7817e-06" iyy="7.9136e-05" iyz="-3.804e-06" izz="7.672e-05"/>
-    </inertial>
-    <visual>
-      <geometry>
-        <mesh filename="package://uuv_d/urdf/mesh/proto_type/meshes/thruster_7.dae"/>
-      </geometry>
-      <material name="__unnamed_material_9"/>
-      <origin xyz="0.0 0.0 0.0" rpy="0.0 -0.0 0.0"/>
-    </visual>
-    <collision>
-      <geometry>
-        <mesh filename="package://uuv_d/urdf/mesh/proto_type/meshes/thruster_7.stl"/>
-      </geometry>
-      <origin xyz="0.0 0.0 0.0" rpy="0.0 -0.0 0.0"/>
-    </collision>
-  </link>
-  <joint name="booster_0" type="continuous">
-    <limit effort="0.0" velocity="0.0"/>
-    <parent link="base_link"/>
-    <child link="booster_0"/>
-    <axis xyz="-0.49999886 -0.49999886  0.70710839"/>
+        <mesh filename="package://uuv_d/urdf/mesh/proto_type/meshes/t5.dae"/>
+      </geometry>
+      <material name="__unnamed_material_10"/>
+      <origin xyz="0.0 0.0 0.0" rpy="0.0 -0.0 0.0"/>
+    </visual>
+    <collision>
+      <geometry>
+        <mesh filename="package://uuv_d/urdf/mesh/proto_type/meshes/t5.stl"/>
+      </geometry>
+      <origin xyz="0.0 0.0 0.0" rpy="0.0 -0.0 0.0"/>
+    </collision>
+  </link>
+  <link name="thrust5"/>
+  <link name="t6">
+    <inertial>
+      <origin xyz="-0.0143000152087087 -0.0142922441739046 -0.0177167300533436" rpy="0.0 -0.0 0.0"/>
+      <mass value="0.0993924873705024"/>
+      <inertia ixx="7.91363117744376e-05" ixy="6.13947103617769e-08" ixz="3.80401853538391e-06" iyy="7.91541243411415e-05" iyz="3.78172056208575e-06" izz="7.67197078219357e-05"/>
+    </inertial>
+    <visual>
+      <geometry>
+        <mesh filename="package://uuv_d/urdf/mesh/proto_type/meshes/t6.dae"/>
+      </geometry>
+      <material name="__unnamed_material_11"/>
+      <origin xyz="0.0 0.0 0.0" rpy="0.0 -0.0 0.0"/>
+    </visual>
+    <collision>
+      <geometry>
+        <mesh filename="package://uuv_d/urdf/mesh/proto_type/meshes/t6.stl"/>
+      </geometry>
+      <origin xyz="0.0 0.0 0.0" rpy="0.0 -0.0 0.0"/>
+    </collision>
+  </link>
+  <link name="thrust6">
+    <inertial>
+      <origin xyz="4.05231403988182e-14 2.86715096109447e-14 0.0010000000000413" rpy="0.0 -0.0 0.0"/>
+      <mass value="0.00283424938765202"/>
+      <inertia ixx="6.52506444942999e-07" ixy="-6.07481441858944e-21" ixz="-1.98523347012727e-22" iyy="6.52506444943014e-07" iyz="-2.38228016415272e-22" izz="1.30312339029425e-06"/>
+    </inertial>
+    <visual>
+      <geometry>
+        <mesh filename="package://uuv_d/urdf/mesh/proto_type/meshes/thrust6.dae"/>
+      </geometry>
+      <material name="__unnamed_material_12"/>
+      <origin xyz="0.0 0.0 0.0" rpy="0.0 -0.0 0.0"/>
+    </visual>
+    <collision>
+      <geometry>
+        <mesh filename="package://uuv_d/urdf/mesh/proto_type/meshes/thrust6.stl"/>
+      </geometry>
+      <origin xyz="0.0 0.0 0.0" rpy="0.0 -0.0 0.0"/>
+    </collision>
+  </link>
+  <link name="t7">
+    <inertial>
+      <origin xyz="0.204997340751786 0.0143000152101347 -0.0177167300564932" rpy="0.0 -0.0 0.0"/>
+      <mass value="0.0993924873705016"/>
+      <inertia ixx="7.91541243411232e-05" ixy="-6.13947103569633e-08" ixz="3.78172056208173e-06" iyy="7.91363117744202e-05" iyz="-3.80401853537825e-06" izz="7.67197078219122e-05"/>
+    </inertial>
+    <visual>
+      <geometry>
+        <mesh filename="package://uuv_d/urdf/mesh/proto_type/meshes/t7.dae"/>
+      </geometry>
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