Commit message: update urdf

File: robots/uuv_d/robots/quad/default_mode_201907/robot.urdf.xacro (robot description, xacro)
@@ -23,6 +23,5 @@
     <inertial>
       <origin xyz="-4.2558e-06 1.1226e-05 -0.2159" rpy="0.0 -0.0 0.0"/>
-      <!-- <mass value="1.9086"/> -->
-      <mass value="0.9086"/>
+      <mass value="1.9086"/>
       <inertia ixx="0.016242" ixy="4.5627e-05" ixz="-4.7038e-11" iyy="0.016844" iyz="-1.7865e-11" izz="0.0050227"/>
     </inertial>
@@ -49,5 +48,5 @@
     <visual>
       <geometry>
-        <mesh filename="package://uuv_d/urdf/mesh/proto_type/meshes/t1.dae"/>
+        <mesh filename="package://uuv_d/urdf/mesh/proto_type/meshes/t1.STL"/>
       </geometry>
       <material name="__unnamed_material_2"/>
@@ -63,11 +62,11 @@
   <link name="thrust1">
     <inertial>
-      <origin xyz="3.3307e-15 3.525e-15 -0.001" rpy="0.0 -0.0 0.0"/>
-      <mass value="0.0028342"/>
-      <inertia ixx="6.5251e-07" ixy="-1.0853e-21" ixz="1.8529e-22" iyy="6.5251e-07" iyz="-3.7058e-22" izz="1.3031e-06"/>
-    </inertial>
-    <visual>
-      <geometry>
-        <mesh filename="package://uuv_d/urdf/mesh/proto_type/meshes/thrust1.dae"/>
+      <origin xyz="0 0 0" rpy="0.0 0.0 0.0"/>
+      <mass value="0.00001"/>
+      <inertia ixx="0.00001" ixy="0.0" ixz="0.0" iyy="0.00001" iyz="0" izz="0.00001"/>
+    </inertial>
+    <visual>
+      <geometry>
+        <mesh filename="package://uuv_d/urdf/mesh/proto_type/meshes/thrust1.STL"/>
       </geometry>
       <material name="__unnamed_material_3"/>
@@ -89,5 +88,5 @@
     <visual>
       <geometry>
-        <mesh filename="package://uuv_d/urdf/mesh/proto_type/meshes/t2.dae"/>
+        <mesh filename="package://uuv_d/urdf/mesh/proto_type/meshes/t2.STL"/>
       </geometry>
       <material name="__unnamed_material_4"/>
@@ -103,11 +102,11 @@
   <link name="thrust2">
     <inertial>
-      <origin xyz="2.2204e-16 8.3267e-17 0.001" rpy="0.0 -0.0 0.0"/>
-      <mass value="0.0028342"/>
-      <inertia ixx="6.5251e-07" ixy="-3.5867e-21" ixz="-2.647e-22" iyy="6.5251e-07" iyz="-1.3235e-22" izz="1.3031e-06"/>
-    </inertial>
-    <visual>
-      <geometry>
-        <mesh filename="package://uuv_d/urdf/mesh/proto_type/meshes/thrust2.dae"/>
+      <origin xyz="0 0 0" rpy="0.0 0.0 0.0"/>
+      <mass value="0.00001"/>
+      <inertia ixx="0.00001" ixy="0.0" ixz="0.0" iyy="0.00001" iyz="0" izz="0.00001"/>
+    </inertial>
+    <visual>
+      <geometry>
+        <mesh filename="package://uuv_d/urdf/mesh/proto_type/meshes/thrust2.STL"/>
       </geometry>
       <material name="__unnamed_material_5"/>
@@ -129,5 +128,5 @@
     <visual>
       <geometry>
-        <mesh filename="package://uuv_d/urdf/mesh/proto_type/meshes/t3.dae"/>
+        <mesh filename="package://uuv_d/urdf/mesh/proto_type/meshes/t3.STL"/>
       </geometry>
       <material name="__unnamed_material_6"/>
@@ -143,11 +142,11 @@
   <link name="thrust3">
     <inertial>
-      <origin xyz="-2.22044604925031e-16 4.9960036108132e-16 0.00100000000000011" rpy="0.0 -0.0 0.0"/>
-      <mass value="0.00283424938765202"/>
-      <inertia ixx="6.52506444943004e-07" ixy="5.12190235292835e-21" ixz="6.35274710440725e-22" iyy="6.52506444943007e-07" iyz="-2.64697796016969e-23" izz="1.30312339029424e-06"/>
-    </inertial>
-    <visual>
-      <geometry>
-        <mesh filename="package://uuv_d/urdf/mesh/proto_type/meshes/thrust3.dae"/>
+      <origin xyz="0 0 0" rpy="0.0 0.0 0.0"/>
+      <mass value="0.00001"/>
+      <inertia ixx="0.00001" ixy="0.0" ixz="0.0" iyy="0.00001" iyz="0" izz="0.00001"/>
+    </inertial>
+    <visual>
+      <geometry>
+        <mesh filename="package://uuv_d/urdf/mesh/proto_type/meshes/thrust3.STL"/>
       </geometry>
       <material name="__unnamed_material_7"/>
@@ -169,5 +168,5 @@
     <visual>
       <geometry>
-        <mesh filename="package://uuv_d/urdf/mesh/proto_type/meshes/t4.dae"/>
+        <mesh filename="package://uuv_d/urdf/mesh/proto_type/meshes/t4.STL"/>
       </geometry>
       <material name="__unnamed_material_8"/>
@@ -183,11 +182,11 @@
   <link name="thrust4">
     <inertial>
-      <origin xyz="-3.33066907387547e-16 -2.4008572907519e-15 0.000999999999999834" rpy="0.0 -0.0 0.0"/>
-      <mass value="0.00283424938765202"/>
-      <inertia ixx="6.52506444943007e-07" ixy="1.87935435172048e-21" ixz="-1.19114008207636e-22" iyy="6.52506444943005e-07" iyz="3.97046694025453e-22" izz="1.30312339029424e-06"/>
-    </inertial>
-    <visual>
-      <geometry>
-        <mesh filename="package://uuv_d/urdf/mesh/proto_type/meshes/thrust4.dae"/>
+      <origin xyz="0 0 0" rpy="0.0 0.0 0.0"/>
+      <mass value="0.00001"/>
+      <inertia ixx="0.00001" ixy="0.0" ixz="0.0" iyy="0.00001" iyz="0" izz="0.00001"/>
+    </inertial>
+    <visual>
+      <geometry>
+        <mesh filename="package://uuv_d/urdf/mesh/proto_type/meshes/thrust4.STL"/>
       </geometry>
       <material name="__unnamed_material_9"/>
@@ -209,5 +208,5 @@
     <visual>
       <geometry>
-        <mesh filename="package://uuv_d/urdf/mesh/proto_type/meshes/t5.dae"/>
+        <mesh filename="package://uuv_d/urdf/mesh/proto_type/meshes/t5.STL"/>
       </geometry>
       <material name="__unnamed_material_10"/>
@@ -223,7 +222,7 @@
   <link name="thrust5">
     <inertial>
-      <origin xyz="0 0 0.001" rpy="0 0 0"/>
-      <mass value="0.0028342"/>
-      <inertia ixx="6.5251e-07" ixy="0.0" ixz="0.0" iyy="6.5251e-07" iyz="0.0" izz="1.3031e-06"/>
+      <origin xyz="0 0 0" rpy="0.0 0.0 0.0"/>
+      <mass value="0.00001"/>
+      <inertia ixx="0.00001" ixy="0.0" ixz="0.0" iyy="0.00001" iyz="0" izz="0.00001"/>
     </inertial>
   </link>
@@ -236,5 +235,5 @@
     <visual>
       <geometry>
-        <mesh filename="package://uuv_d/urdf/mesh/proto_type/meshes/t6.dae"/>
+        <mesh filename="package://uuv_d/urdf/mesh/proto_type/meshes/t6.STL"/>
       </geometry>
       <material name="__unnamed_material_11"/>
@@ -250,11 +249,11 @@
   <link name="thrust6">
     <inertial>
-      <origin xyz="4.05231403988182e-14 2.86715096109447e-14 0.0010000000000413" rpy="0.0 -0.0 0.0"/>
-      <mass value="0.00283424938765202"/>
-      <inertia ixx="6.52506444942999e-07" ixy="-6.07481441858944e-21" ixz="-1.98523347012727e-22" iyy="6.52506444943014e-07" iyz="-2.38228016415272e-22" izz="1.30312339029425e-06"/>
-    </inertial>
-    <visual>
-      <geometry>
-        <mesh filename="package://uuv_d/urdf/mesh/proto_type/meshes/thrust6.dae"/>
+      <origin xyz="0 0 0" rpy="0.0 0.0 0.0"/>
+      <mass value="0.00001"/>
+      <inertia ixx="0.00001" ixy="0.0" ixz="0.0" iyy="0.00001" iyz="0" izz="0.00001"/>
+    </inertial>
+    <visual>
+      <geometry>
+        <mesh filename="package://uuv_d/urdf/mesh/proto_type/meshes/thrust6.STL"/>
       </geometry>
       <material name="__unnamed_material_12"/>
@@ -276,5 +275,5 @@
     <visual>
       <geometry>
-        <mesh filename="package://uuv_d/urdf/mesh/proto_type/meshes/t7.dae"/>
+        <mesh filename="package://uuv_d/urdf/mesh/proto_type/meshes/t7.STL"/>
       </geometry>
       <material name="__unnamed_material_13"/>
@@ -290,11 +289,11 @@
   <link name="thrust7">
     <inertial>
-      <origin xyz="0.189044325927537 -1.16573417585641e-14 0.110144792463057" rpy="0.0 -0.0 0.0"/>
-      <mass value="0.00283424938765199"/>
-      <inertia ixx="1.14046915395644e-06" ixy="-2.35978085149128e-20" ixz="-2.81725401403391e-07" iyy="6.52506444942998e-07" iyz="5.05572790392411e-21" izz="8.15160681280793e-07"/>
-    </inertial>
-    <visual>
-      <geometry>
-        <mesh filename="package://uuv_d/urdf/mesh/proto_type/meshes/thrust7.dae"/>
+      <origin xyz="0 0 0" rpy="0.0 0.0 0.0"/>
+      <mass value="0.00001"/>
+      <inertia ixx="0.00001" ixy="0.0" ixz="0.0" iyy="0.00001" iyz="0" izz="0.00001"/>
+    </inertial>
+    <visual>
+      <geometry>
+        <mesh filename="package://uuv_d/urdf/mesh/proto_type/meshes/thrust7.STL"/>
       </geometry>
       <material name="__unnamed_material_14"/>
@@ -316,5 +315,5 @@
     <visual>
       <geometry>
-        <mesh filename="package://uuv_d/urdf/mesh/proto_type/meshes/t8.dae"/>
+        <mesh filename="package://uuv_d/urdf/mesh/proto_type/meshes/t8.STL"/>
       </geometry>
       <material name="__unnamed_material_15"/>
@@ -330,7 +329,7 @@
   <link name="thrust8">
     <inertial>
-      <origin xyz="0 0 0.001" rpy="0 0 0"/>
-      <mass value="0.0028342"/>
-      <inertia ixx="6.5251e-07" ixy="0.0" ixz="0.0" iyy="6.5251e-07" iyz="0.0" izz="1.3031e-06"/>
+      <origin xyz="0 0 0" rpy="0.0 0.0 0.0"/>
+      <mass value="0.00001"/>
+      <inertia ixx="0.00001" ixy="0.0" ixz="0.0" iyy="0.00001" iyz="0" izz="0.00001"/>
     </inertial>
   </link>
