Commit message: make uuv_d package standalone for roscd and catkin build

File: robots/uuv_d/robots/quad/default_mode_201907/robot.gazebo.xacro (robot description, xacro)
@@ -4,5 +4,5 @@
   <xacro:arg name="robot_name" default="hydrus" />
   <!-- robot urdf -->
-  <xacro:include filename="$(find hydrus)/robots/quad/default_mode_201907/robot.urdf.xacro" />
+  <xacro:include filename="$(find uuv_d)/robots/quad/default_mode_201907/robot.urdf.xacro" />
   <!-- gazebo plugin for default controller and sensors -->
   <xacro:include filename="$(find aerial_robot_simulation)/xacro/spinal.gazebo.xacro" />

File: robots/uuv_d/robots/quad/default_mode_201907/robot.urdf.xacro (robot description, xacro)
@@ -3,6 +3,6 @@
     xmlns:xacro="http://www.ros.org/wiki/xacro" name="hydrus" >
   <!-- basic kinematics model -->
-  <xacro:include filename="$(find hydrus)/urdf/common.xacro" />
-  <xacro:include filename="$(find hydrus)/urdf/link.urdf.xacro" />
+  <xacro:include filename="$(find uuv_d)/urdf/common.xacro" />
+  <xacro:include filename="$(find uuv_d)/urdf/link.urdf.xacro" />
   <xacro:hydrus_link links="4" self="1" rotor_direction="-1" with_battery = "0" />
   <xacro:hydrus_link links="4" self="2" rotor_direction="1"  with_battery = "0" />
@@ -11,5 +11,5 @@
   <!-- special battery arrangement -->
   <xacro:extra_module name = "bat1" parent = "link1" visible = "1"
-                      model_url = "package://hydrus/urdf/mesh/battery/Kypom-3000-6s.dae" >
+                      model_url = "package://uuv_d/urdf/mesh/battery/Kypom-3000-6s.dae" >
     <origin xyz="${link_length/2} 0.0 -0.048" rpy="0 0 0"/>
     <inertial>
@@ -22,5 +22,5 @@
   </xacro:extra_module>
   <xacro:extra_module name = "bat2" parent = "link4" visible = "1"
-                      model_url = "package://hydrus/urdf/mesh/battery/Kypom-3000-6s.dae" >
+                      model_url = "package://uuv_d/urdf/mesh/battery/Kypom-3000-6s.dae" >
     <origin xyz="${link_length/2} 0.0 -0.048" rpy="0 0 0"/>
     <inertial>
@@ -36,5 +36,5 @@
   <!-- 1.1 flight controller -->
   <xacro:extra_module name = "fc" parent = "link2" visible = "1"
-                      model_url = "package://hydrus/urdf/mesh/ver2/flight_controller/spinal.dae"> <!-- same with intel euclid -->
+                      model_url = "package://uuv_d/urdf/mesh/ver2/flight_controller/spinal.dae"> <!-- same with intel euclid -->
     <origin xyz="${link_length / 2 + 0.2221} ${-4.4*0.001} 0.02135" rpy="0 0 0"/>
     <inertial>
@@ -51,5 +51,5 @@
   <!-- confirm the inertial parameter with real machine -->
   <xacro:extra_module name = "pc" parent = "link3" visible = "1"
-                      model_url = "package://hydrus/urdf/mesh/ver2/processor/jetson_tx2_unit.dae" >
+                      model_url = "package://uuv_d/urdf/mesh/ver2/processor/jetson_tx2_unit.dae" >
     <origin xyz="${link_length / 2 - 0.23775} 0.0 ${-0.01}" rpy="0 0 0"/>
     <inertial>
@@ -66,5 +66,5 @@
   <!-- 2.1 leddar one -->
   <xacro:extra_module name = "leddarone" parent = "link3" visible = "1"
-                      model_url = "package://hydrus/urdf/mesh/sensor/leddar_one_tx2_attached_mode.dae">
+                      model_url = "package://uuv_d/urdf/mesh/sensor/leddar_one_tx2_attached_mode.dae">
     <origin xyz="${link_length/2 - 0.1855} 0.0 -0.0626" rpy="${pi} 0 0"/>
     <inertial>
@@ -79,5 +79,5 @@
   <!-- 2.2 gps -->
   <xacro:extra_module name = "gps" parent = "link2" visible = "1"
-                      model_url = "package://hydrus/urdf/mesh/sensor/gps_ublox_m8n.dae">
+                      model_url = "package://uuv_d/urdf/mesh/sensor/gps_ublox_m8n.dae">
     <origin xyz="${link_length/2 + 0.1925} 0.0 0.152" rpy="0 0 0"/>
     <inertial>

File: robots/uuv_d/robots/quad/old_model_tx2_rs_t265_201906/robot.gazebo.xacro (robot description, xacro)
@@ -4,5 +4,5 @@
   <xacro:arg name="robot_name" default="hydrus" />
   <!-- robot urdf -->
-  <xacro:include filename="$(find hydrus)/robots/quad/old_model_tx2_rs_t265_201906/robot.urdf.xacro" />
+  <xacro:include filename="$(find uuv_d)/robots/quad/old_model_tx2_rs_t265_201906/robot.urdf.xacro" />
   <!-- gazebo plugin for default controller and sensors -->
   <xacro:include filename="$(find aerial_robot_simulation)/xacro/spinal.gazebo.xacro" />

File: robots/uuv_d/robots/quad/old_model_tx2_rs_t265_201906/robot.urdf.xacro (robot description, xacro)
@@ -4,6 +4,6 @@
   <!-- basic kinematics model -->
   <m_f_rate value="-0.0182" /> <!-- overwrite -->
-  <xacro:include filename="$(find hydrus)/urdf/common.xacro" />
-  <xacro:include filename="$(find hydrus)/urdf/link.urdf.xacro" />
+  <xacro:include filename="$(find uuv_d)/urdf/common.xacro" />
+  <xacro:include filename="$(find uuv_d)/urdf/link.urdf.xacro" />
   <xacro:hydrus_link links="4" self="1" rotor_direction="-1" with_battery = "0" old_version = "1" />
   <xacro:hydrus_link links="4" self="2" rotor_direction="1"  with_battery = "0" old_version = "1" />
@@ -12,5 +12,5 @@
   <!-- special battery arrangement -->
   <xacro:extra_module name = "bat1" parent = "link1" visible = "1"
-                      model_url = "package://hydrus/urdf/mesh/battery/Kypom-3000-6s.dae" scale="0.001">
+                      model_url = "package://uuv_d/urdf/mesh/battery/Kypom-3000-6s.dae" scale="0.001">
     <origin xyz="${link_length/2} 0.0 -0.048" rpy="0 0 0"/>
     <inertial>
@@ -23,5 +23,5 @@
   </xacro:extra_module>
   <xacro:extra_module name = "bat2" parent = "link4" visible = "1"
-                      model_url = "package://hydrus/urdf/mesh/battery/Kypom-3000-6s.dae" scale="0.001">
+                      model_url = "package://uuv_d/urdf/mesh/battery/Kypom-3000-6s.dae" scale="0.001">
     <origin xyz="${link_length/2} 0.0 -0.048" rpy="0 0 0"/>
     <inertial>
@@ -37,5 +37,5 @@
   <!-- 1.1 flight controller -->
   <xacro:extra_module name = "fc" parent = "link2" visible = "1"
-                      model_url = "package://hydrus/urdf/mesh/ver1/flight_controller/fc_euclid201806.dae"> <!-- same with intel euclid -->
+                      model_url = "package://uuv_d/urdf/mesh/ver1/flight_controller/fc_euclid201806.dae"> <!-- same with intel euclid -->
     <origin xyz="${link_length / 2 + 0.2281} ${-4.4*0.001} 0.03533" rpy="0 0 0"/>
     <inertial>
@@ -51,5 +51,5 @@
   <!-- 1.2 processor: jetson tx2 -->
   <xacro:extra_module name = "pc" parent = "link3" visible = "1"
-                      model_url = "package://hydrus/urdf/mesh/ver1/processor/jetson_tx2.dae"
+                      model_url = "package://uuv_d/urdf/mesh/ver1/processor/jetson_tx2.dae"
                       scale="0.001" >
     <origin xyz="0.086 0.0 ${-0.0192}" rpy="0 0 ${pi}"/>
@@ -67,5 +67,5 @@
   <!-- 2.1 leddar one -->
   <xacro:extra_module name = "leddarone" parent = "link3" visible = "1"
-                      model_url = "package://hydrus/urdf/mesh/sensor/leddar_one_tx2_attached_mode.dae">
+                      model_url = "package://uuv_d/urdf/mesh/sensor/leddar_one_tx2_attached_mode.dae">
     <origin xyz="0.0866 0.0 -0.06267" rpy="0 ${pi} 0"/>
     <inertial>
@@ -80,5 +80,5 @@
   <!-- 2.2 gps -->
   <xacro:extra_module name = "gps" parent = "link2" visible = "1"
-                      model_url = "package://hydrus/urdf/mesh/sensor/gps_ublox_m8n.dae">
+                      model_url = "package://uuv_d/urdf/mesh/sensor/gps_ublox_m8n.dae">
     <origin xyz="${link_length/2 + 0.1925} 0.0 0.152" rpy="0 0 0"/>
     <inertial>
@@ -104,5 +104,5 @@
   <!-- 2.3  side-view  and downwards realsense t265 -->
   <xacro:extra_module name = "realsense_t265_modules_unit" parent = "link2" visible = "1"
-                      model_url = "package://hydrus/urdf/mesh/ver1/sensor/realsense_t265_unit.dae">
+                      model_url = "package://uuv_d/urdf/mesh/ver1/sensor/realsense_t265_unit.dae">
     <origin xyz="${link_length/2 + 0.28715} 0.0 -0.04015" rpy="0 0 0"/>
     <inertial>

File: robots/uuv_d/robots/quad/old_model_tx2_zed_201810/robot.gazebo.xacro (robot description, xacro)
@@ -4,5 +4,5 @@
   <xacro:arg name="robot_name" default="hydrus" />
   <!-- robot urdf -->
-  <xacro:include filename="$(find hydrus)/robots/quad/old_model_tx2_zed_201810/robot.urdf.xacro" />
+  <xacro:include filename="$(find uuv_d)/robots/quad/old_model_tx2_zed_201810/robot.urdf.xacro" />
   <!-- gazebo plugin for default controller and sensors -->
   <xacro:include filename="$(find aerial_robot_simulation)/xacro/spinal.gazebo.xacro" />

File: robots/uuv_d/robots/quad/old_model_tx2_zed_201810/robot.urdf.xacro (robot description, xacro)
@@ -4,6 +4,6 @@
   <!-- basic kinematics model -->
   <m_f_rate value="-0.0182" /> <!-- overwrite -->
-  <xacro:include filename="$(find hydrus)/urdf/common.xacro" />
-  <xacro:include filename="$(find hydrus)/urdf/link.urdf.xacro" />
+  <xacro:include filename="$(find uuv_d)/urdf/common.xacro" />
+  <xacro:include filename="$(find uuv_d)/urdf/link.urdf.xacro" />
   <xacro:hydrus_link links="4" self="1" rotor_direction="-1" with_battery = "0" old_version = "1" />
   <xacro:hydrus_link links="4" self="2" rotor_direction="1"  with_battery = "0" old_version = "1" />
@@ -12,5 +12,5 @@
   <!-- special battery arrangement -->
   <xacro:extra_module name = "bat1" parent = "link1" visible = "1"
-                      model_url = "package://hydrus/urdf/mesh/battery/Kypom-3000-6s.dae" >
+                      model_url = "package://uuv_d/urdf/mesh/battery/Kypom-3000-6s.dae" >
     <origin xyz="${link_length/2} 0.0 -0.048" rpy="0 0 0"/>
     <inertial>
@@ -23,5 +23,5 @@
   </xacro:extra_module>
   <xacro:extra_module name = "bat2" parent = "link4" visible = "1"
-                      model_url = "package://hydrus/urdf/mesh/battery/Kypom-3000-6s.dae" >
+                      model_url = "package://uuv_d/urdf/mesh/battery/Kypom-3000-6s.dae" >
     <origin xyz="${link_length/2} 0.0 -0.048" rpy="0 0 0"/>
     <inertial>
@@ -37,5 +37,5 @@
   <!-- 1.1 flight controller -->
   <xacro:extra_module name = "fc" parent = "link2" visible = "1"
-                      model_url = "package://hydrus/urdf/mesh/ver1/flight_controller/fc_euclid201806.dae"> <!-- same with intel euclid -->
+                      model_url = "package://uuv_d/urdf/mesh/ver1/flight_controller/fc_euclid201806.dae"> <!-- same with intel euclid -->
     <origin xyz="${link_length / 2 + 0.2281} ${-4.4*0.001} 0.03533" rpy="0 0 0"/>
     <inertial>
@@ -51,5 +51,5 @@
   <!-- 1.2 processor: jetson tx2 -->
   <xacro:extra_module name = "pc" parent = "link3" visible = "1"
-                      model_url = "package://hydrus/urdf/mesh/ver1/processor/jetson_tx2.dae"
+                      model_url = "package://uuv_d/urdf/mesh/ver1/processor/jetson_tx2.dae"
                       scale="0.001" >
     <origin xyz="0.086 0.0 ${-0.0192}" rpy="0 0 ${pi}"/>
@@ -67,5 +67,5 @@
   <!-- 2.1 leddar one -->
   <xacro:extra_module name = "leddarone" parent = "link3" visible = "1"
-                      model_url = "package://hydrus/urdf/mesh/sensor/leddar_one_tx2_attached_mode.dae">
+                      model_url = "package://uuv_d/urdf/mesh/sensor/leddar_one_tx2_attached_mode.dae">
     <origin xyz="0.0866 0.0 -0.06267" rpy="0 ${pi} 0"/>
     <inertial>
@@ -80,5 +80,5 @@
   <!-- 2.2 gps -->
   <xacro:extra_module name = "gps" parent = "link2" visible = "1"
-                      model_url = "package://hydrus/urdf/mesh/sensor/gps_ublox_m8n.dae">
+                      model_url = "package://uuv_d/urdf/mesh/sensor/gps_ublox_m8n.dae">
     <origin xyz="${link_length/2 + 0.1925} 0.0 0.152" rpy="0 0 0"/>
     <inertial>
@@ -104,5 +104,5 @@
   <!-- 2.3 sensor: zed mini with servo -->
   <xacro:extra_module name = "zed_mini_servo_up" parent = "link2" visible = "1"
-                      model_url = "package://hydrus/urdf/mesh/ver1/sensor/zed_mini_servo_up.dae">
+                      model_url = "package://uuv_d/urdf/mesh/ver1/sensor/zed_mini_servo_up.dae">
     <origin xyz="${link_length/2 + 0.28715} 0.0 -0.04015" rpy="0 0 0"/>
     <inertial>
@@ -134,5 +134,5 @@
       <origin xyz="${-14.75 * 0.001} 0 ${-19 * 0.001}" rpy="0 ${pi/2} ${pi/2}"/>
       <geometry>
-        <mesh filename="package://hydrus/urdf/mesh/ver1/sensor/zed_mini_servo_down.dae"/>
+        <mesh filename="package://uuv_d/urdf/mesh/ver1/sensor/zed_mini_servo_down.dae"/>
       </geometry>
     </visual>

File: robots/uuv_d/robots/quad/tilt_10deg_15inch_202106/robot.gazebo.xacro (robot description, xacro)
@@ -4,5 +4,5 @@
   <xacro:arg name="robot_name" default="hydrus" />
   <!-- robot urdf -->
-  <xacro:include filename="$(find hydrus)/robots/quad/tilt_10deg_15inch_202106/robot.urdf.xacro" />
+  <xacro:include filename="$(find uuv_d)/robots/quad/tilt_10deg_15inch_202106/robot.urdf.xacro" />
   <!-- gazebo plugin for default controller and sensors -->
   <xacro:include filename="$(find aerial_robot_simulation)/xacro/spinal.gazebo.xacro" />

File: robots/uuv_d/robots/quad/tilt_10deg_15inch_202106/robot.urdf.xacro (robot description, xacro)
@@ -3,6 +3,6 @@
     xmlns:xacro="http://www.ros.org/wiki/xacro" name="hydrus" >
   <!-- basic kinematics model -->
-  <xacro:include filename="$(find hydrus)/urdf/common.xacro" />
-  <xacro:include filename="$(find hydrus)/urdf/link.urdf.xacro" />
+  <xacro:include filename="$(find uuv_d)/urdf/common.xacro" />
+  <xacro:include filename="$(find uuv_d)/urdf/link.urdf.xacro" />
   <xacro:hydrus_link links="4" self="1" rotor_direction="-1" with_battery = "0" tilt_mode="1" tilt_angle="10" prop_15inch="1"/>
   <xacro:hydrus_link links="4" self="2" rotor_direction="1"  with_battery = "0" tilt_mode="1" tilt_angle="10" prop_15inch="1"/>
@@ -11,5 +11,5 @@
   <!-- special battery arrangement -->
   <xacro:extra_module name = "bat1" parent = "link1" visible = "1"
-                      model_url = "package://hydrus/urdf/mesh/battery/Kypom-3000-6s.dae" >
+                      model_url = "package://uuv_d/urdf/mesh/battery/Kypom-3000-6s.dae" >
     <origin xyz="${link_length/2} 0.0 -0.048" rpy="0 0 0"/>
     <inertial>
@@ -22,5 +22,5 @@
   </xacro:extra_module>
   <xacro:extra_module name = "bat2" parent = "link4" visible = "1"
-                      model_url = "package://hydrus/urdf/mesh/battery/Kypom-3000-6s.dae" >
+                      model_url = "package://uuv_d/urdf/mesh/battery/Kypom-3000-6s.dae" >
     <origin xyz="${link_length/2} 0.0 -0.048" rpy="0 0 0"/>
     <inertial>
@@ -36,5 +36,5 @@
   <!-- 1.1 flight controller -->
   <xacro:extra_module name = "fc" parent = "link2" visible = "1"
-                      model_url = "package://hydrus/urdf/mesh/ver2/flight_controller/spinal.dae"> <!-- same with intel euclid -->
+                      model_url = "package://uuv_d/urdf/mesh/ver2/flight_controller/spinal.dae"> <!-- same with intel euclid -->
     <origin xyz="${link_length / 2 + 0.2221} ${-4.4*0.001} 0.02135" rpy="0 0 0"/>
     <inertial>
@@ -51,5 +51,5 @@
   <!-- confirm the inertial parameter with real machine -->
   <xacro:extra_module name = "pc" parent = "link3" visible = "1"
-                      model_url = "package://hydrus/urdf/mesh/ver2/processor/jetson_tx2_unit.dae" >
+                      model_url = "package://uuv_d/urdf/mesh/ver2/processor/jetson_tx2_unit.dae" >
     <origin xyz="${link_length / 2 - 0.23775} 0.0 ${-0.01}" rpy="0 0 0"/>
     <inertial>
@@ -66,5 +66,5 @@
   <!-- 2.1 leddar one -->
   <xacro:extra_module name = "leddarone" parent = "link3" visible = "1"
-                      model_url = "package://hydrus/urdf/mesh/sensor/leddar_one_tx2_attached_mode.dae">
+                      model_url = "package://uuv_d/urdf/mesh/sensor/leddar_one_tx2_attached_mode.dae">
     <origin xyz="${link_length/2 - 0.1855} 0.0 -0.0626" rpy="${pi} 0 0"/>
     <inertial>
@@ -79,5 +79,5 @@
   <!-- 2.2 gps -->
   <xacro:extra_module name = "gps" parent = "link2" visible = "1"
-                      model_url = "package://hydrus/urdf/mesh/sensor/gps_ublox_m8n.dae">
+                      model_url = "package://uuv_d/urdf/mesh/sensor/gps_ublox_m8n.dae">
     <origin xyz="${link_length/2 + 0.1925} 0.0 0.152" rpy="0 0 0"/>
     <inertial>

File: robots/uuv_d/robots/quad/tilt_10deg_201907/robot.gazebo.xacro (robot description, xacro)
@@ -4,5 +4,5 @@
   <xacro:arg name="robot_name" default="hydrus" />
   <!-- robot urdf -->
-  <xacro:include filename="$(find hydrus)/robots/quad/tilt_10deg_201907/robot.urdf.xacro" />
+  <xacro:include filename="$(find uuv_d)/robots/quad/tilt_10deg_201907/robot.urdf.xacro" />
   <!-- gazebo plugin for default controller and sensors -->
   <xacro:include filename="$(find aerial_robot_simulation)/xacro/spinal.gazebo.xacro" />

File: robots/uuv_d/robots/quad/tilt_10deg_201907/robot.urdf.xacro (robot description, xacro)
@@ -3,6 +3,6 @@
     xmlns:xacro="http://www.ros.org/wiki/xacro" name="hydrus" >
   <!-- basic kinematics model -->
-  <xacro:include filename="$(find hydrus)/urdf/common.xacro" />
-  <xacro:include filename="$(find hydrus)/urdf/link.urdf.xacro" />
+  <xacro:include filename="$(find uuv_d)/urdf/common.xacro" />
+  <xacro:include filename="$(find uuv_d)/urdf/link.urdf.xacro" />
   <xacro:hydrus_link links="4" self="1" rotor_direction="-1" with_battery = "0" tilt_mode="1" tilt_angle="10" />
   <xacro:hydrus_link links="4" self="2" rotor_direction="1"  with_battery = "0" tilt_mode="1" tilt_angle="10"/>
@@ -11,5 +11,5 @@
   <!-- special battery arrangement -->
   <xacro:extra_module name = "bat1" parent = "link1" visible = "1"
-                      model_url = "package://hydrus/urdf/mesh/battery/Kypom-3000-6s.dae" >
+                      model_url = "package://uuv_d/urdf/mesh/battery/Kypom-3000-6s.dae" >
     <origin xyz="${link_length/2} 0.0 -0.048" rpy="0 0 0"/>
     <inertial>
@@ -22,5 +22,5 @@
   </xacro:extra_module>
   <xacro:extra_module name = "bat2" parent = "link4" visible = "1"
-                      model_url = "package://hydrus/urdf/mesh/battery/Kypom-3000-6s.dae" >
+                      model_url = "package://uuv_d/urdf/mesh/battery/Kypom-3000-6s.dae" >
     <origin xyz="${link_length/2} 0.0 -0.048" rpy="0 0 0"/>
     <inertial>
@@ -36,5 +36,5 @@
   <!-- 1.1 flight controller -->
   <xacro:extra_module name = "fc" parent = "link2" visible = "1"
-                      model_url = "package://hydrus/urdf/mesh/ver2/flight_controller/spinal.dae"> <!-- same with intel euclid -->
+                      model_url = "package://uuv_d/urdf/mesh/ver2/flight_controller/spinal.dae"> <!-- same with intel euclid -->
     <origin xyz="${link_length / 2 + 0.2221} ${-4.4*0.001} 0.02135" rpy="0 0 0"/>
     <inertial>
@@ -51,5 +51,5 @@
   <!-- confirm the inertial parameter with real machine -->
   <xacro:extra_module name = "pc" parent = "link3" visible = "1"
-                      model_url = "package://hydrus/urdf/mesh/ver2/processor/jetson_tx2_unit.dae" >
+                      model_url = "package://uuv_d/urdf/mesh/ver2/processor/jetson_tx2_unit.dae" >
     <origin xyz="${link_length / 2 - 0.23775} 0.0 ${-0.01}" rpy="0 0 0"/>
     <inertial>
@@ -66,5 +66,5 @@
   <!-- 2.1 leddar one -->
   <xacro:extra_module name = "leddarone" parent = "link3" visible = "1"
-                      model_url = "package://hydrus/urdf/mesh/sensor/leddar_one_tx2_attached_mode.dae">
+                      model_url = "package://uuv_d/urdf/mesh/sensor/leddar_one_tx2_attached_mode.dae">
     <origin xyz="${link_length/2 - 0.1855} 0.0 -0.0626" rpy="${pi} 0 0"/>
     <inertial>
@@ -79,5 +79,5 @@
   <!-- 2.2 gps -->
   <xacro:extra_module name = "gps" parent = "link2" visible = "1"
-                      model_url = "package://hydrus/urdf/mesh/sensor/gps_ublox_m8n.dae">
+                      model_url = "package://uuv_d/urdf/mesh/sensor/gps_ublox_m8n.dae">
     <origin xyz="${link_length/2 + 0.1925} 0.0 0.152" rpy="0 0 0"/>
     <inertial>

File: robots/uuv_d/robots/quad/tilt_20deg_201907/robot.gazebo.xacro (robot description, xacro)
@@ -4,5 +4,5 @@
   <xacro:arg name="robot_name" default="hydrus" />
   <!-- robot urdf -->
-  <xacro:include filename="$(find hydrus)/robots/quad/tilt_20deg_201907/robot.urdf.xacro" />
+  <xacro:include filename="$(find uuv_d)/robots/quad/tilt_20deg_201907/robot.urdf.xacro" />
   <!-- gazebo plugin for default controller and sensors -->
   <xacro:include filename="$(find aerial_robot_simulation)/xacro/spinal.gazebo.xacro" />
