Commit message: make uuv_d package standalone for roscd and catkin build

File: robots/uuv_d/robots/quad/tilt_20deg_201907/robot.urdf.xacro (robot description, xacro)
@@ -3,6 +3,6 @@
     xmlns:xacro="http://www.ros.org/wiki/xacro" name="hydrus" >
   <!-- basic kinematics model -->
-  <xacro:include filename="$(find hydrus)/urdf/common.xacro" />
-  <xacro:include filename="$(find hydrus)/urdf/link.urdf.xacro" />
+  <xacro:include filename="$(find uuv_d)/urdf/common.xacro" />
+  <xacro:include filename="$(find uuv_d)/urdf/link.urdf.xacro" />
   <xacro:hydrus_link links="4" self="1" rotor_direction="-1" with_battery = "0" tilt_mode="1" tilt_angle="20" />
   <xacro:hydrus_link links="4" self="2" rotor_direction="1"  with_battery = "0" tilt_mode="1" tilt_angle="20"/>
@@ -11,5 +11,5 @@
   <!-- special battery arrangement -->
   <xacro:extra_module name = "bat1" parent = "link1" visible = "1"
-                      model_url = "package://hydrus/urdf/mesh/battery/Kypom-3000-6s.dae" >
+                      model_url = "package://uuv_d/urdf/mesh/battery/Kypom-3000-6s.dae" >
     <origin xyz="${link_length/2} 0.0 -0.048" rpy="0 0 0"/>
     <inertial>
@@ -22,5 +22,5 @@
   </xacro:extra_module>
   <xacro:extra_module name = "bat2" parent = "link4" visible = "1"
-                      model_url = "package://hydrus/urdf/mesh/battery/Kypom-3000-6s.dae" >
+                      model_url = "package://uuv_d/urdf/mesh/battery/Kypom-3000-6s.dae" >
     <origin xyz="${link_length/2} 0.0 -0.048" rpy="0 0 0"/>
     <inertial>
@@ -36,5 +36,5 @@
   <!-- 1.1 flight controller -->
   <xacro:extra_module name = "fc" parent = "link2" visible = "1"
-                      model_url = "package://hydrus/urdf/mesh/ver2/flight_controller/spinal.dae"> <!-- same with intel euclid -->
+                      model_url = "package://uuv_d/urdf/mesh/ver2/flight_controller/spinal.dae"> <!-- same with intel euclid -->
     <origin xyz="${link_length / 2 + 0.2221} ${-4.4*0.001} 0.02135" rpy="0 0 0"/>
     <inertial>
@@ -51,5 +51,5 @@
   <!-- confirm the inertial parameter with real machine -->
   <xacro:extra_module name = "pc" parent = "link3" visible = "1"
-                      model_url = "package://hydrus/urdf/mesh/ver2/processor/jetson_tx2_unit.dae" >
+                      model_url = "package://uuv_d/urdf/mesh/ver2/processor/jetson_tx2_unit.dae" >
     <origin xyz="${link_length / 2 - 0.23775} 0.0 ${-0.01}" rpy="0 0 0"/>
     <inertial>
@@ -66,5 +66,5 @@
   <!-- 2.1 leddar one -->
   <xacro:extra_module name = "leddarone" parent = "link3" visible = "1"
-                      model_url = "package://hydrus/urdf/mesh/sensor/leddar_one_tx2_attached_mode.dae">
+                      model_url = "package://uuv_d/urdf/mesh/sensor/leddar_one_tx2_attached_mode.dae">
     <origin xyz="${link_length/2 - 0.1855} 0.0 -0.0626" rpy="${pi} 0 0"/>
     <inertial>
@@ -79,5 +79,5 @@
   <!-- 2.2 gps -->
   <xacro:extra_module name = "gps" parent = "link2" visible = "1"
-                      model_url = "package://hydrus/urdf/mesh/sensor/gps_ublox_m8n.dae">
+                      model_url = "package://uuv_d/urdf/mesh/sensor/gps_ublox_m8n.dae">
     <origin xyz="${link_length/2 + 0.1925} 0.0 0.152" rpy="0 0 0"/>
     <inertial>

File: robots/uuv_d/urdf/common.xacro (robot description, xacro)
@@ -40,5 +40,5 @@
         <origin rpy="0 0 0" xyz="${link_length* 0.5} 0 0"/>
         <geometry>
-          <mesh filename="package://hydrus/urdf/mesh/ver1/link/${type}_link.dae"/>
+          <mesh filename="package://uuv_d/urdf/mesh/ver1/link/${type}_link.dae"/>
         </geometry>
       </xacro:if>
@@ -48,12 +48,12 @@
           <xacro:if value="${tilt_mode == 1}">
             <xacro:if value="${prop_15inch == 1}">
-              <mesh filename="package://hydrus/urdf/mesh/ver2/link/tilt_${tilt_angle}deg_15inch_link${type}.dae"/>
+              <mesh filename="package://uuv_d/urdf/mesh/ver2/link/tilt_${tilt_angle}deg_15inch_link${type}.dae"/>
             </xacro:if>
             <xacro:unless value="${prop_15inch == 1}">
-              <mesh filename="package://hydrus/urdf/mesh/ver2/link/tilt_${tilt_angle}deg_link${type}.dae"/>
+              <mesh filename="package://uuv_d/urdf/mesh/ver2/link/tilt_${tilt_angle}deg_link${type}.dae"/>
             </xacro:unless>
           </xacro:if>
           <xacro:unless value="${tilt_mode == 1}">
-            <mesh filename="package://hydrus/urdf/mesh/ver2/link/link${type}.dae"/>
+            <mesh filename="package://uuv_d/urdf/mesh/ver2/link/link${type}.dae"/>
           </xacro:unless>
         </geometry>
@@ -81,5 +81,5 @@
   <xacro:macro name="standard_leg_old_version" params="parent self:=${self} *origin">
     <xacro:extra_module name = "leg${self}" parent = "${parent}" visible = "1"
-                        model_url = "package://hydrus/urdf/mesh/ver1/leg/standard_legs.dae" >
+                        model_url = "package://uuv_d/urdf/mesh/ver1/leg/standard_legs.dae" >
       <xacro:insert_block name="origin" />
       <inertial>
@@ -102,5 +102,5 @@
   <xacro:macro name="standard_leg_joint" params="parent self:=${self} *origin">
     <xacro:extra_module name = "leg${self}" parent = "${parent}" visible = "1"
-                        model_url = "package://hydrus/urdf/mesh/ver2/leg/joint_leg.dae" >
+                        model_url = "package://uuv_d/urdf/mesh/ver2/leg/joint_leg.dae" >
       <xacro:insert_block name="origin" />
       <inertial>
@@ -115,5 +115,5 @@
   <xacro:macro name="standard_leg_end" params="parent self:=${self} *origin">
     <xacro:extra_module name = "leg${self}" parent = "${parent}" visible = "1"
-                        model_url = "package://hydrus/urdf/mesh/ver2/leg/end_leg.dae" >
+                        model_url = "package://uuv_d/urdf/mesh/ver2/leg/end_leg.dae" >
       <xacro:insert_block name="origin" />
       <inertial>

File: robots/uuv_d/urdf/link.urdf.xacro (robot description, xacro)
@@ -224,8 +224,8 @@
         <geometry>
           <xacro:if value="${rotor_direction == 1}">
-            <mesh filename="package://hydrus/urdf/mesh/propeller/T-motor-CF-14inch-CCW.dae"/>
+            <mesh filename="package://uuv_d/urdf/mesh/propeller/T-motor-CF-14inch-CCW.dae"/>
           </xacro:if>
           <xacro:if value="${rotor_direction == -1}">
-            <mesh filename="package://hydrus/urdf/mesh/propeller/T-motor-CF-14inch-CW.dae"/>
+            <mesh filename="package://uuv_d/urdf/mesh/propeller/T-motor-CF-14inch-CW.dae"/>
           </xacro:if>
         </geometry>
@@ -238,5 +238,5 @@
       <!-- note: use the same configuration between new and old version -->
       <xacro:extra_module name = "bat${self}" parent = "link${self}" visible = "1"
-                          model_url = "package://hydrus/urdf/mesh/battery/VOLTON-PG-1300LP2-6s.stl" scale="0.001">
+                          model_url = "package://uuv_d/urdf/mesh/battery/VOLTON-PG-1300LP2-6s.stl" scale="0.001">
         <origin xyz="${link_length/2} 0.0 -0.048" rpy="0 0 0"/>
         <inertial>

Commit message: enable buoyancy

File: robots/uuv_d/robots/quad/default_mode_201907/robot.gazebo.xacro (robot description, xacro)
@@ -8,12 +8,17 @@
   <xacro:include filename="$(find aerial_robot_simulation)/xacro/spinal.gazebo.xacro" />
   <xacro:gazebo_spinal robot_name="$(arg robot_name)" gps_frame="fc"/>
-  <!-- <gazebo>
+  <gazebo reference="root_joint">
+    <disableFixedJointLumping>true</disableFixedJointLumping>
+  </gazebo>
+  <gazebo>
     <plugin name="uuv_plugin" filename="libuuv_underwater_object_ros_plugin.so">
       <fluid_density>1000.0</fluid_density>
       <flow_velocity_topic>/hydrodynamics/current_velocity</flow_velocity_topic>
       <debug>1</debug>
-      <link name="main_body">
+      <link name="base_link">
         <neutrally_buoyant>0</neutrally_buoyant>
-        <volume>0.0</volume>
+        <!-- todo: adjust the volume according to the real robot -->
+        <volume>0.001</volume>
+        <scaling_volume>0.0</scaling_volume>
         <box>
           <width>0.28</width>
@@ -32,9 +37,9 @@
             0 0 0 0 0 0
           </added_mass>
-          <linear_damping> -0.1 -0.1 -0.1 -0.01 -0.01 -0.01</linear_damping>
-          <quadratic_damping>-0.2 -0.2 -0.4 -0.02 -0.02 -0.02</quadratic_damping>
+          <linear_damping> -1.0 -1.0 -1.0 -0.01 -0.01 -0.01</linear_damping>
+          <quadratic_damping>-10.0 -10.0 -10.0 -0.02 -0.02 -0.02</quadratic_damping>
         </hydrodynamic_model>
       </link>
     </plugin>
-  </gazebo> -->
+  </gazebo>
 </robot>
