Commit message: update to rotate from joint

File: robots/hydrus/mujoco/quad/soft_airframe_202605/robot.urdf (robot description, URDF)
Before this commit: robot serial_soft_airframe, 44 links, 43 joints
Joints:
- joint gimbal_joint1: origin xyz=0.096 0 0 rpy=0 0 0 -> xyz=0.096 0 0 rpy=0 -0.174 0
- joint gimbal_joint2: origin xyz=0.156 0 0 rpy=0 0 0 -> xyz=0.156 0 0 rpy=0 0.174 0
- joint gimbal_joint3: origin xyz=0.096 0 0 rpy=0 0 0 -> xyz=0.096 0 0 rpy=0 -0.174 0
- joint gimbal_joint4: origin xyz=0.096 0 0 rpy=0 0 0 -> xyz=0.096 0 0 rpy=0 0.174 0
- joint soft_joint11: origin xyz=0.147 0 0 rpy=0 0 0 -> xyz=0.147 0 0 rpy=0 -0.174 0
- joint soft_joint16: origin xyz=0.147 0 0 rpy=0 0 0 -> xyz=0.147 0 0 rpy=0 0.174 0
- joint soft_joint6: origin xyz=0.147 0 0 rpy=0 0 0 -> xyz=0.147 0 0 rpy=0 0.174 0

File: robots/hydrus/robots/quad/soft_airframe_202605/robot.urdf.xacro (robot description, xacro)
@@ -53,5 +53,5 @@
   <!-- Four soft-link modules connected in series.
        Module i creates:
-         servo_link{i}, soft_link{5*i-4..5*i}, gimbal_link{i}, thrust{i}
+         servo_link{i}, soft_link{3*i-2}, soft_link{3*i-1}, soft_link{3*i}, gimbal_link{i}, thrust{i}
   -->
   <xacro:soft_link_module
@@ -60,4 +60,5 @@
       rotor_direction="-1"
       parent_to_servo_x="0.0"
+      prev_tilt_angle="0"
       tilt_angle="-0.174" />
   <xacro:soft_link_module
@@ -69,4 +70,5 @@
       servo_size_z="0.01"
       servo_mass="0.18"
+      prev_tilt_angle="0.174"
       tilt_angle="0.174" />
   <!-- The third module has a slightly longer and larger servo body. -->
@@ -75,4 +77,5 @@
       parent="gimbal_link2"
       rotor_direction="-1"
+      prev_tilt_angle="-0.174"
       tilt_angle="-0.174" />
   <xacro:soft_link_module
@@ -80,4 +83,5 @@
       parent="gimbal_link3"
       rotor_direction="1"
+      prev_tilt_angle="0.174"
       tilt_angle="0.174" />
 </robot>

File: robots/hydrus/urdf/soft_link.urdf.xacro (robot description, xacro)
@@ -49,5 +49,6 @@
       leg_mass:=0.04993
       rotor_offset_x:=0.0735
-      tilt_angle:=0.174
+      tilt_angle:=-0.174
+      prev_tilt_angle:=0.174
       gimbal_mesh:=package://hydrus/urdf/mesh/5inch_propeller_duct_right_v2.dae
       propeller_mesh:=package://hydrus/urdf/mesh/TriBlade_5045.dae">
@@ -63,5 +64,5 @@
       <parent link="${parent}"/>
       <child link="soft_link${s0}"/>
-      <origin xyz="${parent_to_servo_x} 0 0" rpy="0 0 0"/>
+      <origin xyz="${parent_to_servo_x} 0 0" rpy="0 ${prev_tilt_angle} 0"/>
     </joint>
     <joint name="soft_joint${s1}" type="revolute">
@@ -347,5 +348,5 @@
       <parent link="servo_link${i}"/>
       <child link="gimbal_link${i}"/>
-      <origin xyz="${servo_size_x} 0 0" rpy="0 0 0"/>
+      <origin xyz="${servo_size_x} 0 0" rpy="0 ${tilt_angle} 0"/>
       <axis xyz="1 0 0"/>
       <dynamics damping="0.9" friction="0.1"/>
