Commit message: tilt to reversed angle

File: robots/hydrus/mujoco/quad/soft_airframe_202605/robot.urdf (robot description, URDF)
Before this commit: robot serial_soft_airframe, 44 links, 43 joints
Joints:
- joint gimbal_joint1: origin xyz=0.096 0 0 rpy=0 -0.174 0 -> xyz=0.096 0 0 rpy=0 0.174 0
- joint gimbal_joint2: origin xyz=0.156 0 0 rpy=0 0.174 0 -> xyz=0.156 0 0 rpy=0 -0.174 0
- joint gimbal_joint3: origin xyz=0.096 0 0 rpy=0 -0.174 0 -> xyz=0.096 0 0 rpy=0 0.174 0
- joint gimbal_joint4: origin xyz=0.096 0 0 rpy=0 0.174 0 -> xyz=0.096 0 0 rpy=0 -0.174 0
- joint soft_joint11: origin xyz=0.147 0 0 rpy=0 -0.174 0 -> xyz=0.147 0 0 rpy=0 0.174 0
- joint soft_joint16: origin xyz=0.147 0 0 rpy=0 0.174 0 -> xyz=0.147 0 0 rpy=0 -0.174 0
- joint soft_joint6: origin xyz=0.147 0 0 rpy=0 0.174 0 -> xyz=0.147 0 0 rpy=0 -0.174 0

File: robots/hydrus/robots/quad/soft_airframe_202605/robot.urdf.xacro (robot description, xacro)
@@ -61,5 +61,5 @@
       parent_to_servo_x="0.0"
       prev_tilt_angle="0"
-      tilt_angle="-0.174" />
+      tilt_angle="0.174" />
   <xacro:soft_link_module
       i="2"
@@ -70,6 +70,6 @@
       servo_size_z="0.01"
       servo_mass="0.18"
-      prev_tilt_angle="0.174"
-      tilt_angle="0.174" />
+      prev_tilt_angle="-0.174"
+      tilt_angle="-0.174" />
   <!-- The third module has a slightly longer and larger servo body. -->
   <xacro:soft_link_module
@@ -77,11 +77,11 @@
       parent="gimbal_link2"
       rotor_direction="-1"
-      prev_tilt_angle="-0.174"
-      tilt_angle="-0.174" />
+      prev_tilt_angle="0.174"
+      tilt_angle="0.174" />
   <xacro:soft_link_module
       i="4"
       parent="gimbal_link3"
       rotor_direction="1"
-      prev_tilt_angle="0.174"
-      tilt_angle="0.174" />
+      prev_tilt_angle="-0.174"
+      tilt_angle="-0.174" />
 </robot>

File: robots/hydrus/urdf/soft_link.urdf.xacro (robot description, xacro)
@@ -354,5 +354,5 @@
     <link name="gimbal_link${i}">
       <inertial>
-        <origin xyz="0.0735 0 0" rpy="0 ${tilt_angle} 0"/>
+        <origin xyz="0.0735 0 0" rpy="0 0 0"/>
         <mass value="0.222"/>
         <inertia
@@ -362,5 +362,5 @@
       </inertial>
       <visual>
-        <origin xyz="0.0735 0 0" rpy="0 ${tilt_angle} 0"/>
+        <origin xyz="0.0735 0 0" rpy="0 0 0"/>
         <geometry>
           <mesh filename="${gimbal_mesh}"/>

Commit message: flatten the model

File: robots/hydrus/mujoco/quad/soft_airframe_202605/robot.urdf (robot description, URDF)
Before this commit: robot serial_soft_airframe, 44 links, 43 joints
Joints:
- joint gimbal_joint1: origin xyz=0.096 0 0 rpy=0 0.174 0 -> xyz=0.096 0 -0.012724564326109165 rpy=0 0.174 0
- joint gimbal_joint2: origin xyz=0.156 0 0 rpy=0 -0.174 0 -> xyz=0.156 0 0.012724564326109165 rpy=0 -0.174 0
- joint gimbal_joint3: origin xyz=0.096 0 0 rpy=0 0.174 0 -> xyz=0.096 0 -0.012724564326109165 rpy=0 0.174 0
- joint gimbal_joint4: origin xyz=0.096 0 0 rpy=0 -0.174 0 -> xyz=0.096 0 0.012724564326109165 rpy=0 -0.174 0
- joint soft_joint1: origin xyz=0.0 0 0 rpy=0 0 0 -> xyz=0.0 0 -0.0 rpy=0 0 0
- joint soft_joint11: origin xyz=0.147 0 0 rpy=0 0.174 0 -> xyz=0.147 0 -0.02544912865221833 rpy=0 0.174 0
- joint soft_joint16: origin xyz=0.147 0 0 rpy=0 -0.174 0 -> xyz=0.147 0 0.02544912865221833 rpy=0 -0.174 0
- joint soft_joint6: origin xyz=0.147 0 0 rpy=0 -0.174 0 -> xyz=0.147 0 0.02544912865221833 rpy=0 -0.174 0

File: robots/hydrus/urdf/soft_link.urdf.xacro (robot description, xacro)
@@ -60,9 +60,12 @@
     <xacro:property name="l0" value="${2 * i - 1}" />
     <xacro:property name="l1" value="${2 * i}" />
+    <!-- Keep tilted module connections close to the original height. -->
+    <xacro:property name="parent_tilt_z_offset" value="${-parent_to_servo_x * sin(prev_tilt_angle)}" />
+    <xacro:property name="gimbal_tilt_z_offset" value="${-rotor_offset_x * sin(tilt_angle)}" />
     <!-- Five-segment soft continuum approximation (1/8, 1/4, 1/4, 1/4, 1/8). -->
     <joint name="soft_joint${s0}" type="fixed">
       <parent link="${parent}"/>
       <child link="soft_link${s0}"/>
-      <origin xyz="${parent_to_servo_x} 0 0" rpy="0 ${prev_tilt_angle} 0"/>
+      <origin xyz="${parent_to_servo_x} 0 ${parent_tilt_z_offset}" rpy="0 ${prev_tilt_angle} 0"/>
     </joint>
     <joint name="soft_joint${s1}" type="revolute">
@@ -348,5 +351,5 @@
       <parent link="servo_link${i}"/>
       <child link="gimbal_link${i}"/>
-      <origin xyz="${servo_size_x} 0 0" rpy="0 ${tilt_angle} 0"/>
+      <origin xyz="${servo_size_x} 0 ${gimbal_tilt_z_offset}" rpy="0 ${tilt_angle} 0"/>
       <axis xyz="1 0 0"/>
       <dynamics damping="0.9" friction="0.1"/>

Commit message: flatten the model

File: robots/hydrus/mujoco/quad/soft_airframe_202605/robot.urdf (robot description, URDF)
Before this commit: robot serial_soft_airframe, 44 links, 43 joints
Joints:
- joint gimbal_joint1: origin xyz=0.096 0 -0.012724564326109165 rpy=0 0.174 0 -> xyz=0.096 0 0.012724564326109165 rpy=0 0.174 0
- joint gimbal_joint2: origin xyz=0.156 0 0.012724564326109165 rpy=0 -0.174 0 -> xyz=0.156 0 -0.012724564326109165 rpy=0 -0.174 0
- joint gimbal_joint3: origin xyz=0.096 0 -0.012724564326109165 rpy=0 0.174 0 -> xyz=0.096 0 0.012724564326109165 rpy=0 0.174 0
- joint gimbal_joint4: origin xyz=0.096 0 0.012724564326109165 rpy=0 -0.174 0 -> xyz=0.096 0 -0.012724564326109165 rpy=0 -0.174 0
- joint soft_joint1: origin xyz=0.0 0 -0.0 rpy=0 0 0 -> xyz=0.0 0 0.0 rpy=0 0 0
- joint soft_joint11: origin xyz=0.147 0 -0.02544912865221833 rpy=0 0.174 0 -> xyz=0.147 0 0.0 rpy=0 0.174 0
- joint soft_joint16: origin xyz=0.147 0 0.02544912865221833 rpy=0 -0.174 0 -> xyz=0.147 0 0.0 rpy=0 -0.174 0
- joint soft_joint6: origin xyz=0.147 0 0.02544912865221833 rpy=0 -0.174 0 -> xyz=0.147 0 0.0 rpy=0 -0.174 0

File: robots/hydrus/urdf/soft_link.urdf.xacro (robot description, xacro)
@@ -60,7 +60,7 @@
     <xacro:property name="l0" value="${2 * i - 1}" />
     <xacro:property name="l1" value="${2 * i}" />
-    <!-- Keep tilted module connections close to the original height. -->
-    <xacro:property name="parent_tilt_z_offset" value="${-parent_to_servo_x * sin(prev_tilt_angle)}" />
-    <xacro:property name="gimbal_tilt_z_offset" value="${-rotor_offset_x * sin(tilt_angle)}" />
+    <!-- Keep gimbal height aligned without shifting the upstream soft-link chain. -->
+    <xacro:property name="parent_tilt_z_offset" value="0.0" />
+    <xacro:property name="gimbal_tilt_z_offset" value="${rotor_offset_x * sin(tilt_angle)}" />
     <!-- Five-segment soft continuum approximation (1/8, 1/4, 1/4, 1/4, 1/8). -->
     <joint name="soft_joint${s0}" type="fixed">

Commit message: update urdf

File: robots/hydrus/mujoco/quad/soft_airframe_202605/robot.urdf (robot description, URDF)
Before this commit: robot serial_soft_airframe, 44 links, 43 joints
Links:
- link gimbal_link1: mass 0.222 -> 0.254
- link gimbal_link2: mass 0.222 -> 0.254
- link gimbal_link3: mass 0.222 -> 0.254
- link gimbal_link4: mass 0.222 -> 0.254
- link servo_link1: mass 0.141 -> 0.189
- link servo_link2: mass 0.18 -> 0.229
- link servo_link3: mass 0.141 -> 0.189
- link servo_link4: mass 0.141 -> 0.189
- link soft_link1: mass 0.0295 -> 0.031375
- link soft_link10: mass 0.0295 -> 0.038875
- link soft_link11: mass 0.0295 -> 0.038875
- link soft_link12: mass 0.059 -> 0.07775
- link soft_link13: mass 0.059 -> 0.07775
- link soft_link14: mass 0.059 -> 0.07775
- link soft_link15: mass 0.0295 -> 0.038875
- link soft_link16: mass 0.0295 -> 0.038875
- link soft_link17: mass 0.059 -> 0.07775
- link soft_link18: mass 0.059 -> 0.07775
- link soft_link19: mass 0.059 -> 0.07775
- link soft_link2: mass 0.059 -> 0.06275
- link soft_link20: mass 0.0295 -> 0.038875
- link soft_link3: mass 0.059 -> 0.06275
- link soft_link4: mass 0.059 -> 0.06275
- link soft_link5: mass 0.0295 -> 0.031375
- link soft_link6: mass 0.0295 -> 0.038875
- link soft_link7: mass 0.059 -> 0.07775
- link soft_link8: mass 0.059 -> 0.07775
- link soft_link9: mass 0.059 -> 0.07775
