Commit message: update urdf

File: robots/hydrus/mujoco/quad/soft_airframe_202605/robot.urdf (robot description, URDF)
Before this commit: robot serial_soft_airframe, 44 links, 43 joints
Links:
- link servo_link1: geometry collision box size=0.099 0.05 0.05; visual box size=0.099 0.05 0.05
- link servo_link2: geometry collision box size=0.149 0.06 0.01; visual box size=0.149 0.06 0.01
- link servo_link3: geometry collision box size=0.099 0.05 0.05; visual box size=0.099 0.05 0.05
- link servo_link4: geometry collision box size=0.099 0.05 0.05; visual box size=0.099 0.05 0.05
- link soft_link1: geometry collision box size=0.0615 0.03 0.04; visual box size=0.0615 0.03 0.04
- link soft_link10: geometry collision box size=0.0615 0.03 0.04; visual box size=0.0615 0.03 0.04
- link soft_link11: geometry collision box size=0.0615 0.03 0.04; visual box size=0.0615 0.03 0.04
- link soft_link12: geometry collision box size=0.123 0.03 0.04; visual box size=0.123 0.03 0.04
- link soft_link13: geometry collision box size=0.123 0.03 0.04; visual box size=0.123 0.03 0.04
- link soft_link14: geometry collision box size=0.123 0.03 0.04; visual box size=0.123 0.03 0.04
- link soft_link15: geometry collision box size=0.0615 0.03 0.04; visual box size=0.0615 0.03 0.04
- link soft_link16: geometry collision box size=0.0615 0.03 0.04; visual box size=0.0615 0.03 0.04
- link soft_link17: geometry collision box size=0.123 0.03 0.04; visual box size=0.123 0.03 0.04
- link soft_link18: geometry collision box size=0.123 0.03 0.04; visual box size=0.123 0.03 0.04
- link soft_link19: geometry collision box size=0.123 0.03 0.04; visual box size=0.123 0.03 0.04
- link soft_link2: geometry collision box size=0.123 0.03 0.04; visual box size=0.123 0.03 0.04
- link soft_link20: geometry collision box size=0.0615 0.03 0.04; visual box size=0.0615 0.03 0.04
- link soft_link3: geometry collision box size=0.123 0.03 0.04; visual box size=0.123 0.03 0.04
- link soft_link4: geometry collision box size=0.123 0.03 0.04; visual box size=0.123 0.03 0.04
- link soft_link5: geometry collision box size=0.0615 0.03 0.04; visual box size=0.0615 0.03 0.04
- link soft_link6: geometry collision box size=0.0615 0.03 0.04; visual box size=0.0615 0.03 0.04
- link soft_link7: geometry collision box size=0.123 0.03 0.04; visual box size=0.123 0.03 0.04
- link soft_link8: geometry collision box size=0.123 0.03 0.04; visual box size=0.123 0.03 0.04
- link soft_link9: geometry collision box size=0.123 0.03 0.04; visual box size=0.123 0.03 0.04
Joints:
- joint gimbal_joint1: origin xyz=0.096 0 0.012724564326109165 rpy=0 0.174 0 -> xyz=0.099 0 0.012724564326109165 rpy=0 0.174 0
- joint gimbal_joint2: origin xyz=0.156 0 -0.012724564326109165 rpy=0 -0.174 0 -> xyz=0.149 0 -0.012724564326109165 rpy=0 -0.174 0
- joint gimbal_joint3: origin xyz=0.096 0 0.012724564326109165 rpy=0 0.174 0 -> xyz=0.099 0 0.012724564326109165 rpy=0 0.174 0
- joint gimbal_joint4: origin xyz=0.096 0 -0.012724564326109165 rpy=0 -0.174 0 -> xyz=0.099 0 -0.012724564326109165 rpy=0 -0.174 0
- joint leg_joint2: origin xyz=0.05875 0 -0.041 rpy=0 0 0 -> xyz=0.0615 0 -0.041 rpy=0 0 0
- joint leg_joint4: origin xyz=0.05875 0 -0.041 rpy=0 0 0 -> xyz=0.0615 0 -0.041 rpy=0 0 0
- joint leg_joint6: origin xyz=0.05875 0 -0.041 rpy=0 0 0 -> xyz=0.0615 0 -0.041 rpy=0 0 0
- joint leg_joint8: origin xyz=0.05875 0 -0.041 rpy=0 0 0 -> xyz=0.0615 0 -0.041 rpy=0 0 0
- joint servo_joint1: origin xyz=0.05875 0 0 rpy=0 0 0 -> xyz=0.0615 0 0 rpy=0 0 0
- joint servo_joint2: origin xyz=0.05875 0 0 rpy=0 0 0 -> xyz=0.0615 0 0 rpy=0 0 0
- joint servo_joint3: origin xyz=0.05875 0 0 rpy=0 0 0 -> xyz=0.0615 0 0 rpy=0 0 0
- joint servo_joint4: origin xyz=0.05875 0 0 rpy=0 0 0 -> xyz=0.0615 0 0 rpy=0 0 0
- joint soft_joint10: origin xyz=0.1175 0 0 rpy=0 0 0 -> xyz=0.123 0 0 rpy=0 0 0
- joint soft_joint11: origin xyz=0.147 0 0.0 rpy=0 0.174 0 -> xyz=0.15 0 0.0 rpy=0 0.174 0
- joint soft_joint12: origin xyz=0.05875 0 0 rpy=0 0 0 -> xyz=0.0615 0 0 rpy=0 0 0
- joint soft_joint13: origin xyz=0.1175 0 0 rpy=0 0 0 -> xyz=0.123 0 0 rpy=0 0 0
- joint soft_joint14: origin xyz=0.1175 0 0 rpy=0 0 0 -> xyz=0.123 0 0 rpy=0 0 0
- joint soft_joint15: origin xyz=0.1175 0 0 rpy=0 0 0 -> xyz=0.123 0 0 rpy=0 0 0
- joint soft_joint16: origin xyz=0.147 0 0.0 rpy=0 -0.174 0 -> xyz=0.15 0 0.0 rpy=0 -0.174 0
- joint soft_joint17: origin xyz=0.05875 0 0 rpy=0 0 0 -> xyz=0.0615 0 0 rpy=0 0 0
- joint soft_joint18: origin xyz=0.1175 0 0 rpy=0 0 0 -> xyz=0.123 0 0 rpy=0 0 0
- joint soft_joint19: origin xyz=0.1175 0 0 rpy=0 0 0 -> xyz=0.123 0 0 rpy=0 0 0
- joint soft_joint2: origin xyz=0.05875 0 0 rpy=0 0 0 -> xyz=0.0615 0 0 rpy=0 0 0
- joint soft_joint20: origin xyz=0.1175 0 0 rpy=0 0 0 -> xyz=0.123 0 0 rpy=0 0 0
- joint soft_joint3: origin xyz=0.1175 0 0 rpy=0 0 0 -> xyz=0.123 0 0 rpy=0 0 0
- joint soft_joint4: origin xyz=0.1175 0 0 rpy=0 0 0 -> xyz=0.123 0 0 rpy=0 0 0
- joint soft_joint5: origin xyz=0.1175 0 0 rpy=0 0 0 -> xyz=0.123 0 0 rpy=0 0 0
- joint soft_joint6: origin xyz=0.147 0 0.0 rpy=0 -0.174 0 -> xyz=0.15 0 0.0 rpy=0 -0.174 0
- joint soft_joint7: origin xyz=0.05875 0 0 rpy=0 0 0 -> xyz=0.0615 0 0 rpy=0 0 0
- joint soft_joint8: origin xyz=0.1175 0 0 rpy=0 0 0 -> xyz=0.123 0 0 rpy=0 0 0
- joint soft_joint9: origin xyz=0.1175 0 0 rpy=0 0 0 -> xyz=0.123 0 0 rpy=0 0 0

File: robots/hydrus/robots/quad/soft_airframe_202605/robot.urdf.xacro (robot description, xacro)
@@ -53,19 +53,19 @@
   <!-- Four soft-link modules connected in series.
        Module i creates:
-         servo_link{i}, soft_link{3*i-2}, soft_link{3*i-1}, soft_link{3*i}, gimbal_link{i}, thrust{i}
+         soft_link{5*i-4} ... soft_link{5*i}, servo_link{i}, leg{2*i-1}, leg{2*i}, gimbal_link{i}, thrust{i}
   -->
   <xacro:soft_link_module
-      i="1"
+      module_index="1"
       parent="root"
       rotor_direction="-1"
-      parent_to_servo_x="0.0"
+      parent_to_soft_root_x="0.0"
       prev_tilt_angle="0"
       tilt_angle="0.174"
       soft_weight_sum="0.251" />
   <xacro:soft_link_module
-      i="2"
+      module_index="2"
       parent="gimbal_link1"
       rotor_direction="1"
-      servo_size_x="0.156"
+      servo_size_x="0.149"
       servo_size_y="0.06"
       servo_size_z="0.01"
@@ -75,5 +75,5 @@
   <!-- The third module has a slightly longer and larger servo body. -->
   <xacro:soft_link_module
-      i="3"
+      module_index="3"
       parent="gimbal_link2"
       rotor_direction="-1"
@@ -81,5 +81,5 @@
       tilt_angle="0.174" />
   <xacro:soft_link_module
-      i="4"
+      module_index="4"
       parent="gimbal_link3"
       rotor_direction="1"

File: robots/hydrus/urdf/soft_link.urdf.xacro (robot description, xacro)
@@ -18,28 +18,28 @@
   <!--
     A macro for one soft-link module.
-    Module i consists of:
-      - soft_link${5*i-4}, soft_link${5*i-3}, soft_link${5*i-2}, soft_link${5*i-1}, soft_link${5*i}
-      - servo_link${i}: a single combined servo body corresponding to old servo_link(2*i-1) + servo_link(2*i)
-      - leg${2*i-1}: attached at the root of soft_link${5*i-4}
-      - leg${2*i}: attached at the tip of soft_link${5*i}
-      - gimbal_link${i}
-      - thrust${i}
-    The next module should usually use parent="gimbal_link${i}".
+    Module ${module_index} consists of:
+      - soft_link${5*module_index-4} ... soft_link${5*module_index}
+      - servo_link${module_index}: a single combined servo body
+      - leg${2*module_index-1}: attached at the root of the first soft link
+      - leg${2*module_index}: attached at the tip of the fifth soft link
+      - gimbal_link${module_index}
+      - thrust${module_index}
+    The next module should usually use parent="gimbal_link${module_index}".
   -->
   <xacro:macro name="soft_link_module" params="
-      i
+      module_index
       parent
       rotor_direction:=1
-      parent_to_servo_x:=0.147
-      parent_to_servo_cog:=0.0567
-      servo_size_x:=0.096
+      parent_to_soft_root_x:=0.150
+      servo_cog_x:=0.0495
+      servo_size_x:=0.099
       servo_size_y:=0.05
       servo_size_z:=0.05
       servo_mass:=0.189
-      soft_l1:=0.05875
-      soft_l2:=0.1175
-      soft_l3:=0.1175
-      soft_l4:=0.1175
-      soft_l5:=0.05875
+      soft_l1:=0.0615
+      soft_l2:=0.123
+      soft_l3:=0.123
+      soft_l4:=0.123
+      soft_l5:=0.0615
       soft_width:=0.03
       soft_height:=0.04
@@ -54,27 +54,19 @@
       gimbal_mesh:=package://hydrus/urdf/mesh/5inch_propeller_duct_right_v2.dae
       propeller_mesh:=package://hydrus/urdf/mesh/TriBlade_5045.dae">
-    <xacro:property name="s0" value="${5 * i - 4}" />
-    <xacro:property name="s1" value="${5 * i - 3}" />
-    <xacro:property name="s2" value="${5 * i - 2}" />
-    <xacro:property name="s3" value="${5 * i - 1}" />
-    <xacro:property name="s4" value="${5 * i}" />
-    <xacro:property name="l0" value="${2 * i - 1}" />
-    <xacro:property name="l1" value="${2 * i}" />
+    <xacro:property name="s1" value="${5 * module_index - 4}" />
+    <xacro:property name="s2" value="${5 * module_index - 3}" />
+    <xacro:property name="s3" value="${5 * module_index - 2}" />
+    <xacro:property name="s4" value="${5 * module_index - 1}" />
+    <xacro:property name="s5" value="${5 * module_index}" />
+    <xacro:property name="l1" value="${2 * module_index - 1}" />
+    <xacro:property name="l2" value="${2 * module_index}" />
     <!-- Keep gimbal height aligned without shifting the upstream soft-link chain. -->
-    <xacro:property name="parent_tilt_z_offset" value="0.0" />
+    <xacro:property name="soft_root_tilt_z_offset" value="0.0" />
     <xacro:property name="gimbal_tilt_z_offset" value="${rotor_offset_x * sin(tilt_angle)}" />
     <!-- Five-segment soft continuum approximation (1/8, 1/4, 1/4, 1/4, 1/8). -->
-    <joint name="soft_joint${s0}" type="fixed">
+    <joint name="soft_joint${s1}" type="fixed">
       <parent link="${parent}"/>
-      <child link="soft_link${s0}"/>
-      <origin xyz="${parent_to_servo_x} 0 ${parent_tilt_z_offset}" rpy="0 ${prev_tilt_angle} 0"/>
-    </joint>
-    <joint name="soft_joint${s1}" type="revolute">
-      <limit effort="5.0" lower="${-pi}" upper="${pi}" velocity="0.5"/>
-      <parent link="soft_link${s0}"/>
       <child link="soft_link${s1}"/>
-      <origin xyz="${soft_l1} 0 0" rpy="0 0 0"/>
-      <axis xyz="0 0 1"/>
-      <dynamics damping="0.2" friction="0.1"/>
+      <origin xyz="${parent_to_soft_root_x} 0 ${soft_root_tilt_z_offset}" rpy="0 ${prev_tilt_angle} 0"/>
     </joint>
     <joint name="soft_joint${s2}" type="revolute">
@@ -82,5 +74,5 @@
       <parent link="soft_link${s1}"/>
       <child link="soft_link${s2}"/>
-      <origin xyz="${soft_l2} 0 0" rpy="0 0 0"/>
+      <origin xyz="${soft_l1} 0 0" rpy="0 0 0"/>
       <axis xyz="0 0 1"/>
       <dynamics damping="0.2" friction="0.1"/>
@@ -90,5 +82,5 @@
       <parent link="soft_link${s2}"/>
       <child link="soft_link${s3}"/>
-      <origin xyz="${soft_l3} 0 0" rpy="0 0 0"/>
+      <origin xyz="${soft_l2} 0 0" rpy="0 0 0"/>
       <axis xyz="0 0 1"/>
       <dynamics damping="0.2" friction="0.1"/>
@@ -98,9 +90,17 @@
       <parent link="soft_link${s3}"/>
       <child link="soft_link${s4}"/>
+      <origin xyz="${soft_l3} 0 0" rpy="0 0 0"/>
+      <axis xyz="0 0 1"/>
+      <dynamics damping="0.2" friction="0.1"/>
+    </joint>
+    <joint name="soft_joint${s5}" type="revolute">
+      <limit effort="5.0" lower="${-pi}" upper="${pi}" velocity="0.5"/>
+      <parent link="soft_link${s4}"/>
+      <child link="soft_link${s5}"/>
       <origin xyz="${soft_l4} 0 0" rpy="0 0 0"/>
       <axis xyz="0 0 1"/>
       <dynamics damping="0.2" friction="0.1"/>
     </joint>
-    <link name="soft_link${s0}">
+    <link name="soft_link${s1}">
       <inertial>
         <origin xyz="${soft_l1 * 0.5} 0.000002 0" rpy="0 0 0"/>
@@ -119,10 +119,10 @@
       </visual>
     </link>
-    <gazebo reference="soft_link${s0}">
-      <mu1>0.1</mu1>
-      <mu2>0.1</mu2>
-    </gazebo>
-    <xacro:damping_factor link="soft_link${s0}"/>
-    <link name="soft_link${s1}">
+    <gazebo reference="soft_link${s1}">
+      <mu1>0.1</mu1>
+      <mu2>0.1</mu2>
+    </gazebo>
+    <xacro:damping_factor link="soft_link${s1}"/>
+    <link name="soft_link${s2}">
       <inertial>
         <origin xyz="${soft_l2 * 0.5} 0.000002 0" rpy="0 0 0"/>
@@ -141,10 +141,10 @@
       </visual>
     </link>
-    <gazebo reference="soft_link${s1}">
-      <mu1>0.1</mu1>
-      <mu2>0.1</mu2>
-    </gazebo>
-    <xacro:damping_factor link="soft_link${s1}"/>
-    <link name="soft_link${s2}">
+    <gazebo reference="soft_link${s2}">
+      <mu1>0.1</mu1>
+      <mu2>0.1</mu2>
+    </gazebo>
+    <xacro:damping_factor link="soft_link${s2}"/>
+    <link name="soft_link${s3}">
       <inertial>
         <origin xyz="${soft_l3 * 0.5} 0.000002 0" rpy="0 0 0"/>
@@ -163,10 +163,10 @@
       </visual>
     </link>
-    <gazebo reference="soft_link${s2}">
-      <mu1>0.1</mu1>
-      <mu2>0.1</mu2>
-    </gazebo>
-    <xacro:damping_factor link="soft_link${s2}"/>
-    <link name="soft_link${s3}">
+    <gazebo reference="soft_link${s3}">
+      <mu1>0.1</mu1>
+      <mu2>0.1</mu2>
+    </gazebo>
+    <xacro:damping_factor link="soft_link${s3}"/>
+    <link name="soft_link${s4}">
       <inertial>
         <origin xyz="${soft_l4 * 0.5} 0.000002 0" rpy="0 0 0"/>
@@ -185,10 +185,10 @@
       </visual>
     </link>
-    <gazebo reference="soft_link${s3}">
-      <mu1>0.1</mu1>
-      <mu2>0.1</mu2>
-    </gazebo>
-    <xacro:damping_factor link="soft_link${s3}"/>
-    <link name="soft_link${s4}">
+    <gazebo reference="soft_link${s4}">
+      <mu1>0.1</mu1>
+      <mu2>0.1</mu2>
+    </gazebo>
+    <xacro:damping_factor link="soft_link${s4}"/>
+    <link name="soft_link${s5}">
       <inertial>
         <origin xyz="${soft_l5 * 0.5} 0.000002 0" rpy="0 0 0"/>
@@ -207,18 +207,18 @@
       </visual>
     </link>
-    <gazebo reference="soft_link${s4}">
-      <mu1>0.1</mu1>
-      <mu2>0.1</mu2>
-    </gazebo>
-    <xacro:damping_factor link="soft_link${s4}"/>
+    <gazebo reference="soft_link${s5}">
+      <mu1>0.1</mu1>
+      <mu2>0.1</mu2>
+    </gazebo>
+    <xacro:damping_factor link="soft_link${s5}"/>
     <!-- Combined servo body after the soft-link chain. -->
-    <joint name="servo_joint${i}" type="fixed">
-      <parent link="soft_link${s4}"/>
-      <child link="servo_link${i}"/>
+    <joint name="servo_joint${module_index}" type="fixed">
+      <parent link="soft_link${s5}"/>
+      <child link="servo_link${module_index}"/>
       <origin xyz="${soft_l5} 0 0" rpy="0 0 0"/>
     </joint>
-    <link name="servo_link${i}">
-      <inertial>
-        <origin xyz="${parent_to_servo_cog} 0 0" rpy="0 0 0"/>
+    <link name="servo_link${module_index}">
+      <inertial>
+        <origin xyz="${servo_cog_x} 0 0" rpy="0 0 0"/>
         <mass value="${servo_mass}"/>
         <inertia
@@ -232,19 +232,19 @@
         </geometry>
         <material name="servo_link_material"/>
-        <origin xyz="${parent_to_servo_cog} 0 0" rpy="0 0 0"/>
-      </visual>
-    </link>
-    <gazebo reference="servo_link${i}">
-      <mu1>0.1</mu1>
-      <mu2>0.1</mu2>
-    </gazebo>
-    <xacro:damping_factor link="servo_link${i}"/>
-    <!-- Leg attached at the root of soft_link${s0}: leg${l0} -->
-    <joint name="leg_joint${l0}" type="fixed">
-      <parent link="soft_link${s0}"/>
-      <child link="leg${l0}"/>
+        <origin xyz="${servo_cog_x} 0 0" rpy="0 0 0"/>
+      </visual>
+    </link>
+    <gazebo reference="servo_link${module_index}">
+      <mu1>0.1</mu1>
+      <mu2>0.1</mu2>
+    </gazebo>
+    <xacro:damping_factor link="servo_link${module_index}"/>
+    <!-- Leg attached at the root of the first soft link: leg${l1} -->
+    <joint name="leg_joint${l1}" type="fixed">
+      <parent link="soft_link${s1}"/>
+      <child link="leg${l1}"/>
       <origin xyz="0 0 -0.041" rpy="0 0 0"/>
     </joint>
-    <link name="leg${l0}">
+    <link name="leg${l1}">
       <inertial>
         <origin xyz="0 0 -0.096" rpy="0 0 0"/>
@@ -269,16 +269,16 @@
       </collision>
     </link>
-    <gazebo reference="leg${l0}">
-      <mu1>0.1</mu1>
-      <mu2>0.1</mu2>
-    </gazebo>
-    <xacro:damping_factor link="leg${l0}"/>
-    <!-- Leg attached at the tip of soft_link${s4}: leg${l1} -->
-    <joint name="leg_joint${l1}" type="fixed">
-      <parent link="soft_link${s4}"/>
-      <child link="leg${l1}"/>
+    <gazebo reference="leg${l1}">
+      <mu1>0.1</mu1>
+      <mu2>0.1</mu2>
+    </gazebo>
+    <xacro:damping_factor link="leg${l1}"/>
+    <!-- Leg attached at the tip of the fifth soft link: leg${l2} -->
+    <joint name="leg_joint${l2}" type="fixed">
+      <parent link="soft_link${s5}"/>
+      <child link="leg${l2}"/>
       <origin xyz="${soft_l5} 0 -0.041" rpy="0 0 0"/>
     </joint>
-    <link name="leg${l1}">
+    <link name="leg${l2}">
       <inertial>
         <origin xyz="0 0 -0.096" rpy="0 0 0"/>
@@ -303,19 +303,9 @@
       </collision>
     </link>
-    <gazebo reference="leg${l1}">
-      <mu1>0.1</mu1>
-      <mu2>0.1</mu2>
-    </gazebo>
-    <xacro:damping_factor link="leg${l1}"/>
-    <transmission name="soft_joint_tran_${s1}">
-      <type>transmission_interface/SimpleTransmission</type>
-      <joint name="soft_joint${s1}">
-        <hardwareInterface>hardware_interface/EffortJointInterface</hardwareInterface>
-      </joint>
-      <actuator name="soft_joint_servo${s1}">
-        <hardwareInterface>hardware_interface/EffortJointInterface</hardwareInterface>
-        <mechanicalReduction>1</mechanicalReduction>
-      </actuator>
-    </transmission>
+    <gazebo reference="leg${l2}">
+      <mu1>0.1</mu1>
+      <mu2>0.1</mu2>
+    </gazebo>
+    <xacro:damping_factor link="leg${l2}"/>
     <transmission name="soft_joint_tran_${s2}">
       <type>transmission_interface/SimpleTransmission</type>
@@ -348,13 +338,23 @@
       </actuator>
     </transmission>
+    <transmission name="soft_joint_tran_${s5}">
+      <type>transmission_interface/SimpleTransmission</type>
+      <joint name="soft_joint${s5}">
+        <hardwareInterface>hardware_interface/EffortJointInterface</hardwareInterface>
+      </joint>
+      <actuator name="soft_joint_servo${s5}">
+        <hardwareInterface>hardware_interface/EffortJointInterface</hardwareInterface>
+        <mechanicalReduction>1</mechanicalReduction>
+      </actuator>
+    </transmission>
     <!-- Gimbal and rotor. -->
-    <joint name="gimbal_joint${i}" type="fixed">
-      <parent link="servo_link${i}"/>
-      <child link="gimbal_link${i}"/>
+    <joint name="gimbal_joint${module_index}" type="fixed">
+      <parent link="servo_link${module_index}"/>
+      <child link="gimbal_link${module_index}"/>
       <origin xyz="${servo_size_x} 0 ${gimbal_tilt_z_offset}" rpy="0 ${tilt_angle} 0"/>
       <axis xyz="1 0 0"/>
       <dynamics damping="0.9" friction="0.1"/>
     </joint>
-    <link name="gimbal_link${i}">
+    <link name="gimbal_link${module_index}">
       <inertial>
         <origin xyz="0.0735 0 0" rpy="0 0 0"/>
@@ -374,17 +374,17 @@
       </visual>
     </link>
-    <gazebo reference="gimbal_link${i}">
-      <mu1>0.1</mu1>
-      <mu2>0.1</mu2>
-    </gazebo>
-    <xacro:damping_factor link="gimbal_link${i}"/>
-    <joint name="rotor${i}" type="continuous">
+    <gazebo reference="gimbal_link${module_index}">
+      <mu1>0.1</mu1>
+      <mu2>0.1</mu2>
+    </gazebo>
+    <xacro:damping_factor link="gimbal_link${module_index}"/>
+    <joint name="rotor${module_index}" type="continuous">
       <limit effort="0.0064" lower="0.0" upper="20.0" velocity="0.5"/>
-      <parent link="gimbal_link${i}"/>
-      <child link="thrust${i}"/>
+      <parent link="gimbal_link${module_index}"/>
+      <child link="thrust${module_index}"/>
       <origin xyz="${rotor_offset_x} 0 0" rpy="0 0 0"/>
       <axis xyz="0 0 ${rotor_direction}"/>
     </joint>
-    <link name="thrust${i}">
+    <link name="thrust${module_index}">
       <inertial>
         <origin xyz="0 0 0" rpy="0 0 0"/>
@@ -403,11 +403,11 @@
       </visual>
     </link>
-    <xacro:damping_factor link="thrust${i}"/>
-    <transmission name="rotor_tran${i}">
+    <xacro:damping_factor link="thrust${module_index}"/>
+    <transmission name="rotor_tran${module_index}">
       <type>transmission_interface/SimpleTransmission</type>
-      <joint name="rotor${i}">
+      <joint name="rotor${module_index}">
         <hardwareInterface>RotorInterface</hardwareInterface>
       </joint>
-      <actuator name="rotor${i}">
+      <actuator name="rotor${module_index}">
         <hardwareInterface>RotorInterface</hardwareInterface>
         <mechanicalReduction>1</mechanicalReduction>
